Commit message: move sonar files

File: sonar_dave_plugins/urdf/sonar_snippets.xacro (robot description, xacro)
@@ -218,5 +218,5 @@
           </save>
         </camera>
-	    <plugin filename="libimage_sonar_ros_plugin.so" name="forward_sonar${suffix}_controller">
+	    <plugin filename="libimage_sonar_dave_plugin.so" name="forward_sonar${suffix}_controller">
 		  <topicName>${topic}</topicName>
           <frameName>forward_sonar${suffix}_optical_frame</frameName>

File: uuv_dave/urdf/rexrov_oberon7.xacro (robot description, xacro)
@@ -51,4 +51,9 @@
     </xacro:fl_multibeam_generic>
 -->
+<!-- creates beam lines in Gazebo view
+  <xacro:forward_multibeam_sonar_m450_130 namespace="$(arg namespace)" parent_link="$(arg namespace)/base_link">
+    <origin xyz="1.4 0 0.65" rpy="0 0 0"/>
+  </xacro:forward_multibeam_sonar_m450_130>
+-->
   <!-- Create the ROV -->
   <xacro:rexrov_base

File: uuv_dave/urdf/sensor_snippets.xacro (robot description, xacro)
@@ -20,5 +20,5 @@
   <xacro:include filename="$(find uuv_sensor_ros_plugins)/urdf/dvl_snippets.xacro" />
   <xacro:include filename="$(find uuv_sensor_ros_plugins)/urdf/rpt_snippets.xacro" />
-  <xacro:include filename="$(find uuv_dave)/urdf/sonar_snippets.xacro" />
+  <xacro:include filename="$(find sonar_dave_plugins)/urdf/sonar_snippets.xacro" />
   <xacro:include filename="$(find uuv_sensor_ros_plugins)/urdf/stereo_snippets.xacro" />
   <xacro:include filename="$(find uuv_sensor_ros_plugins)/urdf/gps_sensor_snippets.xacro" />

Commit message: rename sonar macros

File: sonar_dave_plugins/urdf/sonar_snippets.xacro (robot description, xacro)
@@ -23,5 +23,5 @@
   </xacro:macro>
   <!-- Side scan sonar -->
-  <xacro:macro name="sidescan_sonar" params="namespace parent_link suffix *origin">
+  <xacro:macro name="uuv_sidescan_sonar" params="namespace parent_link suffix *origin">
     <xacro:multibeam_sonar
       namespace="${namespace}"
@@ -48,5 +48,5 @@
   </xacro:macro>
   <!-- Inspired by m450-130: http://www.blueview.com/products/2d-imaging-sonar/m900-series/ -->
-  <xacro:macro name="forward_multibeam_sonar_m450_130" params="namespace parent_link *origin">
+  <xacro:macro name="uuv_forward_multibeam_sonar_m450_130" params="namespace parent_link *origin">
     <xacro:multibeam_sonar
       namespace="${namespace}"
@@ -71,5 +71,5 @@
     </xacro:multibeam_sonar>
   </xacro:macro>
-  <xacro:macro name="forward_multibeam_p900" params="namespace parent_link *origin">
+  <xacro:macro name="uuv_forward_multibeam_p900" params="namespace parent_link *origin">
     <xacro:multibeam_sonar
       namespace="${namespace}"
@@ -95,5 +95,5 @@
   </xacro:macro>
 <!-- forward_looking_multibeam_sonar is not defined.
-  <xacro:macro name="fl_multibeam_generic" params="namespace parent_link *origin">
+  <xacro:macro name="uuv_fl_multibeam_generic" params="namespace parent_link *origin">
     <xacro:forward_looking_multibeam_sonar
       namespace="${namespace}"
@@ -119,5 +119,5 @@
   </xacro:macro>
 -->
-  <xacro:macro name="multibeam_sonar"
+  <xacro:macro name="uuv_multibeam_sonar"
     params="namespace suffix parent_link topic mass update_rate
       samples fov range_min range_max range_stddev mesh
@@ -177,5 +177,5 @@
   </gazebo>
   </xacro:macro>
-  <xacro:macro name="forward_looking_sonar"
+  <xacro:macro name="uuv_forward_looking_sonar"
     params="namespace suffix parent_link topic mass update_rate
       samples fov width height *inertia *origin *visual">

File: uuv_dave/urdf/rexrov_oberon7.xacro (robot description, xacro)
@@ -20,5 +20,5 @@
   <xacro:include filename="$(find uuv_descriptions)/urdf/rexrov.gazebo.xacro"/>
   <xacro:include filename="$(find oberon7_description)/robots/oberon7_default.xacro" />
-  <xacro:forward_looking_sonar
+  <xacro:uuv_forward_looking_sonar
       namespace="${namespace}"
       suffix="down"
@@ -36,23 +36,23 @@
       <visual>
       </visual>
-    </xacro:forward_looking_sonar>
+    </xacro:uuv_forward_looking_sonar>
 <!--
-  <xacro:forward_multibeam_p900
+  <xacro:uuv_forward_multibeam_p900
       namespace="${namespace}"
       parent_link="${namespace}/base_link">
       <origin xyz="1.15 0 0.4" rpy="0 0.3 0"/>
-    </xacro:forward_multibeam_p900>
+    </xacro:uuv_forward_multibeam_p900>
 -->
 <!--
-  <xacro:fl_multibeam_generic
+  <xacro:uuv_fl_multibeam_generic
       namespace="${namespace}"
       parent_link="${namespace}/base_link">
       <origin xyz="1.15 0 0.4" rpy="0 0.3 0"/>
-    </xacro:fl_multibeam_generic>
+    </xacro:uuv_fl_multibeam_generic>
 -->
 <!-- creates beam lines in Gazebo view
-  <xacro:forward_multibeam_sonar_m450_130 namespace="$(arg namespace)" parent_link="$(arg namespace)/base_link">
+  <xacro:uuv_forward_multibeam_sonar_m450_130 namespace="$(arg namespace)" parent_link="$(arg namespace)/base_link">
     <origin xyz="1.4 0 0.65" rpy="0 0 0"/>
-  </xacro:forward_multibeam_sonar_m450_130>
+  </xacro:uuv_forward_multibeam_sonar_m450_130>
 -->
   <!-- Create the ROV -->
