Commit message: Fixed topic naming error in the DVL plugin
Individual beam topic names now set correctly in the DVL plugin.

File: dvl_gazebo/urdf/teledyne_whn.xacro (robot description, xacro)
@@ -60,5 +60,5 @@
   </xacro:macro>
   <!-- Generates a single ranging sonar for the DVL -->
-  <xacro:macro name="dvl_single_sonar" params="namespace suffix index pitch yaw update_rate">
+  <xacro:macro name="dvl_single_sonar" params="namespace topic suffix index pitch yaw update_rate">
     <link name="${namespace}/dvl${suffix}_sonar${index}_link">
       <inertial>
@@ -106,5 +106,5 @@
           <alwaysOn>true</alwaysOn>
           <updateRate>${update_rate}</updateRate>
-          <topicName>${topic}_sonar${index}</topicName>
+          <topicName>${namespace}/${topic}${suffix}_sonar${index}</topicName>
           <frameName>${namespace}/dvl${suffix}_sonar${index}_link</frameName>
           <fov>0.06</fov>
@@ -149,17 +149,17 @@
     </joint>
     <xacro:dvl_single_sonar
-      namespace="${namespace}" suffix=""
+      namespace="${namespace}" topic="${topic}" suffix=""
       index="0" pitch="-0.52" yaw="0.0" update_rate="${update_rate}">
     </xacro:dvl_single_sonar>
     <xacro:dvl_single_sonar
-      namespace="${namespace}" suffix=""
+      namespace="${namespace}" topic="${topic}" suffix=""
       index="1" pitch="0" yaw="0.52" update_rate="${update_rate}">
     </xacro:dvl_single_sonar>
     <xacro:dvl_single_sonar
-      namespace="${namespace}" suffix=""
+      namespace="${namespace}" topic="${topic}" suffix=""
       index="2" pitch="0.52" yaw="0.0" update_rate="${update_rate}">
     </xacro:dvl_single_sonar>
     <xacro:dvl_single_sonar
-      namespace="${namespace}" suffix=""
+      namespace="${namespace}" topic="${topic}" suffix=""
       index="3" pitch="0.0" yaw="-0.52" update_rate="${update_rate}">
     </xacro:dvl_single_sonar>
@@ -168,5 +168,5 @@
         <robot_namespace>${namespace}</robot_namespace> <!-- (string, required): ros namespace in which the messages are published -->
         <link_name>${parent_link}</link_name> <!-- (string, required): name of the body which holds the IMU sensor -->
-        <sensor_topic>${topic}</sensor_topic> <!-- (string): name of the sensor output topic and prefix of service names -->
+        <sensor_topic>${topic}${suffix}</sensor_topic> <!-- (string): name of the sensor output topic and prefix of service names -->
         <update_rate>${update_rate}</update_rate> <!-- Update period [s] -->
         <noise_sigma>${noise_sigma}</noise_sigma> <!-- std dev of position estimates in x, y, z [m/s] -->
@@ -181,8 +181,8 @@
         <beam_link_name_3>${namespace}/dvl_sonar3_link</beam_link_name_3>
         <!-- Declaring the beam output topics -->
-        <beam_topic_0>${topic}_sonar0</beam_topic_0>
-        <beam_topic_1>${topic}_sonar1</beam_topic_1>
-        <beam_topic_2>${topic}_sonar2</beam_topic_2>
-        <beam_topic_3>${topic}_sonar3</beam_topic_3>
+        <beam_topic_0>${topic}${suffix}_sonar0</beam_topic_0>
+        <beam_topic_1>${topic}${suffix}_sonar1</beam_topic_1>
+        <beam_topic_2>${topic}${suffix}_sonar2</beam_topic_2>
+        <beam_topic_3>${topic}${suffix}_sonar3</beam_topic_3>
       </plugin>
     </gazebo>
