Commit message: Created Xacro files for performer identified DVLs
Nortek DVL500-300m
Nortek DVL500-4000m
Nortek DVL1000-300m
Nortek DVL1000-4000m
Sonardyne Syrinx 600
Teledyne Explorer 1000 (Phased Array)
Teledyne Explorer 4000 (Piston)

File: dvl_gazebo/urdf/nortek_dvl500_4000.xacro (robot description, xacro)
@@ -10,5 +10,5 @@
      limitations under the License.
 -->
-<!-- Xacro macros for generating Teledyne Workhorse Navigator (WHN) class URDF models
+<!-- Xacro macros for generating Nortek DVL500-4000 URDF models
      utilizing the uuv_simulator DVL plugin (libuuv_gazebo_ros_dvl_plugin.so)
      Adapted from uuv_simulator version (uuv_sensor_ros_plugins/urdf/dvl_snippets.xacro)
@@ -25,6 +25,6 @@
     </collision>
   </xacro:macro>
-  <!-- Generates a Teledyne WHN URDF model and attaches it to a parent link
-       Sensor parameters align with those in the WHN 600 datasheet -->
+  <!-- Generates a Nortek DVL500-4000m URDF model and attaches it to a parent link
+       Sensor parameters align with those in the DVL500-4000m datasheet -->
   <xacro:macro name="dvl_macro" params="namespace parent_link *origin inertial_reference_frame">
     <xacro:dvl_plugin_macro
@@ -33,5 +33,5 @@
       parent_link="${parent_link}"
       reference_frame="${inertial_reference_frame}"
-      update_rate="7"
+      update_rate="8"
       topic="dvl"
       noise_sigma="0.005"
@@ -41,5 +41,5 @@
     </xacro:dvl_plugin_macro>
   </xacro:macro>
-  <!-- Generates an ENU Teledyne WHN URDF model and attaches it to a parent link -->
+  <!-- Generates an ENU Nortek DVL500-4000 URDF model and attaches it to a parent link -->
   <xacro:macro name="dvl_sensor_enu" params="namespace parent_link *origin">
     <xacro:dvl_macro
@@ -50,5 +50,5 @@
     </xacro:dvl_macro>
   </xacro:macro>
-  <!-- Generates an NED Teledyne WHN URDF model and attaches it to a parent link -->
+  <!-- Generates an NED Nortek DVL500-4000 URDF model and attaches it to a parent link -->
   <xacro:macro name="dvl_sensor_ned" params="namespace parent_link *origin">
     <xacro:dvl_macro
@@ -86,17 +86,17 @@
               <samples>3</samples>
               <resolution>1</resolution>
-              <min_angle>-0.03</min_angle>
-              <max_angle>0.03</max_angle>
+              <min_angle>-0.025</min_angle>
+              <max_angle>0.025</max_angle>
             </horizontal>
             <vertical>
               <samples>3</samples>
               <resolution>1</resolution>
-              <min_angle>-0.03</min_angle>
-              <max_angle>0.03</max_angle>
+              <min_angle>-0.025</min_angle>
+              <max_angle>0.025</max_angle>
             </vertical>
           </scan>
           <range>
-            <min>0.7</min>
-            <max>90</max>
+            <min>0.3</min>
+            <max>200</max>
             <resolution>0.01</resolution>
           </range>
@@ -108,5 +108,5 @@
           <topicName>${namespace}/${topic}${suffix}_sonar${index}</topicName>
           <frameName>${namespace}/dvl${suffix}_sonar${index}_link</frameName>
-          <fov>0.06</fov>
+          <fov>0.05</fov>
           <radiation>ultrasound</radiation>
         </plugin>
@@ -125,10 +125,11 @@
     <link name="${namespace}/dvl${suffix}_link">
       <inertial>
-        <mass value="8.8"/>
+        <mass value="0.5"/>
         <origin xyz="0 0 0" rpy="0 0 0"/>
-        <inertia ixx="0.071732122" ixy="0" ixz="0" iyy="0.071732122" iyz="0" izz="0.055786544"/>
+        <inertia ixx="0.017348633333333" ixy="0" ixz="0" iyy="0.017348633333333" iyz="0" izz="0.01340595"/>
       </inertial>
       <visual>
         <geometry>
+        <!-- Replace with Nortek DVL500 mesh when available -->
         <mesh filename="package://dvl_gazebo/models/teledyne_whn/meshes/teledyne_whn.dae"/>
         </geometry>
@@ -136,5 +137,5 @@
       <collision>
         <geometry>
-          <cylinder length="0.2445" radius="0.1126"/>
+          <cylinder length="0.203" radius="0.093"/>
         </geometry>
         <origin xyz="0 0 0" rpy="0 1.5707963267948966 0"/>
@@ -150,25 +151,25 @@
     <xacro:dvl_single_sonar
       namespace="${namespace}" topic="${topic}" suffix=""
-      index="0" pitch="-0.52" yaw="0.0" update_rate="${update_rate}">
+      index="0" pitch="-0.4363" yaw="0.0" update_rate="${update_rate}">
     </xacro:dvl_single_sonar>
     <xacro:dvl_single_sonar
       namespace="${namespace}" topic="${topic}" suffix=""
-      index="1" pitch="0" yaw="0.52" update_rate="${update_rate}">
+      index="1" pitch="0" yaw="0.4363" update_rate="${update_rate}">
     </xacro:dvl_single_sonar>
     <xacro:dvl_single_sonar
       namespace="${namespace}" topic="${topic}" suffix=""
-      index="2" pitch="0.52" yaw="0.0" update_rate="${update_rate}">
+      index="2" pitch="0.4363" yaw="0.0" update_rate="${update_rate}">
     </xacro:dvl_single_sonar>
     <xacro:dvl_single_sonar
       namespace="${namespace}" topic="${topic}" suffix=""
-      index="3" pitch="0.0" yaw="-0.52" update_rate="${update_rate}">
+      index="3" pitch="0.0" yaw="-0.4363" update_rate="${update_rate}">
     </xacro:dvl_single_sonar>
     <gazebo>
       <plugin filename="libuuv_gazebo_ros_dvl_plugin.so" name="libuuv_gazebo_dvl${suffix}_plugin">
-        <robot_namespace>${namespace}</robot_namespace> <!-- (string, required): ros namespace in which the messages are published -->
-        <link_name>${parent_link}</link_name> <!-- (string, required): name of the body which holds the IMU sensor -->
-        <sensor_topic>${topic}${suffix}</sensor_topic> <!-- (string): name of the sensor output topic and prefix of service names -->
-        <update_rate>${update_rate}</update_rate> <!-- Update period [s] -->
-        <noise_sigma>${noise_sigma}</noise_sigma> <!-- std dev of position estimates in x, y, z [m/s] -->
+        <robot_namespace>${namespace}</robot_namespace>
+        <link_name>${parent_link}</link_name>
+        <sensor_topic>${topic}${suffix}</sensor_topic>
+        <update_rate>${update_rate}</update_rate>
+        <noise_sigma>${noise_sigma}</noise_sigma>
         <noise_amplitude>${noise_amplitude}</noise_amplitude>
         <enable_gazebo_messages>false</enable_gazebo_messages>

File: dvl_gazebo/urdf/sonardyne_syrinx600.xacro (robot description, xacro)
@@ -10,5 +10,5 @@
      limitations under the License.
 -->
-<!-- Xacro macros for generating Teledyne Workhorse Navigator (WHN) class URDF models
+<!-- Xacro macros for generating Sonardyne Syrinx 600 URDF models
      utilizing the uuv_simulator DVL plugin (libuuv_gazebo_ros_dvl_plugin.so)
      Adapted from uuv_simulator version (uuv_sensor_ros_plugins/urdf/dvl_snippets.xacro)
@@ -25,6 +25,6 @@
     </collision>
   </xacro:macro>
-  <!-- Generates a Teledyne WHN URDF model and attaches it to a parent link
-       Sensor parameters align with those in the WHN 600 datasheet -->
+  <!-- Generates a Sonardyne Syrinx 600 URDF model and attaches it to a parent link
+       Sensor parameters align with those in the Syrinx 600 datasheet -->
   <xacro:macro name="dvl_macro" params="namespace parent_link *origin inertial_reference_frame">
     <xacro:dvl_plugin_macro
@@ -33,13 +33,13 @@
       parent_link="${parent_link}"
       reference_frame="${inertial_reference_frame}"
-      update_rate="7"
+      update_rate="25"
       topic="dvl"
-      noise_sigma="0.005"
-      noise_amplitude="0.005"
+      noise_sigma="0.0022"
+      noise_amplitude="0.0022"
       scale="1">
       <xacro:insert_block name="origin"/>
     </xacro:dvl_plugin_macro>
   </xacro:macro>
-  <!-- Generates an ENU Teledyne WHN URDF model and attaches it to a parent link -->
+  <!-- Generates an ENU Sonardyne Syrinx 600 URDF model and attaches it to a parent link -->
   <xacro:macro name="dvl_sensor_enu" params="namespace parent_link *origin">
     <xacro:dvl_macro
@@ -50,5 +50,5 @@
     </xacro:dvl_macro>
   </xacro:macro>
-  <!-- Generates an NED Teledyne WHN URDF model and attaches it to a parent link -->
+  <!-- Generates an NED Sonardyne Syrinx 600 URDF model and attaches it to a parent link -->
   <xacro:macro name="dvl_sensor_ned" params="namespace parent_link *origin">
     <xacro:dvl_macro
@@ -86,17 +86,17 @@
               <samples>3</samples>
               <resolution>1</resolution>
-              <min_angle>-0.03</min_angle>
-              <max_angle>0.03</max_angle>
+              <min_angle>-0.013</min_angle>
+              <max_angle>0.013</max_angle>
             </horizontal>
             <vertical>
               <samples>3</samples>
               <resolution>1</resolution>
-              <min_angle>-0.03</min_angle>
-              <max_angle>0.03</max_angle>
+              <min_angle>-0.013</min_angle>
+              <max_angle>0.013</max_angle>
             </vertical>
           </scan>
           <range>
-            <min>0.7</min>
-            <max>90</max>
+            <min>0.4</min>
+            <max>175</max>
             <resolution>0.01</resolution>
           </range>
@@ -108,5 +108,5 @@
           <topicName>${namespace}/${topic}${suffix}_sonar${index}</topicName>
           <frameName>${namespace}/dvl${suffix}_sonar${index}_link</frameName>
-          <fov>0.06</fov>
+          <fov>0.026</fov>
           <radiation>ultrasound</radiation>
         </plugin>
@@ -125,10 +125,11 @@
     <link name="${namespace}/dvl${suffix}_link">
       <inertial>
-        <mass value="8.8"/>
+        <mass value="7.0"/>
         <origin xyz="0 0 0" rpy="0 0 0"/>
-        <inertia ixx="0.071732122" ixy="0" ixz="0" iyy="0.071732122" iyz="0" izz="0.055786544"/>
+        <inertia ixx="0.0429856875" ixy="0" ixz="0" iyy="0.0429856875" iyz="0" izz="0.044296875"/>
       </inertial>
       <visual>
         <geometry>
+        <!-- Replace with Sonardyne Syrinx 600 mesh when available -->
         <mesh filename="package://dvl_gazebo/models/teledyne_whn/meshes/teledyne_whn.dae"/>
         </geometry>
@@ -136,5 +137,5 @@
       <collision>
         <geometry>
-          <cylinder length="0.2445" radius="0.1126"/>
+          <cylinder length="0.189" radius="0.1125"/>
         </geometry>
         <origin xyz="0 0 0" rpy="0 1.5707963267948966 0"/>
@@ -166,9 +167,9 @@
     <gazebo>
       <plugin filename="libuuv_gazebo_ros_dvl_plugin.so" name="libuuv_gazebo_dvl${suffix}_plugin">
-        <robot_namespace>${namespace}</robot_namespace> <!-- (string, required): ros namespace in which the messages are published -->
-        <link_name>${parent_link}</link_name> <!-- (string, required): name of the body which holds the IMU sensor -->
-        <sensor_topic>${topic}${suffix}</sensor_topic> <!-- (string): name of the sensor output topic and prefix of service names -->
-        <update_rate>${update_rate}</update_rate> <!-- Update period [s] -->
-        <noise_sigma>${noise_sigma}</noise_sigma> <!-- std dev of position estimates in x, y, z [m/s] -->
+        <robot_namespace>${namespace}</robot_namespace>
+        <link_name>${parent_link}</link_name>
+        <sensor_topic>${topic}${suffix}</sensor_topic>
+        <update_rate>${update_rate}</update_rate>
+        <noise_sigma>${noise_sigma}</noise_sigma>
         <noise_amplitude>${noise_amplitude}</noise_amplitude>
         <enable_gazebo_messages>false</enable_gazebo_messages>

File: dvl_gazebo/urdf/teledyne_explorer_1000.xacro (robot description, xacro)
@@ -10,5 +10,5 @@
      limitations under the License.
 -->
-<!-- Xacro macros for generating Teledyne Workhorse Navigator (WHN) class URDF models
+<!-- Xacro macros for generating Teledyne Explorer 1000m (phased array) URDF models
      utilizing the uuv_simulator DVL plugin (libuuv_gazebo_ros_dvl_plugin.so)
      Adapted from uuv_simulator version (uuv_sensor_ros_plugins/urdf/dvl_snippets.xacro)
@@ -25,6 +25,7 @@
     </collision>
   </xacro:macro>
-  <!-- Generates a Teledyne WHN URDF model and attaches it to a parent link
-       Sensor parameters align with those in the WHN 600 datasheet -->
+  <!-- Generates a Teledyne Explorer 1000m (phased array) URDF model
+       and attaches it to a parent link in an "inline" configuration.
+       Sensor parameters align with those in the Explorer 1000m (phased array) datasheet -->
   <xacro:macro name="dvl_macro" params="namespace parent_link *origin inertial_reference_frame">
     <xacro:dvl_plugin_macro
@@ -33,13 +34,13 @@
       parent_link="${parent_link}"
       reference_frame="${inertial_reference_frame}"
-      update_rate="7"
+      update_rate="12"
       topic="dvl"
-      noise_sigma="0.005"
-      noise_amplitude="0.005"
+      noise_sigma="0.018"
+      noise_amplitude="0.018"
       scale="1">
       <xacro:insert_block name="origin"/>
     </xacro:dvl_plugin_macro>
   </xacro:macro>
-  <!-- Generates an ENU Teledyne WHN URDF model and attaches it to a parent link -->
+  <!-- Generates an ENU Teledyne Explorer 1000m URDF model and attaches it to a parent link -->
   <xacro:macro name="dvl_sensor_enu" params="namespace parent_link *origin">
     <xacro:dvl_macro
@@ -50,5 +51,5 @@
     </xacro:dvl_macro>
   </xacro:macro>
-  <!-- Generates an NED Teledyne WHN URDF model and attaches it to a parent link -->
+  <!-- Generates an NED Teledyne Explorer 1000m URDF model and attaches it to a parent link -->
   <xacro:macro name="dvl_sensor_ned" params="namespace parent_link *origin">
     <xacro:dvl_macro
@@ -86,17 +87,17 @@
               <samples>3</samples>
               <resolution>1</resolution>
-              <min_angle>-0.03</min_angle>
-              <max_angle>0.03</max_angle>
+              <min_angle>-0.019</min_angle>
+              <max_angle>0.019</max_angle>
             </horizontal>
             <vertical>
               <samples>3</samples>
               <resolution>1</resolution>
-              <min_angle>-0.03</min_angle>
-              <max_angle>0.03</max_angle>
+              <min_angle>-0.019</min_angle>
+              <max_angle>0.019</max_angle>
             </vertical>
           </scan>
           <range>
-            <min>0.7</min>
-            <max>90</max>
+            <min>0.5</min>
+            <max>81</max>
             <resolution>0.01</resolution>
           </range>
@@ -108,5 +109,5 @@
           <topicName>${namespace}/${topic}${suffix}_sonar${index}</topicName>
           <frameName>${namespace}/dvl${suffix}_sonar${index}_link</frameName>
-          <fov>0.06</fov>
+          <fov>0.038</fov>
           <radiation>ultrasound</radiation>
         </plugin>
@@ -125,10 +126,11 @@
     <link name="${namespace}/dvl${suffix}_link">
       <inertial>
-        <mass value="8.8"/>
+        <mass value="0.8"/>
         <origin xyz="0 0 0" rpy="0 0 0"/>
-        <inertia ixx="0.071732122" ixy="0" ixz="0" iyy="0.071732122" iyz="0" izz="0.055786544"/>
+        <inertia ixx="0.007853866666667" ixy="0" ixz="0" iyy="0.007853866666667" iyz="0" izz="0.0015376"/>
       </inertial>
       <visual>
         <geometry>
+        <!-- Replace with Explorer mesh when available -->
         <mesh filename="package://dvl_gazebo/models/teledyne_whn/meshes/teledyne_whn.dae"/>
         </geometry>
@@ -136,7 +138,7 @@
       <collision>
         <geometry>
-          <cylinder length="0.2445" radius="0.1126"/>
+          <cylinder length="0.326" radius="0.062"/>
         </geometry>
-        <origin xyz="0 0 0" rpy="0 1.5707963267948966 0"/>
+        <origin xyz="0 0 0" rpy="0 0 0"/>
       </collision>
     </link>
@@ -166,9 +168,9 @@
     <gazebo>
       <plugin filename="libuuv_gazebo_ros_dvl_plugin.so" name="libuuv_gazebo_dvl${suffix}_plugin">
-        <robot_namespace>${namespace}</robot_namespace> <!-- (string, required): ros namespace in which the messages are published -->
-        <link_name>${parent_link}</link_name> <!-- (string, required): name of the body which holds the IMU sensor -->
-        <sensor_topic>${topic}${suffix}</sensor_topic> <!-- (string): name of the sensor output topic and prefix of service names -->
-        <update_rate>${update_rate}</update_rate> <!-- Update period [s] -->
-        <noise_sigma>${noise_sigma}</noise_sigma> <!-- std dev of position estimates in x, y, z [m/s] -->
+        <robot_namespace>${namespace}</robot_namespace>
+        <link_name>${parent_link}</link_name>
+        <sensor_topic>${topic}${suffix}</sensor_topic>
+        <update_rate>${update_rate}</update_rate>
+        <noise_sigma>${noise_sigma}</noise_sigma>
         <noise_amplitude>${noise_amplitude}</noise_amplitude>
         <enable_gazebo_messages>false</enable_gazebo_messages>

File: dvl_gazebo/urdf/teledyne_explorer_4000.xacro (robot description, xacro)
@@ -10,5 +10,5 @@
      limitations under the License.
 -->
-<!-- Xacro macros for generating Teledyne Workhorse Navigator (WHN) class URDF models
+<!-- Xacro macros for generating Teledyne Explorer 4000m (piston) URDF models
      utilizing the uuv_simulator DVL plugin (libuuv_gazebo_ros_dvl_plugin.so)
      Adapted from uuv_simulator version (uuv_sensor_ros_plugins/urdf/dvl_snippets.xacro)
@@ -25,6 +25,7 @@
     </collision>
   </xacro:macro>
-  <!-- Generates a Teledyne WHN URDF model and attaches it to a parent link
-       Sensor parameters align with those in the WHN 600 datasheet -->
+  <!-- Generates a Teledyne Explorer 4000m (piston) URDF model and
+       attaches it to a parent link in an "inline" configuration.
+       Sensor parameters align with those in the Explorer 4000m (piston) datasheet -->
   <xacro:macro name="dvl_macro" params="namespace parent_link *origin inertial_reference_frame">
     <xacro:dvl_plugin_macro
@@ -33,13 +34,13 @@
       parent_link="${parent_link}"
       reference_frame="${inertial_reference_frame}"
-      update_rate="7"
+      update_rate="12"
       topic="dvl"
-      noise_sigma="0.005"
-      noise_amplitude="0.005"
+      noise_sigma="0.019"
+      noise_amplitude="0.019"
       scale="1">
       <xacro:insert_block name="origin"/>
     </xacro:dvl_plugin_macro>
   </xacro:macro>
-  <!-- Generates an ENU Teledyne WHN URDF model and attaches it to a parent link -->
+  <!-- Generates an ENU Teledyne Explorer 4000m URDF model and attaches it to a parent link -->
   <xacro:macro name="dvl_sensor_enu" params="namespace parent_link *origin">
     <xacro:dvl_macro
@@ -50,5 +51,5 @@
     </xacro:dvl_macro>
   </xacro:macro>
-  <!-- Generates an NED Teledyne WHN URDF model and attaches it to a parent link -->
+  <!-- Generates an NED Teledyne Explorer 4000m URDF model and attaches it to a parent link -->
   <xacro:macro name="dvl_sensor_ned" params="namespace parent_link *origin">
     <xacro:dvl_macro
@@ -86,17 +87,17 @@
               <samples>3</samples>
               <resolution>1</resolution>
-              <min_angle>-0.03</min_angle>
-              <max_angle>0.03</max_angle>
+              <min_angle>-0.033</min_angle>
+              <max_angle>0.033</max_angle>
             </horizontal>
             <vertical>
               <samples>3</samples>
               <resolution>1</resolution>
-              <min_angle>-0.03</min_angle>
-              <max_angle>0.03</max_angle>
+              <min_angle>-0.033</min_angle>
+              <max_angle>0.033</max_angle>
             </vertical>
           </scan>
           <range>
-            <min>0.7</min>
-            <max>90</max>
+            <min>0.5</min>
+            <max>66</max>
             <resolution>0.01</resolution>
           </range>
@@ -108,5 +109,5 @@
           <topicName>${namespace}/${topic}${suffix}_sonar${index}</topicName>
           <frameName>${namespace}/dvl${suffix}_sonar${index}_link</frameName>
-          <fov>0.06</fov>
+          <fov>0.066</fov>
           <radiation>ultrasound</radiation>
         </plugin>
@@ -125,10 +126,11 @@
     <link name="${namespace}/dvl${suffix}_link">
       <inertial>
-        <mass value="8.8"/>
+        <mass value="3.3"/>
         <origin xyz="0 0 0" rpy="0 0 0"/>
-        <inertia ixx="0.071732122" ixy="0" ixz="0" iyy="0.071732122" iyz="0" izz="0.055786544"/>
+        <inertia ixx="0.03676000625" ixy="0" ixz="0" iyy="0.03676000625" iyz="0" izz="0.0084352125"/>
       </inertial>
       <visual>
         <geometry>
+        <!-- Replace with Explorer mesh when available -->
         <mesh filename="package://dvl_gazebo/models/teledyne_whn/meshes/teledyne_whn.dae"/>
         </geometry>
@@ -136,7 +138,7 @@
       <collision>
         <geometry>
-          <cylinder length="0.2445" radius="0.1126"/>
+          <cylinder length="0.344" radius="0.0715"/>
         </geometry>
-        <origin xyz="0 0 0" rpy="0 1.5707963267948966 0"/>
+        <origin xyz="0 0 0" rpy="0 0 0"/>
       </collision>
     </link>
@@ -166,9 +168,9 @@
     <gazebo>
       <plugin filename="libuuv_gazebo_ros_dvl_plugin.so" name="libuuv_gazebo_dvl${suffix}_plugin">
-        <robot_namespace>${namespace}</robot_namespace> <!-- (string, required): ros namespace in which the messages are published -->
-        <link_name>${parent_link}</link_name> <!-- (string, required): name of the body which holds the IMU sensor -->
-        <sensor_topic>${topic}${suffix}</sensor_topic> <!-- (string): name of the sensor output topic and prefix of service names -->
-        <update_rate>${update_rate}</update_rate> <!-- Update period [s] -->
-        <noise_sigma>${noise_sigma}</noise_sigma> <!-- std dev of position estimates in x, y, z [m/s] -->
+        <robot_namespace>${namespace}</robot_namespace>
+        <link_name>${parent_link}</link_name>
+        <sensor_topic>${topic}${suffix}</sensor_topic>
+        <update_rate>${update_rate}</update_rate>
+        <noise_sigma>${noise_sigma}</noise_sigma>
         <noise_amplitude>${noise_amplitude}</noise_amplitude>
         <enable_gazebo_messages>false</enable_gazebo_messages>
