Commit message: Cleaned up UUV Simulator models and launch files some

File: dvl_gazebo/urdf/nortek_dvl500_6000.xacro (robot description, xacro)
@@ -125,5 +125,5 @@
     <link name="${namespace}/dvl${suffix}_link">
       <inertial>
-        <mass value="0.5"/>
+        <mass value="3.1"/>
         <origin xyz="0 0 0" rpy="0 0 0"/>
         <inertia ixx="0.017348633333333" ixy="0" ixz="0" iyy="0.017348633333333" iyz="0" izz="0.01340595"/>

File: dvl_gazebo/urdf/teledyne_explorer_1000.xacro (robot description, xacro)
@@ -128,10 +128,11 @@
         <mass value="0.8"/>
         <origin xyz="0 0 0" rpy="0 0 0"/>
-        <inertia ixx="0.007853866666667" ixy="0" ixz="0" iyy="0.007853866666667" iyz="0" izz="0.0015376"/>
+        <!-- Different mounting orientation than other DVLs -->
+        <inertia ixx="0.0015376" ixy="0" ixz="0" iyy="0.007853866666667" iyz="0" izz="0.007853866666667"/>
       </inertial>
       <visual>
         <geometry>
-        <!-- Replace with Explorer mesh when available -->
-        <mesh filename="package://dvl_gazebo/meshes/teledyne_whn.dae"/>
+          <!-- Replace with Explorer mesh when available -->
+          <mesh filename="package://dvl_gazebo/meshes/teledyne_whn.dae"/>
         </geometry>
       </visual>
