Commit message: Pre-pull update for documentation, clarity & quick fixes
Significant updates/changes include:
Developed Xacro files to generate URDF models from templates
Developed an example Xacro file adding a DVL to a simple "uuv" model
Created a mounted DVL example (executed from a launch file)
Added README.md with instructions for use (will allso add this as a
tutorial in the DAVE wiki.

File: dvl_gazebo/models/teledyne_whn_urdf/model.urdf (robot description, URDF)
Before this commit: robot teledyne_whn, 5 links, 4 joints
Links:
- added link dvl_base_link
- link dvl_link: mass 0.001 -> 8.8; geometry collision cylinder length=0.2445 radius=0.1126; visual mesh filename=package://dvl_gazebo/models/teledyne_whn/meshes/teledyne_wh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
- link dvl_sonar0_link: geometry 
Joints:
- added joint dvl_base_joint: type fixed, parent dvl_base_link, child dvl_link, origin xyz=0 0 0 rpy=0 1.5707963267948966 0

Commit message: Changed mesh location to a "meshes" directory to facilitate re-use
Moving to a single location (for now anyway) will make re-use of meshes
by SDF, URDF, and Xacro models using both the UUV Simulator and WHOI
plugins.

File: dvl_gazebo/models/teledyne_whn_urdf/model.urdf (robot description, URDF)
Before this commit: robot teledyne_whn, 6 links, 5 joints
Links:
- link dvl_link: geometry collision cylinder length=0.2445 radius=0.1126; visual mesh filename=package://dvl_gazebo/meshes/teledyne_whn.dae

File: dvl_gazebo/urdf/nortek_dvl1000_300.xacro (robot description, xacro)
@@ -132,5 +132,5 @@
         <geometry>
         <!-- Replace with Nortek DVL1000 mesh when available -->
-        <mesh filename="package://dvl_gazebo/models/teledyne_whn/meshes/teledyne_whn.dae"/>
+        <mesh filename="package://dvl_gazebo/meshes/teledyne_whn.dae"/>
         </geometry>
       </visual>

File: dvl_gazebo/urdf/nortek_dvl1000_4000.xacro (robot description, xacro)
@@ -132,5 +132,5 @@
         <geometry>
         <!-- Replace with Nortek DVL1000 mesh when available -->
-        <mesh filename="package://dvl_gazebo/models/teledyne_whn/meshes/teledyne_whn.dae"/>
+        <mesh filename="package://dvl_gazebo/meshes/teledyne_whn.dae"/>
         </geometry>
       </visual>

File: dvl_gazebo/urdf/nortek_dvl500_300.xacro (robot description, xacro)
@@ -132,5 +132,5 @@
         <geometry>
         <!-- Replace with Nortek DVL500 mesh when available -->
-        <mesh filename="package://dvl_gazebo/models/teledyne_whn/meshes/teledyne_whn.dae"/>
+        <mesh filename="package://dvl_gazebo/meshes/teledyne_whn.dae"/>
         </geometry>
       </visual>

File: dvl_gazebo/urdf/nortek_dvl500_4000.xacro (robot description, xacro)
@@ -132,5 +132,5 @@
         <geometry>
         <!-- Replace with Nortek DVL500 mesh when available -->
-        <mesh filename="package://dvl_gazebo/models/teledyne_whn/meshes/teledyne_whn.dae"/>
+        <mesh filename="package://dvl_gazebo/meshes/teledyne_whn.dae"/>
         </geometry>
       </visual>

File: dvl_gazebo/urdf/sonardyne_syrinx600.xacro (robot description, xacro)
@@ -132,5 +132,5 @@
         <geometry>
         <!-- Replace with Sonardyne Syrinx 600 mesh when available -->
-        <mesh filename="package://dvl_gazebo/models/teledyne_whn/meshes/teledyne_whn.dae"/>
+        <mesh filename="package://dvl_gazebo/meshes/teledyne_whn.dae"/>
         </geometry>
       </visual>

File: dvl_gazebo/urdf/teledyne_explorer_1000.xacro (robot description, xacro)
@@ -133,5 +133,5 @@
         <geometry>
         <!-- Replace with Explorer mesh when available -->
-        <mesh filename="package://dvl_gazebo/models/teledyne_whn/meshes/teledyne_whn.dae"/>
+        <mesh filename="package://dvl_gazebo/meshes/teledyne_whn.dae"/>
         </geometry>
       </visual>

File: dvl_gazebo/urdf/teledyne_explorer_4000.xacro (robot description, xacro)
@@ -133,5 +133,5 @@
         <geometry>
         <!-- Replace with Explorer mesh when available -->
-        <mesh filename="package://dvl_gazebo/models/teledyne_whn/meshes/teledyne_whn.dae"/>
+        <mesh filename="package://dvl_gazebo/meshes/teledyne_whn.dae"/>
         </geometry>
       </visual>

File: dvl_gazebo/urdf/teledyne_whn.xacro (robot description, xacro)
@@ -131,5 +131,5 @@
       <visual>
         <geometry>
-        <mesh filename="package://dvl_gazebo/models/teledyne_whn/meshes/teledyne_whn.dae"/>
+        <mesh filename="package://dvl_gazebo/meshes/teledyne_whn.dae"/>
         </geometry>
       </visual>

Commit message: Updated meshes in dvl_gazebo models to use the ones Ryan created
Models for which a specific meshes are not yet available are updated to
use the closest match (collision models use correct-sized cylinders)
as follows:

DVL500-300m, DVL500-6000m, and DVL1000-300m use the DVL1000-4000m mesh
Explorer-4000 uses the Explorer 1000 mesh
Syrinx600 uses the Workhorse Navigator mesh

The Explorer 1000 texture (tx-Explorer.jpg) is corrupt and causes an
error when loaded, but the error doesn't affect how anything runs or
displays (just no texture on the Teledyne Explorer visual).

File: dvl_gazebo/models/teledyne_whn_urdf/model.urdf (robot description, URDF)
Before this commit: robot teledyne_whn, 6 links, 5 joints
Links:
- link dvl_link: geometry collision cylinder length=0.2445 radius=0.1126; visual mesh filename=package://dvl_gazebo/meshes/WorkhorseNavigator.dae

File: dvl_gazebo/urdf/nortek_dvl1000_300.xacro (robot description, xacro)
@@ -131,7 +131,7 @@
       <visual>
         <geometry>
-        <!-- Replace with Nortek DVL1000 mesh when available -->
-        <mesh filename="package://dvl_gazebo/meshes/teledyne_whn.dae"/>
+          <mesh filename="package://dvl_gazebo/meshes/DVL1000-4000m.dae"/>
         </geometry>
+        <origin xyz="0 0 0" rpy="0 -1.5707963267948966 0"/>
       </visual>
       <collision>

File: dvl_gazebo/urdf/nortek_dvl1000_4000.xacro (robot description, xacro)
@@ -131,7 +131,7 @@
       <visual>
         <geometry>
-        <!-- Replace with Nortek DVL1000 mesh when available -->
-        <mesh filename="package://dvl_gazebo/meshes/teledyne_whn.dae"/>
+          <mesh filename="package://dvl_gazebo/meshes/DVL1000-4000m.dae"/>
         </geometry>
+        <origin xyz="0 0 0" rpy="0 -1.5707963267948966 0"/>
       </visual>
       <collision>

File: dvl_gazebo/urdf/nortek_dvl500_300.xacro (robot description, xacro)
@@ -131,7 +131,8 @@
       <visual>
         <geometry>
-        <!-- Replace with Nortek DVL500 mesh when available -->
-        <mesh filename="package://dvl_gazebo/meshes/teledyne_whn.dae"/>
+          <!-- Replace with Nortek DVL500 mesh when available -->
+          <mesh filename="package://dvl_gazebo/meshes/DVL1000-4000m.dae"/>
         </geometry>
+        <origin xyz="0 0 0" rpy="0 -1.5707963267948966 0"/>
       </visual>
       <collision>

File: dvl_gazebo/urdf/nortek_dvl500_6000.xacro (robot description, xacro)
@@ -131,7 +131,8 @@
       <visual>
         <geometry>
-        <!-- Replace with Nortek DVL500 mesh when available -->
-        <mesh filename="package://dvl_gazebo/meshes/teledyne_whn.dae"/>
+          <!-- Replace with Nortek DVL500 mesh when available -->
+          <mesh filename="package://dvl_gazebo/meshes/DVL1000-4000m.dae"/>
         </geometry>
+        <origin xyz="0 0 0" rpy="0 -1.5707963267948966 0"/>
       </visual>
       <collision>

File: dvl_gazebo/urdf/sonardyne_syrinx600.xacro (robot description, xacro)
@@ -131,7 +131,8 @@
       <visual>
         <geometry>
-        <!-- Replace with Sonardyne Syrinx 600 mesh when available -->
-        <mesh filename="package://dvl_gazebo/meshes/teledyne_whn.dae"/>
+          <!-- Replace with Sonardyne Syrinx 600 mesh when available -->
+          <mesh filename="package://dvl_gazebo/meshes/WorkhorseNavigator.dae"/>
         </geometry>
+        <origin xyz="0 0 0" rpy="0 1.5707963267948966 0"/>
       </visual>
       <collision>

File: dvl_gazebo/urdf/teledyne_explorer_1000.xacro (robot description, xacro)
@@ -133,7 +133,7 @@
       <visual>
         <geometry>
-          <!-- Replace with Explorer mesh when available -->
-          <mesh filename="package://dvl_gazebo/meshes/teledyne_whn.dae"/>
+          <mesh filename="package://dvl_gazebo/meshes/TeledyneMarineExplorer.dae"/>
         </geometry>
+        <origin xyz="0 0 0" rpy="0 0 1.5707963267948966"/>
       </visual>
       <collision>

File: dvl_gazebo/urdf/teledyne_explorer_4000.xacro (robot description, xacro)
@@ -132,7 +132,7 @@
       <visual>
         <geometry>
-        <!-- Replace with Explorer mesh when available -->
-        <mesh filename="package://dvl_gazebo/meshes/teledyne_whn.dae"/>
+          <mesh filename="package://dvl_gazebo/meshes/TeledyneMarineExplorer.dae"/>
         </geometry>
+        <origin xyz="0 0 0" rpy="0 0 1.5707963267948966"/>
       </visual>
       <collision>

File: dvl_gazebo/urdf/teledyne_whn.xacro (robot description, xacro)
@@ -131,6 +131,7 @@
       <visual>
         <geometry>
-        <mesh filename="package://dvl_gazebo/meshes/teledyne_whn.dae"/>
+          <mesh filename="package://dvl_gazebo/meshes/WorkhorseNavigator.dae"/>
         </geometry>
+        <origin xyz="0 0 0" rpy="0 1.5707963267948966 0"/>
       </visual>
       <collision>

File: dvl_gazebo/urdf_whoi/nortek_dvl1000_300.xacro (robot description, xacro)
@@ -44,8 +44,7 @@
       <visual>
         <geometry>
-          <!-- Replace mesh with correct one once it's available -->
-          <mesh filename="package://dvl_gazebo/meshes/teledyne_whn.dae"/>
+          <mesh filename="package://dvl_gazebo/meshes/DVL1000-4000m.dae"/>
         </geometry>
-        <origin xyz="${xyz}" rpy="0 ${-0.5*pi} 0"/>
+        <origin xyz="${xyz}" rpy="0 3.141592653589793 0"/>
       </visual>
       <collision>
@@ -54,5 +53,5 @@
           <cylinder length="0.158" radius="0.057"/>
         </geometry>
-        <origin xyz="${xyz}" rpy="0 ${-0.5*pi} 0"/>
+        <origin xyz="${xyz}" rpy="0 0 0"/>
       </collision>
     </link>

File: dvl_gazebo/urdf_whoi/nortek_dvl1000_4000.xacro (robot description, xacro)
@@ -44,8 +44,7 @@
       <visual>
         <geometry>
-          <!-- Replace mesh with correct one once it's available -->
-          <mesh filename="package://dvl_gazebo/meshes/teledyne_whn.dae"/>
+          <mesh filename="package://dvl_gazebo/meshes/DVL1000-4000m.dae"/>
         </geometry>
-        <origin xyz="${xyz}" rpy="0 ${-0.5*pi} 0"/>
+        <origin xyz="${xyz}" rpy="0 3.141592653589793 0"/>
       </visual>
       <collision>
@@ -54,5 +53,5 @@
           <cylinder length="0.164" radius="0.057"/>
         </geometry>
-        <origin xyz="${xyz}" rpy="0 ${-0.5*pi} 0"/>
+        <origin xyz="${xyz}" rpy="0 0 0"/>
       </collision>
     </link>

File: dvl_gazebo/urdf_whoi/nortek_dvl500_300.xacro (robot description, xacro)
@@ -45,7 +45,7 @@
         <geometry>
           <!-- Replace mesh with correct one once it's available -->
-          <mesh filename="package://dvl_gazebo/meshes/teledyne_whn.dae"/>
+          <mesh filename="package://dvl_gazebo/meshes/DVL1000-4000m.dae"/>
         </geometry>
-        <origin xyz="${xyz}" rpy="0 ${-0.5*pi} 0"/>
+        <origin xyz="${xyz}" rpy="0 3.141592653589793 0"/>
       </visual>
       <collision>
@@ -54,5 +54,5 @@
           <cylinder length="0.203" radius="0.093"/>
         </geometry>
-        <origin xyz="${xyz}" rpy="0 ${-0.5*pi} 0"/>
+        <origin xyz="${xyz}" rpy="0 0 0"/>
       </collision>
     </link>

File: dvl_gazebo/urdf_whoi/nortek_dvl500_6000.xacro (robot description, xacro)
@@ -45,7 +45,7 @@
         <geometry>
           <!-- Replace mesh with correct one once it's available -->
-          <mesh filename="package://dvl_gazebo/meshes/teledyne_whn.dae"/>
+          <mesh filename="package://dvl_gazebo/meshes/DVL1000-4000m.dae"/>
         </geometry>
-        <origin xyz="${xyz}" rpy="0 ${-0.5*pi} 0"/>
+        <origin xyz="${xyz}" rpy="0 3.141592653589793 0"/>
       </visual>
       <collision>
@@ -54,5 +54,5 @@
           <cylinder length="0.203" radius="0.093"/>
         </geometry>
-        <origin xyz="${xyz}" rpy="0 ${-0.5*pi} 0"/>
+        <origin xyz="${xyz}" rpy="0 0 0"/>
       </collision>
     </link>

File: dvl_gazebo/urdf_whoi/sonardyne_syrinx600.xacro (robot description, xacro)
@@ -45,7 +45,7 @@
         <geometry>
           <!-- Replace mesh with correct one once it's available -->
-          <mesh filename="package://dvl_gazebo/meshes/teledyne_whn.dae"/>
+          <mesh filename="package://dvl_gazebo/meshes/WorkhorseNavigator.dae"/>
         </geometry>
-        <origin xyz="${xyz}" rpy="0 ${-0.5*pi} 0"/>
+        <origin xyz="${xyz}" rpy="0 0 0"/>
       </visual>
       <collision>
@@ -54,5 +54,5 @@
           <cylinder length="0.189" radius="0.1125"/>
         </geometry>
-        <origin xyz="${xyz}" rpy="0 ${-0.5*pi} 0"/>
+        <origin xyz="${xyz}" rpy="0 0 0"/>
       </collision>
     </link>

File: dvl_gazebo/urdf_whoi/teledyne_explorer_1000.xacro (robot description, xacro)
@@ -45,8 +45,7 @@
       <visual>
         <geometry>
-          <!-- Replace mesh with correct one once it's available -->
-          <mesh filename="package://dvl_gazebo/meshes/teledyne_whn.dae"/>
+          <mesh filename="package://dvl_gazebo/meshes/TeledyneMarineExplorer.dae"/>
         </geometry>
-        <origin xyz="${xyz}" rpy="0 0 0"/>
+        <origin xyz="${xyz}" rpy="-1.5707963267948966 0 -1.5707963267948966"/>
       </visual>
       <collision>
@@ -55,5 +54,5 @@
           <cylinder length="0.326" radius="0.062"/>
         </geometry>
-        <origin xyz="${xyz}" rpy="0 0 0"/>
+        <origin xyz="${xyz}" rpy="0 1.5707963267948966 0"/>
       </collision>
     </link>

File: dvl_gazebo/urdf_whoi/teledyne_explorer_4000.xacro (robot description, xacro)
@@ -45,8 +45,7 @@
       <visual>
         <geometry>
-          <!-- Replace mesh with correct one once it's available -->
-          <mesh filename="package://dvl_gazebo/meshes/teledyne_whn.dae"/>
+          <mesh filename="package://dvl_gazebo/meshes/TeledyneMarineExplorer.dae"/>
         </geometry>
-        <origin xyz="${xyz}" rpy="0 0 0"/>
+        <origin xyz="${xyz}" rpy="-1.5707963267948966 0 -1.5707963267948966"/>
       </visual>
       <collision>
@@ -55,5 +54,5 @@
           <cylinder length="0.344" radius="0.0715"/>
         </geometry>
-        <origin xyz="${xyz}" rpy="0 0 0"/>
+        <origin xyz="${xyz}" rpy="0 1.5707963267948966 0"/>
       </collision>
     </link>

File: dvl_gazebo/urdf_whoi/teledyne_whn.xacro (robot description, xacro)
@@ -44,7 +44,7 @@
       <visual>
         <geometry>
-          <mesh filename="package://dvl_gazebo/meshes/teledyne_whn.dae"/>
+          <mesh filename="package://dvl_gazebo/meshes/WorkhorseNavigator.dae"/>
         </geometry>
-        <origin xyz="${xyz}" rpy="0 ${-0.5*pi} 0"/>
+        <origin xyz="${xyz}" rpy="0 0 0"/>
       </visual>
       <collision>
@@ -52,5 +52,5 @@
           <cylinder length="0.2445" radius="0.1126"/>
         </geometry>
-        <origin xyz="${xyz}" rpy="0 ${-0.5*pi} 0"/>
+        <origin xyz="${xyz}" rpy="0 0 0"/>
       </collision>
     </link>
