Commit message: added ft xacro and implemented for all manipulator joints
added the xacro cleaned up the files

File: uuv_dave/urdf/serial_arm.gazebo.xacro (robot description, xacro)
@@ -78,54 +78,16 @@
       <implicitSpringDamper>1</implicitSpringDamper>
     </gazebo>
-    <gazebo reference="${namespace}/azimuth">
-      <sensor name="arm_azimuth" type="force_torque">
-        <force_torque>
-          <frame>child</frame>
-          <measure_direction>child_to_parent</measure_direction>
-          <always_on>true</always_on>
-          <update_rate>30</update_rate>
-        </force_torque>
-      </sensor>
-    </gazebo>
-    <gazebo reference="${namespace}/shoulder">
-      <sensor name="arm_shoulder" type="force_torque">
-        <force_torque>
-          <frame>child</frame>
-          <measure_direction>child_to_parent</measure_direction>
-          <always_on>true</always_on>
-          <update_rate>30</update_rate>
-        </force_torque>
-      </sensor>
-    </gazebo>
-    <gazebo reference="${namespace}/elbow">
-      <sensor name="arm_elbow" type="force_torque">
-        <force_torque>
-          <frame>child</frame>
-          <measure_direction>child_to_parent</measure_direction>
-          <always_on>true</always_on>
-          <update_rate>30</update_rate>
-        </force_torque>
-      </sensor>
-    </gazebo>
-    <gazebo reference="${namespace}/roll">
-      <sensor name="arm_roll" type="force_torque">
-        <force_torque>
-          <frame>child</frame>
-          <measure_direction>child_to_parent</measure_direction>
-          <always_on>true</always_on>
-          <update_rate>30</update_rate>
-        </force_torque>
-      </sensor>
-    </gazebo>
-    <gazebo reference="${namespace}/pitch">
-      <sensor name="arm_pitch" type="force_torque">
-        <force_torque>
-          <frame>child</frame>
-          <measure_direction>child_to_parent</measure_direction>
-          <always_on>true</always_on>
-          <update_rate>30</update_rate>
-        </force_torque>
-      </sensor>
-    </gazebo>
+    <!-- Gripper FT sensors -->
+    <xacro:joint_ft_sensor joint_name="wrist" namespace="${namespace}"/>
+    <xacro:joint_ft_sensor joint_name="finger_left_joint" namespace="${namespace}"/>
+    <xacro:joint_ft_sensor joint_name="finger_tip_left_joint" namespace="${namespace}"/>
+    <xacro:joint_ft_sensor joint_name="finger_right_joint" namespace="${namespace}"/>
+    <xacro:joint_ft_sensor joint_name="finger_tip_right_joint" namespace="${namespace}"/>
+    <!-- Arm FT sensors -->
+    <xacro:joint_ft_sensor joint_name="azimuth" namespace="${namespace}"/>
+    <xacro:joint_ft_sensor joint_name="shoulder" namespace="${namespace}"/>
+    <xacro:joint_ft_sensor joint_name="elbow" namespace="${namespace}"/>
+    <xacro:joint_ft_sensor joint_name="roll" namespace="${namespace}"/>
+    <xacro:joint_ft_sensor joint_name="pitch" namespace="${namespace}"/>
   </xacro:macro>
   <!--

File: uuv_dave/urdf/serial_arm.xacro (robot description, xacro)
@@ -41,4 +41,19 @@
       </transmission>
     </xacro:macro>
+    <!-- Force Feedback Macro -->
+    <xacro:macro name="joint_ft_sensor" params="joint_name namespace">
+      <!-- Enable the Joint Feedback -->
+      <gazebo reference="${namespace}/${joint_name}">
+        <provideFeedback>true</provideFeedback>
+      </gazebo>
+      <!-- The ft_sensor plugin -->
+      <gazebo>
+        <plugin name="ft_sensor" filename="libgazebo_ros_ft_sensor.so">
+          <updateRate>30.0</updateRate>
+          <topicName>ft_sensor_${joint_name}</topicName>
+          <jointName>${namespace}/${joint_name}</jointName>
+        </plugin>
+      </gazebo>
+    </xacro:macro>
     <xacro:macro name="oberon7_serial_arm" params="namespace">
         <!-- Ground base -->
@@ -225,7 +240,4 @@
         <xacro:include filename="$(find oberon7_description)/urdf/parallel_gripper.xacro" />
         <xacro:oberon7_gazebo_macro namespace="${namespace}"/>
-        <!-- Torque Force Sensor  -->
-        <xacro:include filename="$(find uuv_dave)/urdf/parallel_gripper.gazebo.xacro" />
-        <xacro:parallel_gripper_gazebo_macro namespace="${namespace}"/>
     </xacro:macro>
 </robot>

Commit message: put ft macro in its own file

File: uuv_dave/urdf/serial_arm.gazebo.xacro (robot description, xacro)
@@ -13,4 +13,5 @@
 -->
 <robot xmlns:xacro="http://www.ros.org/wiki/xacro">
+  <xacro:include filename="$(find uuv_dave)/urdf/serial_arm_ft_sensor.xacro" />
   <xacro:macro name="oberon7_gazebo_macro" params="namespace">
     <gazebo reference="${namespace}/base">

File: uuv_dave/urdf/serial_arm.xacro (robot description, xacro)
@@ -41,20 +41,4 @@
       </transmission>
     </xacro:macro>
-    <!-- Force Feedback Macro -->
-    <xacro:macro name="joint_ft_sensor" params="joint_name namespace">
-      <!-- Enable the Joint Feedback -->
-      <gazebo reference="${namespace}/${joint_name}">
-        <provideFeedback>true</provideFeedback>
-      </gazebo>
-      <!-- The ft_sensor plugin -->
-      <gazebo>
-        <plugin name="ft_sensor" filename="libgazebo_ros_ft_sensor.so">
-          <updateRate>30.0</updateRate>
-          <topicName>ft_sensor_${joint_name}</topicName>
-          <jointName>${namespace}/${joint_name}</jointName>
-          <gaussianNoise>0.0</gaussianNoise>
-        </plugin>
-      </gazebo>
-    </xacro:macro>
     <xacro:macro name="oberon7_serial_arm" params="namespace">
         <!-- Ground base -->
