Commit message: Finalize arm

File: uuv_dave/urdf/rexrov_oberon7.xacro (robot description, xacro)
@@ -74,5 +74,5 @@
   </xacro:rexrov_base>
   <xacro:oberon7 namespace="oberon7" parent="$(arg namespace)/base_link">
-    <origin xyz="1.3 -0.5 -0.615" rpy="0 0 0"/>
+    <origin xyz="1.15 -0.5 -0.615" rpy="0 0 0"/>
   </xacro:oberon7>
   <gazebo>

File: uuv_dave/urdf/serial_arm_predator.xacro (robot description, xacro)
@@ -51,7 +51,7 @@
             </xacro:link_box_inertial>
             <visual>
-                <origin xyz="0 0 0" rpy="0 0 0"/>
-                <geometry>
-                    <mesh filename="file://$(find oberon7_description)/meshes/serial_arm/collision/Base.stl"/>
+                <origin xyz="0 0 ${-base_height/2.5}" rpy="0 0 0"/>
+                <geometry>
+                    <box size="${predator_base_width} ${predator_base_width} ${predator_shoulder_height/4}" />
                 </geometry>
             </visual>
@@ -68,5 +68,5 @@
                         width="${shoulder_link_width}"
                         length="${shoulder_link_length}"
-                        height="${shoulder_link_height}">
+                        height="${predator_shoulder_height}">
                 <origin xyz="${shoulder_link_com}" rpy="0 0 0"/>
             </xacro:link_box_inertial>
@@ -74,5 +74,5 @@
                 <origin xyz="${shoulder_link_com}" rpy="0 0 0"/>
                 <geometry>
-                    <cylinder radius="${0.5 * shoulder_link_width}" length="${shoulder_link_height}" />
+                    <cylinder radius="${predator_shoulder_radius}" length="${predator_shoulder_height}" />
                 </geometry>
             </visual>
@@ -80,5 +80,5 @@
                 <origin xyz="${shoulder_link_com}" rpy="0 0 0"/>
                 <geometry>
-                    <cylinder radius="${0.5 * shoulder_link_width}" length="${shoulder_link_height}" />
+                    <cylinder radius="${predator_shoulder_radius}" length="${predator_shoulder_height}" />
                 </geometry>
             </collision>
@@ -103,13 +103,13 @@
             </xacro:link_box_inertial>
             <visual>
-                <origin xyz="${upper_arm_com}" rpy="0 ${0.5*pi} 0"/>
-                <geometry>
-                    <cylinder radius="${0.5 * upper_arm_width}" length="${upper_arm_length}"/>
-                </geometry>
-            </visual>
-            <collision>
-                <origin xyz="${upper_arm_com}" rpy="0 ${0.5*pi} 0"/>
-                <geometry>
-                    <cylinder radius="${0.5 * upper_arm_width}" length="${upper_arm_length}"/>
+                <origin xyz="${predator_upper_arm_length/2} 0 0" rpy="0 ${0.5*pi} 0"/>
+                <geometry>
+                    <cylinder radius="${0.5 * upper_arm_width}" length="${predator_upper_arm_length}"/>
+                </geometry>
+            </visual>
+            <collision>
+                <origin xyz="${predator_upper_arm_length/2} 0 0" rpy="0 ${0.5*pi} 0"/>
+                <geometry>
+                    <cylinder radius="${0.5 * upper_arm_width}" length="${predator_upper_arm_length}"/>
                 </geometry>
             </collision>
@@ -118,5 +118,6 @@
             <parent link="${namespace}/shoulder_link"/>
             <child link="${namespace}/upper_arm"/>
-            <origin xyz="0.06955 0.00015 0.01536" rpy="${0.5*pi} 0 0"/>
+            <!-- <origin xyz="0.06955 0.00015 0.01536" rpy="${0.5*pi} 0 0"/> -->
+            <origin xyz="${predator_joint_1_2_x} 0 ${predator_joint_1_2_z}" rpy="${0.5*pi} 0 0"/>
             <axis xyz="0 0 1"/>
             <!-- <dynamics damping="50" friction="200"/> -->
@@ -131,17 +132,17 @@
                         width="${elbow_link_width}"
                         length="${elbow_link_length}"
-                        height="${elbow_link_height}">
+                        height="${predator_elbow_length}">
                 <origin xyz="${elbow_link_com}" rpy="0 0 0"/>
             </xacro:link_box_inertial>
             <visual>
-                <origin xyz="${elbow_link_com}" rpy="0 ${0.5*pi} ${0.5*pi}"/>
-                <geometry>
-                    <cylinder radius="${0.5 * elbow_link_height}" length="${elbow_link_length}"/>
-                </geometry>
-            </visual>
-            <collision>
-                <origin xyz="${elbow_link_com}" rpy="0 ${0.5*pi} ${0.5*pi}"/>
-                <geometry>
-                    <cylinder radius="${0.5 * elbow_link_height}" length="${elbow_link_length}"/>
+                <origin xyz="${elbow_link_x_disp} ${-predator_elbow_length/2} 0" rpy="0 ${0.5*pi} ${0.5*pi}"/>
+                <geometry>
+                    <cylinder radius="${0.5 * elbow_link_height}" length="${predator_elbow_length}"/>
+                </geometry>
+            </visual>
+            <collision>
+                <origin xyz="${elbow_link_x_disp} ${-predator_elbow_length/2} 0" rpy="0 ${0.5*pi} ${0.5*pi}"/>
+                <geometry>
+                    <cylinder radius="${0.5 * elbow_link_height}" length="${predator_elbow_length}"/>
                 </geometry>
             </collision>
@@ -150,5 +151,6 @@
             <parent link="${namespace}/upper_arm"/>
             <child link="${namespace}/elbow_link"/>
-            <origin xyz="0.55616 -0.01229 0" rpy="0 0 0"/>
+            <!-- <origin xyz="0.55616 -0.01229 0" rpy="0 0 0"/> -->
+            <origin xyz="${predator_upper_arm_length} -0.01229 0" rpy="0 0 0"/>
             <!-- <dynamics damping="50" friction="200"/> -->
             <dynamics damping="50" friction="150"/>
@@ -182,5 +184,5 @@
             <parent link="${namespace}/elbow_link"/>
             <child link="${namespace}/forearm"/>
-            <origin xyz="${elbow_link_x_disp} -0.1936267 0" rpy="0 0 0"/>
+            <origin xyz="${elbow_link_x_disp} ${-predator_joint_3_4_y} 0" rpy="0 0 0"/>
             <axis xyz="0 0 1"/>
             <dynamics damping="150" friction="500"/>
@@ -194,18 +196,18 @@
             <xacro:link_box_inertial mass="${total_mass * wrist_volume / total_volume_bbox}"
                         width="${wrist_width}"
-                        length="${wrist_length}"
+                        length="${predator_wrist_height}"
                         height="${wrist_height}">
                 <origin xyz="${wrist_com}" rpy="0 0 0"/>
             </xacro:link_box_inertial>
             <visual>
+                <origin xyz="${predator_wrist_height/2} 0 0" rpy="0 ${0.5*pi} 0"/>
+                <geometry>
+                    <cylinder radius="${0.5 * wrist_height}" length="${predator_wrist_height}"/>
+                </geometry>
+            </visual>
+            <collision>
                 <origin xyz="${wrist_com}" rpy="0 ${0.5*pi} 0"/>
                 <geometry>
-                    <cylinder radius="${0.5 * wrist_height}" length="${wrist_length}"/>
-                </geometry>
-            </visual>
-            <collision>
-                <origin xyz="${wrist_com}" rpy="0 ${0.5*pi} 0"/>
-                <geometry>
-                    <cylinder radius="${0.5 * wrist_height}" length="${wrist_length}"/>
+                    <cylinder radius="${0.5 * wrist_height}" length="${predator_wrist_height}"/>
                 </geometry>
             </collision>
@@ -215,5 +217,7 @@
             <child link="${namespace}/wrist_link"/>
             <!-- <origin xyz="0 0 0.31595760629823427" rpy="${-0.5*PI} ${-0.5*PI} 0"/> -->
-            <origin xyz="0 ${-forearm_height} 0" rpy="0 ${0.5*PI} 0"/>
+            <origin xyz="0 ${-forearm_height} 0" rpy="${1.5*PI} ${PI} ${0.5*PI}"/>
+            <!-- <origin xyz="0 ${-forearm_height} 0" rpy="${1.5*PI} ${PI} ${0.5*PI}"/> -->
+            <!-- <origin xyz="0 ${-forearm_height} 0" rpy="${-0.5*PI} ${-0.5*PI} 0"/> -->
             <axis xyz="0 0 1"/>
             <!-- <dynamics damping="50" friction="200"/> -->
@@ -224,5 +228,5 @@
         <xacro:simple_transmission joint="${namespace}/pitch" />
         <!-- Adding parallel gripper  -->
-        <xacro:include filename="$(find oberon7_description)/urdf/parallel_gripper.xacro" />
+        <xacro:include filename="$(find uuv_dave)/urdf/parallel_gripper_predator.xacro" />
         <xacro:oberon7_gazebo_macro namespace="${namespace}"/>
     </xacro:macro>
