Commit message: Revert back some files that were changed
Files were related to oberon7 and should have not been touched.

File: uuv_dave/urdf/oberon7_default.xacro (robot description, xacro)
@@ -14,5 +14,5 @@
 <robot name="oberon7" xmlns:xacro="http://www.ros.org/wiki/xacro">
   <!-- Import serial arm -->
-  <xacro:include filename="$(find uuv_dave)/urdf/serial_arm_predator.xacro" />
+  <xacro:include filename="$(find uuv_dave)/urdf/serial_arm.xacro" />
   <!-- Import Gazebo specific macros -->
   <xacro:include filename="$(find uuv_dave)/urdf/serial_arm.gazebo.xacro" />

File: uuv_dave/urdf/rexrov_oberon7.xacro (robot description, xacro)
@@ -74,5 +74,5 @@
   </xacro:rexrov_base>
   <xacro:oberon7 namespace="oberon7" parent="$(arg namespace)/base_link">
-    <origin xyz="1.15 -0.5 -0.615" rpy="0 0 0"/>
+    <origin xyz="1.3 -0.5 -0.615" rpy="0 0 0"/>
   </xacro:oberon7>
   <gazebo>
