Commit message: Change visual mesh to be cylinders

File: uuv_dave/urdf/serial_arm_predator.xacro (robot description, xacro)
@@ -53,5 +53,5 @@
                 <origin xyz="0 0 0" rpy="0 0 0"/>
                 <geometry>
-                    <mesh filename="file://$(find oberon7_description)/meshes/serial_arm/visual/Base.dae"/>
+                    <mesh filename="file://$(find oberon7_description)/meshes/serial_arm/collision/Base.stl"/>
                 </geometry>
             </visual>
@@ -72,7 +72,7 @@
             </xacro:link_box_inertial>
             <visual>
-                <origin xyz="0 0 0" rpy="0 0 0"/>
-                <geometry>
-                    <mesh filename="file://$(find oberon7_description)/meshes/serial_arm/visual/ShoulderLink.dae"/>
+                <origin xyz="${shoulder_link_com}" rpy="0 0 0"/>
+                <geometry>
+                    <cylinder radius="${0.5 * shoulder_link_width}" length="${shoulder_link_height}" />
                 </geometry>
             </visual>
@@ -103,7 +103,7 @@
             </xacro:link_box_inertial>
             <visual>
-                <origin xyz="0 0 0" rpy="0 0 0"/>
-                <geometry>
-                    <mesh filename="file://$(find oberon7_description)/meshes/serial_arm/visual/UpperArm.dae"/>
+                <origin xyz="${upper_arm_com}" rpy="0 ${0.5*pi} 0"/>
+                <geometry>
+                    <cylinder radius="${0.5 * upper_arm_width}" length="${upper_arm_length}"/>
                 </geometry>
             </visual>
@@ -135,7 +135,7 @@
             </xacro:link_box_inertial>
             <visual>
-                <origin xyz="0 0 0" rpy="0 0 0"/>
-                <geometry>
-                    <mesh filename="file://$(find oberon7_description)/meshes/serial_arm/visual/ElbowLink.dae"/>
+                <origin xyz="${elbow_link_com}" rpy="0 ${0.5*pi} ${0.5*pi}"/>
+                <geometry>
+                    <cylinder radius="${0.5 * elbow_link_height}" length="${elbow_link_length}"/>
                 </geometry>
             </visual>
@@ -167,7 +167,7 @@
             </xacro:link_box_inertial>
             <visual>
-                <origin xyz="0 0 0" rpy="0 0 0"/>
-                <geometry>
-                    <mesh filename="file://$(find oberon7_description)/meshes/serial_arm/visual/Forearm.dae"/>
+                <origin xyz="${forearm_com}" rpy="0 0 0"/>
+                <geometry>
+                    <cylinder radius="${0.5 * forearm_width}" length="${forearm_height}"/>
                 </geometry>
             </visual>
@@ -199,7 +199,7 @@
             </xacro:link_box_inertial>
             <visual>
-                <origin xyz="0 0 0" rpy="0 0 0"/>
-                <geometry>
-                    <mesh filename="file://$(find oberon7_description)/meshes/serial_arm/visual/Wrist.dae"/>
+                <origin xyz="${wrist_com}" rpy="0 ${0.5*pi} 0"/>
+                <geometry>
+                    <cylinder radius="${0.5 * wrist_height}" length="${wrist_length}"/>
                 </geometry>
             </visual>

Commit message: Change axis of rotation to be the Z axis
Done to abide by DH conventions. The convention was also maintained by in the oberon7

File: uuv_dave/urdf/serial_arm_predator.xacro (robot description, xacro)
@@ -14,5 +14,5 @@
 <robot xmlns:xacro="http://www.ros.org/wiki/xacro">
     <!-- Import arm parameters -->
-    <xacro:include filename="$(find oberon7_description)/urdf/parameters/serial_arm.xacro" />
+    <xacro:include filename="$(find uuv_dave)/urdf/parameters/serial_arm_predator.xacro" />
     <!-- Transmission Macro -->
     <!-- <xacro:macro name="simple_transmission" params="joint">
@@ -167,5 +167,5 @@
             </xacro:link_box_inertial>
             <visual>
-                <origin xyz="${forearm_com}" rpy="0 0 0"/>
+                <origin xyz="${forearm_com}" rpy="${0.5*PI} 0 0"/>
                 <geometry>
                     <cylinder radius="${0.5 * forearm_width}" length="${forearm_height}"/>
@@ -173,5 +173,5 @@
             </visual>
             <collision>
-                <origin xyz="${forearm_com}" rpy="0 0 0"/>
+                <origin xyz="${forearm_com}" rpy="${0.5*PI} 0 0"/>
                 <geometry>
                     <cylinder radius="${0.5 * forearm_width}" length="${forearm_height}"/>
@@ -182,6 +182,6 @@
             <parent link="${namespace}/elbow_link"/>
             <child link="${namespace}/forearm"/>
-            <origin xyz="0.1349014 -0.1936267 0" rpy="${0.5*PI} 0 0"/>
-            <axis xyz="0 1 0"/>
+            <origin xyz="${elbow_link_x_disp} -0.1936267 0" rpy="0 0 0"/>
+            <axis xyz="0 0 1"/>
             <dynamics damping="150" friction="500"/>
             <!-- <dynamics damping="300" friction="1000"/> -->
@@ -214,6 +214,7 @@
             <parent link="${namespace}/forearm"/>
             <child link="${namespace}/wrist_link"/>
-            <origin xyz="0 0 0.31595760629823427" rpy="${-0.5*PI} ${-0.5*PI} 0"/>
-            <axis xyz="0 1 0"/>
+            <!-- <origin xyz="0 0 0.31595760629823427" rpy="${-0.5*PI} ${-0.5*PI} 0"/> -->
+            <origin xyz="0 ${-forearm_height} 0" rpy="0 ${0.5*PI} 0"/>
+            <axis xyz="0 0 1"/>
             <!-- <dynamics damping="50" friction="200"/> -->
             <dynamics damping="10" friction="10"/>

Commit message: Remove all mention of oberon7 for the predator launch
Copied many filed over from uuv_manipulator file

File: uuv_dave/urdf/serial_arm_predator.xacro (robot description, xacro)
@@ -41,5 +41,5 @@
       </transmission>
     </xacro:macro>
-    <xacro:macro name="oberon7_serial_arm" params="namespace">
+    <xacro:macro name="predator_serial_arm" params="namespace">
         <!-- Ground base -->
         <link name="${namespace}/base">
@@ -59,5 +59,6 @@
                 <origin xyz="0 0 0" rpy="0 0 0"/>
                 <geometry>
-                    <mesh filename="file://$(find oberon7_description)/meshes/serial_arm/collision/Base.stl"/>
+                    <box size="${predator_base_width} ${predator_base_width} ${predator_shoulder_height/4}" />
+                    <!-- <mesh filename="file://$(find oberon7_description)/meshes/serial_arm/collision/Base.stl"/> -->
                 </geometry>
             </collision>
@@ -216,8 +217,5 @@
             <parent link="${namespace}/forearm"/>
             <child link="${namespace}/wrist_link"/>
-            <!-- <origin xyz="0 0 0.31595760629823427" rpy="${-0.5*PI} ${-0.5*PI} 0"/> -->
             <origin xyz="0 ${-forearm_height} 0" rpy="${1.5*PI} ${PI} ${0.5*PI}"/>
-            <!-- <origin xyz="0 ${-forearm_height} 0" rpy="${1.5*PI} ${PI} ${0.5*PI}"/> -->
-            <!-- <origin xyz="0 ${-forearm_height} 0" rpy="${-0.5*PI} ${-0.5*PI} 0"/> -->
             <axis xyz="0 0 1"/>
             <!-- <dynamics damping="50" friction="200"/> -->
