Commit message: Fix position of manipulator

File: uuv_dave/urdf/rexrov_predator.xacro (robot description, xacro)
@@ -74,5 +74,5 @@
   </xacro:rexrov_base>
   <xacro:predator namespace="predator" parent="$(arg namespace)/base_link">
-    <origin xyz="1.3 -0.5 -0.615" rpy="0 0 0"/>
+    <origin xyz="1.15 -0.5 -0.615" rpy="0 0 0"/>
   </xacro:predator>
   <gazebo>

Commit message: Place the predator base at right height

File: uuv_dave/urdf/rexrov_predator.xacro (robot description, xacro)
@@ -74,5 +74,5 @@
   </xacro:rexrov_base>
   <xacro:predator namespace="predator" parent="$(arg namespace)/base_link">
-    <origin xyz="1.15 -0.5 -0.615" rpy="0 0 0"/>
+    <origin xyz="1.15 -0.5 -0.7" rpy="0 0 0"/>
   </xacro:predator>
   <gazebo>
