Commit message: Added rviz and improved settings for SLOCUM glider

File: uuv_dave/urdf/glider_slocum.xacro (robot description, xacro)
@@ -16,8 +16,7 @@
   <xacro:include filename="$(find uuv_descriptions)/urdf/common.urdf.xacro" />
   <xacro:include filename="$(find uuv_dave)/urdf/sensor_snippets.xacro"/>
-  <xacro:include filename="$(find uuv_dave)/urdf/glider_slocum_snippets.xacro"/>
   <xacro:include filename="$(find uuv_gazebo_ros_plugins)/urdf/snippets.xacro"/>
   <!-- Properties -->
-  <xacro:property name="mass" value="90.0" />
+  <xacro:property name="mass" value="50.0" />
   <xacro:property name="length" value="1.5" />
   <xacro:property name="diameter" value="0.22" />
@@ -32,5 +31,5 @@
   <xacro:property name="collision_mesh_file" value="file://$(find uuv_dave)/models/glider_slocum/mesh/COLLISION-Slocum-Glider.dae" />
   <xacro:property name="prop_mesh_file" value="file://$(find uuv_dave)/models/glider_slocum/mesh/Slocum-Glider-Propeller.dae" />
-  <xacro:property name="rudder_mesh_file" value="file://$(find uuv_dave)/models/glider_slocum/mesh/Slocum-Glider-TopRudder.dae" />
+  <!-- <xacro:property name="rudder_mesh_file" value="file://$(find uuv_dave)/models/glider_slocum/mesh/Slocum-Glider-TopRudder.dae" /> -->
   <xacro:macro name="glider_slocum" params="namespace debug inertial_reference_frame">
     <link name="${namespace}/base_link">
@@ -53,44 +52,5 @@
       </inertial>
     </link>
-    <link name="${namespace}/propeller_link">
-      <visual>
-        <origin xyz="0 0 0" rpy="0 0 0" />
-        <geometry>
-          <mesh filename="${prop_mesh_file}" scale="1 1 1" />
-        </geometry>
-      </visual>
-    </link>
-    <joint name="${namespace}/propeller_joint" type="continuous">
-      <origin xyz="0 0 0" rpy="0 0 0" />
-      <parent link="${namespace}/base_link"/>
-      <child link="${namespace}/propeller_link"/>
-      <axis xyz="0 1 0" />
-    </joint>
-    <link name="${namespace}/rudder_link">
-      <visual>
-        <origin xyz="0 0 0" rpy="0 0 0" />
-        <geometry>
-          <mesh filename="${rudder_mesh_file}" scale="1 1 1" />
-        </geometry>
-      </visual>
-    </link>
-    <joint name="${namespace}/rudder_joint" type="fixed">
-      <origin xyz="0 0 0" rpy="0 0 0" />
-      <parent link="${namespace}/base_link"/>
-      <child link="${namespace}/rudder_link"/>
-    </joint>
-    <link name='${namespace}/battery_link2'>
-      <origin xyz="0 0 0" rpy="0 0 0" />
-      <battery name='${namespace}/battery'>
-        <voltage>4.2</voltage>
-      </battery>
-    </link>
-    <joint name='${namespace}/battery_joint2' type='fixed'>
-      <origin xyz="0 0 0" rpy="0 0 0" />
-      <parent link="${namespace}/base_link"/>
-      <child link="${namespace}/battery_link2"/>
-    </joint>
     <!-- Set up hydrodynamic plugin -->
-    <!-- TODO: vehicle properties and add buoyancy engine and sliding mass plugins -->
     <gazebo>
       <plugin name="${namespace}_uuv_plugin" filename="libuuv_underwater_object_ros_plugin.so">
@@ -101,5 +61,5 @@
           <volume>${volume}</volume>
           <center_of_buoyancy>${cob}</center_of_buoyancy>
-          <neutrally_buoyant>0</neutrally_buoyant>
+          <neutrally_buoyant>1</neutrally_buoyant>
           <hydrodynamic_model>
             <type>fossen</type>
@@ -123,48 +83,35 @@
         </link>
       </plugin>
-      <!-- <plugin name='glider_slocum_thruster_model' filename='libuuv_thruster_ros_plugin.so'>
-        <linkName>${namespace}/propeller_link</linkName>
-        <jointName>${namespace}/propeller_joint</jointName>
-        <thrusterID>0</thrusterID>
-        <dynamics>
-          <type>FirstOrder</type>
-          <timeConstant>0.1</timeConstant>
-        </dynamics>
-        <conversion>
-          <type>Basic</type>
-          <rotorConstant>4.9e-05</rotorConstant>
-        </conversion>
-        <robotNamespace>/</robotNamespace>
-      </plugin> -->
-  <!--    <plugin name='fin0_model' filename='libuuv_fin_ros_plugin.so'>
-        <dynamics>
-          <type>FirstOrder</type>
-          <timeConstant>0.1</timeConstant>
-        </dynamics>
-        <liftdrag>
-          <type>TwoLines</type>
-          <area>0.04155</area>
-          <fluid_density>1027.0</fluid_density>
-          <a0>0.0</a0>
-          <alpha_stall>0.174533</alpha_stall>
-          <cla>13.98</cla>
-          <cla_stall>0.0</cla_stall>
-          <cda>0.0</cda>
-          <cda_stall/>
-        </liftdrag>
-        <current_velocity_topic>hydrodynamics/current_velocity</current_velocity_topic>
-        <fin_id>0</fin_id>
-        <link_name>fin0</link_name>
-        <joint_name>fin0_joint</joint_name>
-        <robotNamespace>/</robotNamespace>
-      </plugin> -->
     </gazebo>
-    <!-- TODO: Correct propeller origins and parameters -->
-    <xacro:thruster_module_first_order_basic_fcn_macro namespace="${namespace}" thruster_id="0" mesh_filename="${prop_mesh_file}" dyn_time_constant="0.1" rotor_constant="0.000049">
-      <origin xyz="0 0 0" rpy="0 0 0" />
-    </xacro:thruster_module_first_order_basic_fcn_macro>
-    <!-- TODO: Parametrize the battery unit -->
-    <xacro:basic_linear_battery_macro namespace="${namespace}" parent_link="${namespace}/base_link" prefix="" open_circuit_voltage_constant_coef="3.7" open_circuit_voltage_linear_coef="-3.1424" initial_charge="1.1665" capacity="0.5" resistance="0.002" smooth_current_tau="1.9499" voltage="4.2" update_rate="2.0" />
-    <xacro:include filename="$(find uuv_dave)/urdf/glider_slocum_sensors.xacro" />
+    <!-- Include the battery modules -->
+    <xacro:basic_linear_battery_macro
+      namespace="${namespace}"
+      parent_link="${namespace}/base_link"
+      prefix=""
+      open_circuit_voltage_constant_coef="3.7"
+      open_circuit_voltage_linear_coef="-3.1424"
+      initial_charge="1.1665"
+      capacity="0.5"
+      resistance="0.002"
+      smooth_current_tau="1.9499"
+      voltage="4.2"
+      update_rate="2.0"/>
+    <!-- Include the thruster modules -->
+    <xacro:macro name="thruster_macro"
+      params="namespace thruster_id *origin">
+      <xacro:thruster_module_first_order_basic_fcn_macro
+        namespace="${namespace}"
+        thruster_id="${thruster_id}"
+        mesh_filename="${prop_mesh_file}"
+        dyn_time_constant="0.05"
+        rotor_constant="0.00031">
+        <xacro:insert_block name="origin"/>
+      </xacro:thruster_module_first_order_basic_fcn_macro>
+    </xacro:macro>
+    <xacro:thruster_macro namespace="${namespace}" thruster_id="0">
+        <origin xyz="0 0 0" rpy="0 0 0"/>
+    </xacro:thruster_macro>
+    <!-- Include sensor modules -->
+    <xacro:include filename="$(find uuv_dave)/urdf/glider_slocum_sensors.xacro"/>
   </xacro:macro>
 </robot>

File: uuv_dave/urdf/glider_slocum_sensors.xacro (robot description, xacro)
@@ -19,5 +19,5 @@
       inertial_reference_frame="${inertial_reference_frame}" />
     <!-- DVL sensor -->
-    <xacro:dvl_plugin_macro
+    <!-- <xacro:dvl_plugin_macro
       namespace="${namespace}"
       suffix=""
@@ -29,35 +29,14 @@
       update_rate="7"
       reference_frame="world">
-      <origin xyz="0.0 0.4785 -0.0825" rpy="${0.5*pi} 0 0" />
-    </xacro:dvl_plugin_macro>
-    <xacro:switchable_battery_consumer_macro
+      <origin xyz="0.0 4.785 -0.825" rpy="${0.5*pi} 0 0" />
+    </xacro:dvl_plugin_macro> -->
+    <!-- <xacro:switchable_battery_consumer_macro
       link_name="${namespace}/dvl_link"
       battery_link="${namespace}/battery_link"
       battery_name="${namespace}/battery"
       power_load="25"
-      topic="${namespace}/dvl/state"/>
-    <!-- Side scan sonar left -->
-    <!--<xacro:sidescan_sonar namespace="${namespace}" parent_link="${namespace}/base_link" suffix="left">
-      <origin xyz="0.41225 0.1498 -0.04615" rpy="${0.5*pi} ${-5*d2r+pi/3.0} ${0.5*pi}" />
-    </xacro:sidescan_sonar>-->
-    <xacro:switchable_battery_consumer_macro
-      link_name="${namespace}/sonarleft_link"
-      battery_link="${namespace}/battery_link"
-      battery_name="${namespace}/battery"
-      power_load="25"
-      topic="${namespace}/sonarleft/state"/>
-    <!-- Side scan sonar right -->
-    <!--<xacro:sidescan_sonar
-      namespace="${namespace}" parent_link="${namespace}/base_link" suffix="right">
-      <origin xyz="0.41225 -0.1498 -0.04615" rpy="${0.5*pi} ${-5*d2r+pi/3.0} ${-0.5*pi}" />
-    </xacro:sidescan_sonar>-->
-    <xacro:switchable_battery_consumer_macro
-      link_name="${namespace}/sonarright_link"
-      battery_link="${namespace}/battery_link"
-      battery_name="${namespace}/battery"
-      power_load="25"
-      topic="${namespace}/sonarright/state"/>
-    <!-- RPT
-    <xacro:default_rpt namespace="${namespace}" parent_link="${namespace}/base_link">
+      topic="${namespace}/dvl/state"/> -->
+    <!-- RPT -->
+    <!-- <xacro:default_rpt namespace="${namespace}" parent_link="${namespace}/base_link">
       <origin xyz="0 0 0" rpy="0 0 0"/>
     </xacro:default_rpt>  -->
@@ -83,5 +62,5 @@
       topic="${namespace}/imu/state"/>
     <!-- Mount a camera -->
-    <xacro:regular_camera_plugin_macro
+    <!-- <xacro:regular_camera_plugin_macro
         namespace="${namespace}"
         suffix=""
@@ -96,12 +75,12 @@
         scale="0.5">
         <inertia ixx="0.00001" ixy="0.0" ixz="0.0" iyy="0.00001" iyz="0.0" izz="0.00001" />
-        <origin xyz="0 -0.375 -0.16" rpy="0.3 0 0"/>
-    </xacro:regular_camera_plugin_macro>
-    <xacro:switchable_battery_consumer_macro
+        <origin xyz="0 -3.75 -1.6" rpy="0.3 0 0"/>
+    </xacro:regular_camera_plugin_macro> -->
+    <!-- <xacro:switchable_battery_consumer_macro
       link_name="${namespace}/camera_link"
       battery_link="${namespace}/battery_link"
       battery_name="${namespace}/battery"
       power_load="25"
-      topic=""/>
+      topic=""/> -->
     <!-- Mount a GPS. -->
     <xacro:default_gps namespace="${namespace}" parent_link="${namespace}/base_link" />
