Commit message: Correcting orientation of visual and collision mesh in URDF, changing initial position

File: uuv_dave/urdf/glider_hybrid_whoi.xacro (robot description, xacro)
@@ -36,5 +36,5 @@
     <link name="${namespace}/base_link">
       <visual>
-        <origin xyz="0 0 0" rpy="0 0 0" />
+        <origin xyz="0 0 0" rpy="0 0 -1.5708" />
         <geometry>
           <mesh filename="${visual_mesh_file}" scale="1 1 1" />
@@ -42,5 +42,5 @@
       </visual>
       <collision>
-        <origin xyz="0 0 0" rpy="0 0 0" />
+        <origin xyz="0 0 0" rpy="0 0 -1.5708" />
         <geometry>
           <mesh filename="${collision_mesh_file}" scale="1 1 1" />
@@ -55,5 +55,5 @@
     <link name="${namespace}/left_propeller_link">
       <visual>
-        <origin xyz="0 0 0" rpy="0 0 0" />
+        <origin xyz="0 0 0" rpy="0 0 0 " />
         <geometry>
           <mesh filename="${left_prop_mesh_file}" scale="1 1 1" />
@@ -163,8 +163,8 @@
     <!-- TODO: Correct propeller origins and parameters -->
     <xacro:thruster_module_first_order_basic_fcn_macro namespace="${namespace}" thruster_id="0" mesh_filename="${left_prop_mesh_file}" dyn_time_constant="0.1" rotor_constant="0.000049">
-      <origin xyz="0 0 0" rpy="0 0 0" />
+      <origin xyz="0 0 0" rpy="0 0 -1.5708" />
     </xacro:thruster_module_first_order_basic_fcn_macro>
     <xacro:thruster_module_first_order_basic_fcn_macro namespace="${namespace}" thruster_id="1" mesh_filename="${right_prop_mesh_file}" dyn_time_constant="0.1" rotor_constant="0.000049">
-      <origin xyz="0 0 0" rpy="0 0 0" />
+      <origin xyz="0 0 0" rpy="0 0 -1.5708" />
     </xacro:thruster_module_first_order_basic_fcn_macro>
     <!-- TODO: Parametrize the battery unit -->

File: uuv_dave/urdf/glider_slocum.xacro (robot description, xacro)
@@ -30,10 +30,10 @@
   <xacro:property name="visual_mesh_file" value="file://$(find uuv_dave)/models/glider_slocum/mesh/Slocum-Glider.dae" />
   <xacro:property name="collision_mesh_file" value="file://$(find uuv_dave)/models/glider_slocum/mesh/COLLISION-Slocum-Glider.dae" />
-  <xacro:property name="prop_mesh_file" value="file://$(find uuv_dave)/models/glider_slocum/mesh/Slocum-Glider-Propeller.dae" />
+  <!--<xacro:property name="prop_mesh_file" value="file://$(find uuv_dave)/models/glider_slocum/mesh/Slocum-Glider-Propeller.dae" />-->
   <!-- <xacro:property name="rudder_mesh_file" value="file://$(find uuv_dave)/models/glider_slocum/mesh/Slocum-Glider-TopRudder.dae" /> -->
   <xacro:macro name="glider_slocum" params="namespace debug inertial_reference_frame">
     <link name="${namespace}/base_link">
       <visual>
-        <origin xyz="0 0 0" rpy="0 0 0" />
+        <origin xyz="0 0 0" rpy="0 0 -1.5708" />
         <geometry>
           <mesh filename="${visual_mesh_file}" scale="1 1 1" />
@@ -41,5 +41,5 @@
       </visual>
       <collision>
-        <origin xyz="0 0 0" rpy="0 0 0" />
+        <origin xyz="0 0 0" rpy="0 0 -1.5708" />
         <geometry>
           <mesh filename="${collision_mesh_file}" scale="1 1 1" />
@@ -97,19 +97,4 @@
       voltage="4.2"
       update_rate="2.0"/>
-    <!-- Include the thruster modules -->
-    <xacro:macro name="thruster_macro"
-      params="namespace thruster_id *origin">
-      <xacro:thruster_module_first_order_basic_fcn_macro
-        namespace="${namespace}"
-        thruster_id="${thruster_id}"
-        mesh_filename="${prop_mesh_file}"
-        dyn_time_constant="0.05"
-        rotor_constant="0.00031">
-        <xacro:insert_block name="origin"/>
-      </xacro:thruster_module_first_order_basic_fcn_macro>
-    </xacro:macro>
-    <xacro:thruster_macro namespace="${namespace}" thruster_id="0">
-        <origin xyz="0 0 0" rpy="0 0 0"/>
-    </xacro:thruster_macro>
     <!-- Include sensor modules -->
     <xacro:include filename="$(find uuv_dave)/urdf/glider_slocum_sensors.xacro"/>

File: uuv_dave/urdf/glider_wave.xacro (robot description, xacro)
@@ -16,5 +16,5 @@
   <xacro:include filename="$(find uuv_descriptions)/urdf/common.urdf.xacro" />
   <xacro:include filename="$(find uuv_dave)/urdf/sensor_snippets.xacro" />
-  <xacro:include filename="$(find uuv_dave)/urdf/glider_wave_liquidrobotics_snippets.xacro" />
+  <xacro:include filename="$(find uuv_dave)/urdf/glider_wave_snippets.xacro" />
   <xacro:include filename="$(find uuv_gazebo_ros_plugins)/urdf/snippets.xacro" />
   <!-- Properties -->
@@ -30,16 +30,16 @@
   <xacro:property name="area" value="0.04155" />
   <xacro:property name="length" value="1.5" />
-  <xacro:property name="namespace" value="glider_wave_liquidrobotics" />
-  <xacro:property name="visual_mesh_file" value="file://$(find uuv_dave)/models/glider_wave_liquidrobotics/mesh/Wave Glider-Float.dae" />
-  <xacro:property name="collision_mesh_file" value="file://$(find uuv_dave)/models/glider_wave_liquidrobotics/mesh/COLLISION-Wave Glider-float.dae" />
-  <xacro:property name="sub_visual_mesh_file" value="file://$(find uuv_dave)/models/glider_wave_liquidrobotics/mesh/Wave Glider-Sub.dae" />
-  <xacro:property name="sub_collision_mesh_file" value="file://$(find uuv_dave)/models/glider_wave_liquidrobotics/mesh/COLLISION-Wave Glider-sub.dae" />
-  <xacro:property name="umbilicaljoint_visual_mesh_file" value="file://$(find uuv_dave)/models/glider_wave_liquidrobotics/mesh/Wave Glider-Joint.dae" />
-  <xacro:property name="umbilical_visual_mesh_file" value="file://$(find uuv_dave)/models/glider_wave_liquidrobotics/mesh/Wave Glider-Umbilical.dae" />
-  <xacro:property name="umbilical_collision_mesh_file" value="file://$(find uuv_dave)/models/glider_wave_liquidrobotics/mesh/COLLISION-Wave Glider-umbilical.dae" />
-  <xacro:macro name="glider_wave_liquidrobotics" params="namespace debug inertial_reference_frame">
+  <xacro:property name="namespace" value="glider_wave" />
+  <xacro:property name="visual_mesh_file" value="file://$(find uuv_dave)/models/glider_wave/mesh/Wave Glider-Float.dae" />
+  <xacro:property name="collision_mesh_file" value="file://$(find uuv_dave)/models/glider_wave/mesh/COLLISION-Wave Glider-float.dae" />
+  <xacro:property name="sub_visual_mesh_file" value="file://$(find uuv_dave)/models/glider_wave/mesh/Wave Glider-Sub.dae" />
+  <xacro:property name="sub_collision_mesh_file" value="file://$(find uuv_dave)/models/glider_wave/mesh/COLLISION-Wave Glider-sub.dae" />
+  <xacro:property name="umbilicaljoint_visual_mesh_file" value="file://$(find uuv_dave)/models/glider_wave/mesh/Wave Glider-Joint.dae" />
+  <xacro:property name="umbilical_visual_mesh_file" value="file://$(find uuv_dave)/models/glider_wave/mesh/Wave Glider-Umbilical.dae" />
+  <xacro:property name="umbilical_collision_mesh_file" value="file://$(find uuv_dave)/models/glider_wave/mesh/COLLISION-Wave Glider-umbilical.dae" />
+  <xacro:macro name="glider_wave" params="namespace debug inertial_reference_frame">
     <link name="${namespace}/base_link">
       <visual>
-        <origin xyz="0 0 0" rpy="0 0 0" />
+        <origin xyz="0 0 0" rpy="0 0 1.570" />
         <geometry>
           <mesh filename="${visual_mesh_file}" scale="1 1 1" />
@@ -47,5 +47,5 @@
       </visual>
       <collision>
-        <origin xyz="0 0 0" rpy="0 0 0" />
+        <origin xyz="0 0 0" rpy="0 0 1.570" />
         <geometry>
           <mesh filename="${collision_mesh_file}" scale="1 1 1" />
@@ -75,5 +75,5 @@
     <link name="${namespace}/umbilical_link">
       <visual>
-        <origin xyz="0 0 0" rpy="0 0 0" />
+        <origin xyz="0 0 0" rpy="0 0 1.570" />
         <geometry>
           <mesh filename="${umbilical_visual_mesh_file}" scale="1 1 1" />
@@ -81,5 +81,5 @@
       </visual>
       <collision>
-        <origin xyz="0 0 0" rpy="0 0 0" />
+        <origin xyz="0 0 0" rpy="0 0 1.570" />
         <geometry>
           <mesh filename="${umbilical_collision_mesh_file}" scale="1 1 1" />
@@ -101,5 +101,5 @@
     <link name="${namespace}/sub_link">
       <visual>
-        <origin xyz="0 0 0" rpy="0 0 0" />
+        <origin xyz="0 0 0" rpy="0 0 -1.570" />
         <geometry>
           <mesh filename="${sub_visual_mesh_file}" scale="1 1 1" />
@@ -107,5 +107,5 @@
       </visual>
       <collision>
-        <origin xyz="0 0 0" rpy="0 0 0" />
+        <origin xyz="0 0 0" rpy="0 0 -1.570" />
         <geometry>
           <mesh filename="${sub_collision_mesh_file}" scale="1 1 1" />
@@ -157,5 +157,5 @@
         </link>
       </plugin> -->
-      <!-- <plugin name='glider_wave_liquidrobotics_thruster_model' filename='libuuv_thruster_ros_plugin.so'>
+      <!-- <plugin name='glider_wave_thruster_model' filename='libuuv_thruster_ros_plugin.so'>
         <linkName>${namespace}/propeller_link</linkName>
         <jointName>${namespace}/propeller_joint</jointName>
@@ -194,5 +194,5 @@
       </plugin> -->
     </gazebo>
-    <xacro:include filename="$(find uuv_dave)/urdf/glider_wave_liquidrobotics_sensors.xacro" />
+    <xacro:include filename="$(find uuv_dave)/urdf/glider_wave_sensors.xacro" />
   </xacro:macro>
 </robot>

File: uuv_dave/urdf/glider_wave_default.urdf.xacro (robot description, xacro)
@@ -12,12 +12,12 @@
      limitations under the License.
 -->
-<robot name="glider_wave_liquidrobotics" xmlns:xacro="http://www.ros.org/wiki/xacro" >
+<robot name="glider_wave" xmlns:xacro="http://www.ros.org/wiki/xacro" >
   <xacro:arg name="debug" default="0"/>
-  <xacro:arg name="namespace" default="glider_wave_liquidrobotics"/>
+  <xacro:arg name="namespace" default="glider_wave"/>
   <xacro:arg name="inertial_reference_frame" default="world"/>
   <!-- Include the UUV macro file -->
-  <xacro:include filename="$(find uuv_dave)/urdf/glider_wave_liquidrobotics.xacro"/>
-  <!-- Create the glider_wave_liquidrobotics -->
-  <xacro:glider_wave_liquidrobotics
+  <xacro:include filename="$(find uuv_dave)/urdf/glider_wave.xacro"/>
+  <!-- Create the glider_wave_ -->
+  <xacro:glider_wave
     namespace="$(arg namespace)"
     debug="$(arg debug)"
