Commit message: flip wave glider sub

File: uuv_dave/urdf/glider_wave.xacro (robot description, xacro)
@@ -101,5 +101,5 @@
     <link name="${namespace}/sub_link">
       <visual>
-        <origin xyz="0 0 0" rpy="0 0 -1.570" />
+        <origin xyz="0 0 0" rpy="0 0 1.570" />
         <geometry>
           <mesh filename="${sub_visual_mesh_file}" scale="1 1 1" />
@@ -107,5 +107,5 @@
       </visual>
       <collision>
-        <origin xyz="0 0 0" rpy="0 0 -1.570" />
+        <origin xyz="0 0 0" rpy="0 0 1.570" />
         <geometry>
           <mesh filename="${sub_collision_mesh_file}" scale="1 1 1" />
