Commit message: Add properties to parameter file for arm

File: uuv_dave/urdf/parameters/serial_arm_predator.xacro (robot description, xacro)
@@ -45,4 +45,15 @@
     | 0.000008 0.000022 0.000016 |
   -->
+  <xacro:property name="predator_base_width" value="0.197"/>
+  <xacro:property name="unit" value="${predator_base_width/2}"/>
+  <xacro:property name="predator_shoulder_radius" value="${predator_base_width/2}"/>
+  <xacro:property name="predator_shoulder_height" value="0.203"/>
+  <xacro:property name="predator_joint_1_2_x" value="${predator_base_width/2*1.5}"/>
+  <xacro:property name="predator_joint_1_2_z" value="${predator_shoulder_height/2}"/>
+  <xacro:property name="predator_joint_3_4_y" value="0.56"/>
+  <!-- <xacro:property name="predator_joint_3_4_z" value="${predator_shoulder_height/2}"/> -->
+  <xacro:property name="predator_upper_arm_length" value="${unit*8.5}"/>
+  <!-- <xacro:property name="predator_elbow_length" value="0.56"/> -->
+  <xacro:property name="predator_elbow_length" value="0.56"/>
   <xacro:property name="base_width" value="0.198133"/>
   <xacro:property name="base_length" value="0.282087"/>
@@ -74,5 +85,5 @@
   <xacro:property name="shoulder_link_volume" value="${shoulder_link_width * shoulder_link_length * shoulder_link_height}"/>
   <!-- <xacro:property name="shoulder_link_com" value="0.039670 0.005441 0.017383"/> -->
-  <xacro:property name="shoulder_link_com" value="0.0 0.005441 0.017383"/>
+  <xacro:property name="shoulder_link_com" value="0 0 0.017383"/>
   <!--
     UPPER ARM
@@ -135,6 +146,6 @@
   <xacro:property name="forearm_width" value="0.151455"/>
   <xacro:property name="forearm_length" value="0.151505"/>
-  <xacro:property name="forearm_height" value="0.15"/>
-  <!-- <xacro:property name="forearm_height" value="0.334827"/> -->
+  <xacro:property name="predator_forearm_height" value="0.15"/>
+  <xacro:property name="forearm_height" value="0.334827"/>
   <xacro:property name="forearm_volume" value="${forearm_width * forearm_length * forearm_height}" />
   <!-- <xacro:property name="forearm_com" value="0 0 ${0.5*0.31595760629823427}"/> -->
@@ -162,4 +173,5 @@
   <xacro:property name="wrist_length" value="0.219204"/>
   <xacro:property name="wrist_height" value="0.130374"/>
+  <xacro:property name="predator_wrist_height" value="0.05"/>
   <xacro:property name="wrist_volume" value="${wrist_width * wrist_length * wrist_height}" />
   <xacro:property name="wrist_com" value="0.104016 0.003308 -0.000027"/>
