Commit message: Migration to xacro, urdf format with less sensors attached

File: uuv_dave/models/glider_slocum/urdf/glider_slocum.xacro (robot description, xacro)
@@ -57,7 +57,7 @@
         <mass value="${mass}" />
         <origin xyz="0 0 0" rpy="0 0 0"/>
-        <inertia ixx="0.6" ixy="0" ixz="0"
-                 iyy="30.0" iyz="0"
-                 izz="35.0" />
+        <inertia ixx="30.0" ixy="0" ixz="0"
+                 iyy="0.6" iyz="0"
+                 izz="5.0" />
       </inertial>
     </link>
@@ -96,5 +96,5 @@
     </gazebo>
     <!-- TODO: Correct fin origins -->
-    <xacro:fin_macro namespace="${namespace}" fin_id="0">
+    <!-- <xacro:fin_macro namespace="${namespace}" fin_id="0">
       <origin xyz="-0.70777 -0.07876 0.078586" rpy="0.7904 -0.0998 -0.1003" />
     </xacro:fin_macro>
@@ -104,5 +104,5 @@
     <xacro:fin_macro namespace="${namespace}" fin_id="2">
       <origin xyz="-0.70777 0.07876 -0.078586" rpy="-2.3512 0.0998 0.1003" />
-    </xacro:fin_macro>
+    </xacro:fin_macro> -->
     <!-- TODO: Correct propeller origins and parameters -->
     <xacro:thruster_module_first_order_basic_fcn_macro
@@ -112,5 +112,5 @@
       dyn_time_constant="0.1"
       rotor_constant="0.000049">
-      <origin xyz="-0.9676 0 0" rpy="0 0 ${pi}" />
+      <origin xyz="0 -0.4 0" rpy="0 0 ${pi}" />
     </xacro:thruster_module_first_order_basic_fcn_macro>
     <!-- TODO: Parametrize the battery unit -->

File: uuv_dave/models/glider_slocum/urdf/glider_slocum_sensors.xacro (robot description, xacro)
@@ -29,5 +29,5 @@
       update_rate="7"
       reference_frame="world">
-      <origin xyz="0.4785 0.0 -0.0825" rpy="0 ${0.5*pi} 0" />
+      <origin xyz="0.0 0.4785 -0.0825" rpy="${0.5*pi} 0 0" />
     </xacro:dvl_plugin_macro>
     <xacro:switchable_battery_consumer_macro
@@ -96,5 +96,5 @@
         scale="0.5">
         <inertia ixx="0.00001" ixy="0.0" ixz="0.0" iyy="0.00001" iyz="0.0" izz="0.00001" />
-        <origin xyz="-0.375 0 -0.16" rpy="0 0.3 0"/>
+        <origin xyz="0 -0.375 -0.16" rpy="0.3 0 0"/>
     </xacro:regular_camera_plugin_macro>
     <xacro:switchable_battery_consumer_macro
@@ -113,6 +113,6 @@
       topic=""/>
     <!-- Mount the chemical concentration sensor -->
-    <xacro:default_chemical_concentration_sensor namespace="${namespace}" parent_link="${namespace}/base_link">
+    <!-- <xacro:default_chemical_concentration_sensor namespace="${namespace}" parent_link="${namespace}/base_link">
       <origin xyz="0 0 0" rpy="0 0 0"/>
-    </xacro:default_chemical_concentration_sensor>
+    </xacro:default_chemical_concentration_sensor> -->
 </robot>
