Commit message: first cut at all six thruster

File: robots/smilodon_gazebo/urdf/smilodon_gazebo.xacro (robot description, xacro)
@@ -17,13 +17,9 @@
   <xacro:arg name="inertial_reference_frame" default="world"/>
   <!-- Includes -->
-  <!-- A collection of generic macros for colors, shapes, inertia, etc. -->
-  <xacro:include filename="$(find uuv_descriptions)/urdf/common.urdf.xacro"/>
-  <xacro:include filename="$(find uuv_dave)/urdf/sensor_snippets.xacro"/>
-  <xacro:include filename="$(find uuv_gazebo_ros_plugins)/urdf/snippets.xacro"/>
+  <!--xacro:include filename="$(find uuv_dave)/urdf/sensor_snippets.xacro"/>-->
+  <!---->
   <xacro:property name="visual_mesh_file" value="file://$(find smilodon_description)/meshes/smilodon_visual.dae"/>
   <xacro:property name="prop_mesh_file" value="file://$(find uuv_descriptions)/meshes/prop.dae"/>
  <xacro:property name="mass" value="1862.87"/>
-   <!-- Hydro parameters -->
-  <xacro:include filename="$(find smilodon_gazebo)/urdf/smilodon_hydro.xacro"/>
  <!-- base_link according to ROS conventions: x forward, z up -->
  <link name="$(arg namespace)/base_link">
@@ -34,5 +30,5 @@
    </inertial>
    <visual>
-     <origin xyz="0 0 0" rpy="0 0 0"/>
+     <origin xyz="0 0 0" rpy="0 0 1.5708"/>
      <geometry>
        <mesh filename="package://smilodon_description/meshes/smilodon_visual.dae" scale="1 1 1"/>
@@ -40,5 +36,5 @@
    </visual>
    <collision>
-     <origin xyz="0 0 0" rpy="0 0 0"/>
+     <origin xyz="0 0 0" rpy="0 0 1.5708"/>
      <geometry>
        <mesh filename="package://smilodon_description/meshes/smilodon_collision.dae" scale="1 1 1"/>
@@ -48,9 +44,44 @@
  <gazebo>
    <plugin name="uuv_plugin" filename="libuuv_underwater_object_ros_plugin.so">
+     <!-- Hydro parameters for the vehicle-->
      <fluid_density>1028.0</fluid_density>
      <flow_velocity_topic>hydrodynamics/current_velocity</flow_velocity_topic>
      <debug>$(arg debug)</debug>
-     <!-- Adding hydro parameters for the vehicle-->
-     <xacro:smilodon_hydro namespace="$(arg namespace)"/>
+     <link name="$(arg namespace)/base_link">
+       <neutrally_buoyant>1</neutrally_buoyant>
+       <!-- Volume, see p.31 in Berg2012 -->
+       <volume>1.8382</volume>
+       <box>
+         <width>1.5</width>
+         <length>2.6</length>
+         <height>1.6</height>
+       </box>
+       <!--
+	   Center of buoyancy according to eq. (3.1) p. 28 in Berg2012.
+	   The original values, [0.0822, -0.00773, 0.3872] however, seem to
+	   assume NWU (otherwise cob is below cog?).
+       -->
+       <center_of_buoyancy>0.0 0.0 0.3</center_of_buoyancy>
+       <hydrodynamic_model>
+         <type>fossen</type>
+         <!-- Added mass: see p.28 in Berg2012 -->
+         <added_mass>
+           779.79 -6.8773 -103.32  8.5426 -165.54 -7.8033
+           -6.8773    1222   51.29  409.44 -5.8488  62.726
+           -103.32   51.29  3659.9  6.1112 -386.42  10.774
+           8.5426  409.44  6.1112   534.9 -10.027  21.019
+           -165.54 -5.8488 -386.42 -10.027  842.69 -1.1162
+           -7.8033  62.726  10.775  21.019 -1.1162  224.32
+         </added_mass>
+         <!-- Linear damping: see p.31 in Berg2012 -->
+         <linear_damping>
+           -74.82 -69.48 -728.4 -268.8 -309.77 -105
+         </linear_damping>
+         <!-- Non-linear damping: see p.30 in Berg2012 -->
+         <quadratic_damping>
+           -748.22 -992.53 -1821.01 -672 -774.44 -523.27
+         </quadratic_damping>
+       </hydrodynamic_model>
+     </link>
    </plugin>
  </gazebo>
@@ -61,5 +92,61 @@
    </plugin>
  </gazebo>
- <!-- Joint state publisher plugin -->
- <xacro:default_joint_state_publisher namespace="$(arg namespace)" update_rate="50"/>
+ <!-- Define thrusters for propulsion -->
+ <!-- Common values, colors, converstion, standard shapes/inertia etc.
+      Dependency for the thruster_snippets.xacro-->
+ <xacro:include filename="$(find uuv_descriptions)/urdf/common.urdf.xacro"/>
+ <!-- Various thruster models -->
+ <xacro:include filename="$(find uuv_gazebo_ros_plugins)/urdf/thruster_snippets.xacro"/>
+ <xacro:property name="prop_mesh_file" value="file://$(find uuv_descriptions)/meshes/prop.dae"/>
+ <!-- Thruster joint and link snippet
+      Wrapper for the the thruster_module_first_order_basic_fcn_macro
+      defined in uuv_gazebo_ros_plugins/urdf/thruster_snippet.
+      Uses the "thruster_cf_basic_macro"
+        1) Basic curve
+	Input: x
+	Output: thrust
+	Function: thrust = rotorConstant * x * abs(x)
+ -->
+ <xacro:macro name="thruster_macro"
+	      params="thruster_id *origin">
+   <xacro:thruster_module_first_order_basic_fcn_macro
+       namespace="$(arg namespace)"
+       thruster_id="${thruster_id}"
+       mesh_filename="${prop_mesh_file}"
+       dyn_time_constant="0.05"
+       rotor_constant="0.00031">
+     <xacro:insert_block name="origin"/>
+   </xacro:thruster_module_first_order_basic_fcn_macro>
+ </xacro:macro>
+ <!-- Port-Aft -->
+ <xacro:thruster_macro thruster_id="0">
+   <origin xyz="-3.3 0.8 -0.1" rpy="${0*d2r} ${0*d2r} ${200.0*d2r}"/>
+ </xacro:thruster_macro>
+ <!-- Stbd-Aft -->
+ <xacro:thruster_macro thruster_id="1">
+   <origin xyz="-3.3 -0.8 -0.1" rpy="${0*d2r} ${0*d2r} ${160.0*d2r}"/>
+ </xacro:thruster_macro>
+ <!-- Port-Vert -->
+ <xacro:thruster_macro thruster_id="2">
+   <origin xyz="1.8 0.8 0.4" rpy="${0*d2r} ${-110.0*d2r} ${90.0*d2r}"/>
+ </xacro:thruster_macro>
+  <!-- Stbd-Vert -->
+ <xacro:thruster_macro thruster_id="3">
+   <origin xyz="1.8 -0.8 0.4" rpy="${0*d2r} ${-110*d2r} ${-90.0*d2r}"/>
+ </xacro:thruster_macro>
+  <!-- Port-Lat -->
+ <xacro:thruster_macro thruster_id="4">
+   <origin xyz="1.8 1.3 -0.07" rpy="${0*d2r} ${0*d2r} ${90.0*d2r}"/>
+ </xacro:thruster_macro>
+   <!-- Stbd-Lat -->
+ <xacro:thruster_macro thruster_id="5">
+   <origin xyz="1.8 -1.3 -0.07" rpy="${0*d2r} ${0*d2r} ${-90.0*d2r}"/>
+ </xacro:thruster_macro>
+ <!-- Default joint state publisher -->
+ <gazebo>
+   <plugin name="uuv_joint_state_publisher" filename="libuuv_joint_state_publisher.so">
+     <robotNamespace>$(arg namespace)</robotNamespace>
+     <updateRate>50</updateRate>
+   </plugin>
+ </gazebo>
 </robot>

Commit message: Adding a no logo texture and cleaned up mesh

File: robots/smilodon_gazebo/urdf/smilodon_gazebo.xacro (robot description, xacro)
@@ -19,11 +19,8 @@
   <!--xacro:include filename="$(find uuv_dave)/urdf/sensor_snippets.xacro"/>-->
   <!---->
-  <xacro:property name="visual_mesh_file" value="file://$(find smilodon_description)/meshes/smilodon_visual.dae"/>
-  <xacro:property name="prop_mesh_file" value="file://$(find uuv_descriptions)/meshes/prop.dae"/>
- <xacro:property name="mass" value="1862.87"/>
  <!-- base_link according to ROS conventions: x forward, z up -->
  <link name="$(arg namespace)/base_link">
    <inertial>
-     <mass value="${mass}"/>
+     <mass value="1862.87"/>
      <origin xyz="0 0 0"/>
      <inertia ixx="525.39" ixy="1.44" ixz="33.41" iyy="794.20" iyz="2.6" izz="691.23"/>
@@ -32,5 +29,5 @@
      <origin xyz="0 0 0" rpy="0 0 1.5708"/>
      <geometry>
-       <mesh filename="package://smilodon_description/meshes/smilodon_visual.dae" scale="1 1 1"/>
+       <mesh filename="package://smilodon_description/meshes/smilodon_nologo_visual.dae" scale="1 1 1"/>
      </geometry>
    </visual>
@@ -93,4 +90,5 @@
  </gazebo>
  <!-- Define thrusters for propulsion -->
+ <xacro:property name="prop_mesh_file" value="file://$(find uuv_descriptions)/meshes/prop.dae"/>
  <!-- Common values, colors, converstion, standard shapes/inertia etc.
       Dependency for the thruster_snippets.xacro-->
