Commit message: Remove lag from roll joint

File: dave_manipulator/predator_description/urdf/serial_arm_predator.xacro (robot description, xacro)
@@ -183,5 +183,5 @@
             <origin xyz="0.11275 -0.55503 0" rpy="0 0 -1.57079632679"/>
             <axis xyz="0 0 1"/>
-            <dynamics damping="50" friction="150"/>
+            <dynamics damping="30" friction="50"/>
             <limit lower="${-135 * d2r}" upper="${135 * d2r}" velocity=".25" effort="1000"/>
         </joint>

Commit message: restoring old predator dae files with link to texture

File: dave_manipulator/predator_description/urdf/serial_arm_predator.xacro (robot description, xacro)
@@ -105,5 +105,5 @@
                 <origin xyz="0 0 0" rpy="0 ${0.5*pi} 0"/>
                 <geometry>
-                    <mesh filename="file://$(find predator_description)/meshes/upperarm.dae"/>
+                    <mesh scale="0.7 0.7 0.4" filename="file://$(find predator_description)/meshes/upperarm.dae"/>
                 </geometry>
             </visual>
@@ -111,5 +111,5 @@
                 <origin xyz="0 0 0" rpy="0 ${0.5*pi} 0"/>
                 <geometry>
-                    <mesh filename="file://$(find predator_description)/meshes/upperarm.dae"/>
+                    <mesh scale="0.7 0.7 0.4" filename="file://$(find predator_description)/meshes/upperarm.dae"/>
                 </geometry>
             </collision>
@@ -165,5 +165,5 @@
                 <origin xyz="0 0 0" rpy="1.57079632679 1.57079632679 -1.57079632679"/>
                 <geometry>
-                    <mesh filename="file://$(find predator_description)/meshes/knuckle.dae"/>
+                    <mesh filename="file://$(find predator_description)/meshes/wrist.dae"/>
                 </geometry>
             </visual>
@@ -171,5 +171,5 @@
                 <origin xyz="0 0 0" rpy="1.57079632679 1.57079632679 -1.57079632679"/>
                 <geometry>
-                    <mesh filename="file://$(find predator_description)/meshes/knuckle.dae"/>
+                    <mesh filename="file://$(find predator_description)/meshes/wrist.dae"/>
                 </geometry>
             </collision>

Commit message: removing need for scaling attribute for upper arm

File: dave_manipulator/predator_description/urdf/serial_arm_predator.xacro (robot description, xacro)
@@ -105,5 +105,5 @@
                 <origin xyz="0 0 0" rpy="0 ${0.5*pi} 0"/>
                 <geometry>
-                    <mesh scale="0.7 0.7 0.4" filename="file://$(find predator_description)/meshes/upperarm.dae"/>
+                    <mesh filename="file://$(find predator_description)/meshes/upperarm.dae"/>
                 </geometry>
             </visual>
@@ -111,5 +111,5 @@
                 <origin xyz="0 0 0" rpy="0 ${0.5*pi} 0"/>
                 <geometry>
-                    <mesh scale="0.7 0.7 0.4" filename="file://$(find predator_description)/meshes/upperarm.dae"/>
+                    <mesh filename="file://$(find predator_description)/meshes/upperarm.dae"/>
                 </geometry>
             </collision>
