Commit message: Testing Predator Meshes

File: dave_manipulator/predator_description/urdf/parallel_gripper_predator.xacro (robot description, xacro)
@@ -21,10 +21,10 @@
         <origin xyz="${gripper_base_com}" rpy="0 0 0"/>
         </xacro:link_box_inertial>
-        <visual>
+        <!-- <visual>
             <origin xyz="0 0 0" rpy="0 0 0"/>
             <geometry>
                 <mesh filename="file://$(find oberon7_description)/meshes/parallel_gripper/visual/BaseGripper.dae"/>
             </geometry>
-        </visual>
+        </visual> -->
         <collision>
             <origin xyz="${gripper_base_com}" rpy="0 0 0"/>
@@ -52,10 +52,10 @@
         <origin xyz="${finger_com}" rpy="0 0 0"/>
         </xacro:link_box_inertial>
-        <visual>
+        <!-- <visual>
             <origin xyz="0 0 0" rpy="0 0 0"/>
             <geometry>
                 <mesh filename="file://$(find oberon7_description)/meshes/parallel_gripper/visual/Finger.dae"/>
             </geometry>
-        </visual>
+        </visual> -->
         <collision>
             <origin xyz="0 0 0" rpy="0 0 0"/>
@@ -82,10 +82,10 @@
         <origin xyz="${finger_tip_com}" rpy="0 0 0"/>
         </xacro:link_box_inertial>
-        <visual>
+        <!-- <visual>
             <origin xyz="0 0 0" rpy="0 0 0"/>
             <geometry>
                 <mesh filename="file://$(find oberon7_description)/meshes/parallel_gripper/visual/FingerTip.dae"/>
             </geometry>
-        </visual>
+        </visual> -->
         <collision>
             <origin xyz="0 0 0" rpy="0 0 0"/>
@@ -111,10 +111,10 @@
         <origin xyz="${finger_com}" rpy="0 0 0"/>
         </xacro:link_box_inertial>
-        <visual>
+        <!-- <visual>
             <origin xyz="0 0 0" rpy="${PI} 0 0"/>
             <geometry>
                 <mesh filename="file://$(find oberon7_description)/meshes/parallel_gripper/visual/Finger.dae"/>
             </geometry>
-        </visual>
+        </visual> -->
         <collision>
             <origin xyz="0 0 0" rpy="${PI} 0 0"/>
@@ -141,10 +141,10 @@
         <origin xyz="${finger_tip_com}" rpy="0 0 0"/>
         </xacro:link_box_inertial>
-        <visual>
+        <!-- <visual>
             <origin xyz="0 0 0" rpy="0 0 0"/>
             <geometry>
                 <mesh filename="file://$(find oberon7_description)/meshes/parallel_gripper/visual/FingerTip.dae"/>
             </geometry>
-        </visual>
+        </visual> -->
         <collision>
             <origin xyz="0 0 0" rpy="0 0 0"/>

File: dave_manipulator/predator_description/urdf/serial_arm_predator.xacro (robot description, xacro)
@@ -53,5 +53,9 @@
                 <origin xyz="0 0 ${-base_height/2.5}" rpy="0 0 0"/>
                 <geometry>
-                    <box size="${predator_base_width} ${predator_base_width} ${predator_shoulder_height/4}" />
+                    <!-- <box size="${predator_base_width} ${predator_base_width} ${predator_shoulder_height/4}" /> -->
+                    <!-- <mesh filename="file://$(find predator_description)/meshes/Predator.dae"/> -->
+                    <!-- <mesh filename="file://$(find predator_description)/meshes/Predator-base-bigarm.dae"/> -->
+                    <mesh filename="file://$(find predator_description)/meshes/Predator-root.dae"/>
+                    <!-- <box size="${predator_base_width} ${predator_base_width} ${predator_shoulder_height/4}" /> -->
                 </geometry>
             </visual>
@@ -75,5 +79,5 @@
                 <origin xyz="${shoulder_link_com}" rpy="0 0 0"/>
                 <geometry>
-                    <cylinder radius="${predator_shoulder_radius}" length="${predator_shoulder_height}" />
+                    <mesh filename="file://$(find predator_description)/meshes/Predator-base.dae"/>
                 </geometry>
             </visual>
@@ -106,5 +110,7 @@
                 <origin xyz="${predator_upper_arm_length/2} 0 0" rpy="0 ${0.5*pi} 0"/>
                 <geometry>
-                    <cylinder radius="${0.5 * upper_arm_width}" length="${predator_upper_arm_length}"/>
+                    <mesh filename="file://$(find predator_description)/meshes/Predator-upperarm.dae"/>
+                <!-- Predator-upperarm.dae -->
+                    <!-- <cylinder radius="${0.5 * upper_arm_width}" length="${predator_upper_arm_length}"/> -->
                 </geometry>
             </visual>
@@ -139,5 +145,8 @@
                 <origin xyz="${elbow_link_x_disp} ${-predator_elbow_length/2} 0" rpy="0 ${0.5*pi} ${0.5*pi}"/>
                 <geometry>
-                    <cylinder radius="${0.5 * elbow_link_height}" length="${predator_elbow_length}"/>
+                    <mesh filename="file://$(find predator_description)/meshes/Predator-forearm.dae"/>
+                    <!-- <mesh filename="file://$(find predator_description)/meshes/Predator-base-bigarm.dae"/> -->
+                    <!-- <mesh filename="file://$(find predator_description)/meshes/Predator-claw-left.dae"/> -->
+                    <!-- <cylinder radius="${0.5 * elbow_link_height}" length="${predator_elbow_length}"/> -->
                 </geometry>
             </visual>
@@ -170,7 +179,10 @@
             </xacro:link_box_inertial>
             <visual>
-                <origin xyz="${forearm_com}" rpy="${0.5*PI} 0 0"/>
-                <geometry>
-                    <cylinder radius="${0.5 * forearm_width}" length="${forearm_height}"/>
+                <origin xyz="0 0 0" rpy="${0.5*PI} 0 0"/>
+                <!-- <origin xyz="${forearm_com}" rpy="${0.5*PI} 0 0"/> -->
+                <geometry>
+                    <mesh filename="file://$(find predator_description)/meshes/Predator-knuckle.dae"/>
+                    <!-- <mesh filename="file://$(find predator_description)/meshes/Predator-hand.dae"/> -->
+                    <!-- <cylinder radius="${0.5 * forearm_width}" length="${forearm_height}"/> -->
                 </geometry>
             </visual>
@@ -201,10 +213,10 @@
                 <origin xyz="${wrist_com}" rpy="0 0 0"/>
             </xacro:link_box_inertial>
-            <visual>
+            <!-- <visual>
                 <origin xyz="${predator_wrist_height/2} 0 0" rpy="0 ${0.5*pi} 0"/>
                 <geometry>
                     <cylinder radius="${0.5 * wrist_height}" length="${predator_wrist_height}"/>
                 </geometry>
-            </visual>
+            </visual> -->
             <collision>
                 <origin xyz="${wrist_com}" rpy="0 ${0.5*pi} 0"/>

Commit message: Place visual meshes in their right place

File: dave_manipulator/predator_description/urdf/parallel_gripper_predator.xacro (robot description, xacro)
@@ -21,10 +21,10 @@
         <origin xyz="${gripper_base_com}" rpy="0 0 0"/>
         </xacro:link_box_inertial>
-        <!-- <visual>
-            <origin xyz="0 0 0" rpy="0 0 0"/>
+        <visual>
+            <origin xyz="0 0 0" rpy="${PI*0.5} 0 ${-PI*0.5}"/>
             <geometry>
-                <mesh filename="file://$(find oberon7_description)/meshes/parallel_gripper/visual/BaseGripper.dae"/>
+                <mesh filename="file://$(find predator_description)/meshes/Predator-hand_centralized.dae"/>
             </geometry>
-        </visual> -->
+        </visual>
         <collision>
             <origin xyz="${gripper_base_com}" rpy="0 0 0"/>
@@ -35,9 +35,10 @@
     </link>
     <joint name="${namespace}/wrist" type="revolute">
-      <parent link="${namespace}/wrist_link"/>
+      <parent link="${namespace}/forearm"/>
       <child link="${namespace}/end_effector"/>
-       <origin xyz="${predator_wrist_height} 0 0" rpy="${-PI*0.5} 0 0"/>
-       <!-- <origin xyz="0.19304 0 0" rpy="${-PI*0.5} 0 0"/> -->
-      <axis xyz="1 0 0"/>
+       <!-- <origin xyz="${predator_wrist_height} 0 0" rpy="${-PI*0.5} 0 0"/> -->
+<!-- 0.00038	-0.12137 -->
+       <origin xyz="0.12137 -0.00038 0" rpy="${PI*0.5} 0 0"/>
+      <axis xyz="0 0 1"/>
       <dynamics damping="10" friction="5"/>
       <limit effort="10" lower="${-2*PI}" upper="${2*PI}" velocity="${gripper_velocity}"/>
@@ -52,10 +53,11 @@
         <origin xyz="${finger_com}" rpy="0 0 0"/>
         </xacro:link_box_inertial>
-        <!-- <visual>
-            <origin xyz="0 0 0" rpy="0 0 0"/>
+        <visual>
+            <!-- <origin xyz="0 0 0" rpy="0 0 0"/> -->
+            <origin xyz="0 0 0" rpy="${PI*0.5} 0 ${-PI*0.5}"/>
             <geometry>
-                <mesh filename="file://$(find oberon7_description)/meshes/parallel_gripper/visual/Finger.dae"/>
+                <mesh filename="file://$(find predator_description)/meshes/Predator-claw-right_centralized.dae"/>
             </geometry>
-        </visual> -->
+        </visual>
         <collision>
             <origin xyz="0 0 0" rpy="0 0 0"/>
@@ -68,6 +70,6 @@
         <parent link="${namespace}/end_effector"/>
         <child link="${namespace}/finger_left"/>
-        <origin xyz="0.0444267 0.0391376 0" rpy="0 0 0"/>
-        <axis xyz="0 0 1"/>
+        <origin xyz="0.23387 -0.02401 -0.017121" rpy="0 0 0"/>
+        <axis xyz="0 0 -1"/>
         <dynamics damping="5" friction="10"/>
         <limit effort="${gripper_effort}" lower="0" upper="${PI*0.3333}" velocity="${gripper_velocity}"/>
@@ -82,10 +84,12 @@
         <origin xyz="${finger_tip_com}" rpy="0 0 0"/>
         </xacro:link_box_inertial>
-        <!-- <visual>
-            <origin xyz="0 0 0" rpy="0 0 0"/>
+        <visual>
+            <!-- <origin xyz="0 0 0" rpy="${PI/2} 0 ${-PI/2}"/> -->
+            <origin xyz="0 0 0" rpy="${PI/2}  0  ${-PI/2}"/>
+            <!-- <origin xyz="0 0 0" rpy="1.57079632679  1.57079632679  1.57079632679"/> -->
             <geometry>
-                <mesh filename="file://$(find oberon7_description)/meshes/parallel_gripper/visual/FingerTip.dae"/>
+                <mesh filename="file://$(find predator_description)/meshes/Predator-tip-right_centralized.dae"/>
             </geometry>
-        </visual> -->
+        </visual>
         <collision>
             <origin xyz="0 0 0" rpy="0 0 0"/>
@@ -98,5 +102,5 @@
         <parent link="${namespace}/finger_left"/>
         <child link="${namespace}/finger_tip_left"/>
-        <origin xyz="0.06431 0 0" rpy="${PI} 0 0"/>
+        <origin xyz="0.0805 0.006578 0" rpy="0 0 0"/>
         <axis xyz="0 0 1"/>
         <dynamics damping="5" friction="10"/>
@@ -111,10 +115,11 @@
         <origin xyz="${finger_com}" rpy="0 0 0"/>
         </xacro:link_box_inertial>
-        <!-- <visual>
-            <origin xyz="0 0 0" rpy="${PI} 0 0"/>
+        <visual>
+            <!-- <origin xyz="0 0 0" rpy="0 0 0"/> -->
+            <origin xyz="0 0 0" rpy="${PI/2} 0 ${-PI/2}"/>
             <geometry>
-                <mesh filename="file://$(find oberon7_description)/meshes/parallel_gripper/visual/Finger.dae"/>
+                <mesh filename="file://$(find predator_description)/meshes/Predator-claw-left_centralized.dae"/>
             </geometry>
-        </visual> -->
+        </visual>
         <collision>
             <origin xyz="0 0 0" rpy="${PI} 0 0"/>
@@ -127,6 +132,7 @@
         <parent link="${namespace}/end_effector"/>
         <child link="${namespace}/finger_right"/>
-        <origin xyz="0.0444267 -0.0391376 0" rpy="${PI} ${PI} ${PI}"/>
-        <axis xyz="0 0 -1"/>
+        <!-- <origin xyz="0.0444267 -0.0391376 0" rpy="${PI} ${PI} ${PI}"/> -->
+        <origin xyz="0.23387 0.02401 -0.017121" rpy="0 0 0"/>
+        <axis xyz="0 0 1"/>
         <dynamics damping="5" friction="10"/>
         <limit effort="${gripper_effort}" lower="0" upper="${PI*0.3333}" velocity="${gripper_velocity}"/>
@@ -141,10 +147,10 @@
         <origin xyz="${finger_tip_com}" rpy="0 0 0"/>
         </xacro:link_box_inertial>
-        <!-- <visual>
-            <origin xyz="0 0 0" rpy="0 0 0"/>
+        <visual>
+            <origin xyz="0 0 0" rpy="${PI/2} 0 ${-PI/2}"/>
             <geometry>
-                <mesh filename="file://$(find oberon7_description)/meshes/parallel_gripper/visual/FingerTip.dae"/>
+                <mesh filename="file://$(find predator_description)/meshes/Predator-tip-left_centralized.dae"/>
             </geometry>
-        </visual> -->
+        </visual>
         <collision>
             <origin xyz="0 0 0" rpy="0 0 0"/>
@@ -157,6 +163,6 @@
         <parent link="${namespace}/finger_right"/>
         <child link="${namespace}/finger_tip_right"/>
-        <origin xyz="0.06431 0 0" rpy="0 0 0"/>
-        <axis xyz="0 0 1"/>
+        <origin xyz="0.0805 -0.006578 0" rpy="0 0 0"/>
+        <axis xyz="0 0 -1"/>
         <dynamics damping="5" friction="10"/>
         <limit effort="0" lower="0" upper="0" velocity="0"/>

File: dave_manipulator/predator_description/urdf/serial_arm_predator.xacro (robot description, xacro)
@@ -51,18 +51,13 @@
             </xacro:link_box_inertial>
             <visual>
-                <origin xyz="0 0 ${-base_height/2.5}" rpy="0 0 0"/>
-                <geometry>
-                    <!-- <box size="${predator_base_width} ${predator_base_width} ${predator_shoulder_height/4}" /> -->
-                    <!-- <mesh filename="file://$(find predator_description)/meshes/Predator.dae"/> -->
-                    <!-- <mesh filename="file://$(find predator_description)/meshes/Predator-base-bigarm.dae"/> -->
-                    <mesh filename="file://$(find predator_description)/meshes/Predator-root.dae"/>
-                    <!-- <box size="${predator_base_width} ${predator_base_width} ${predator_shoulder_height/4}" /> -->
-                </geometry>
-            </visual>
-            <collision>
                 <origin xyz="0 0 0" rpy="0 0 0"/>
                 <geometry>
                     <box size="${predator_base_width} ${predator_base_width} ${predator_shoulder_height/4}" />
-                    <!-- <mesh filename="file://$(find oberon7_description)/meshes/serial_arm/collision/Base.stl"/> -->
+                </geometry>
+            </visual>
+            <collision>
+                <origin xyz="0 0 0" rpy="0 0 0"/>
+                <geometry>
+                    <box size="${predator_base_width} ${predator_base_width} ${predator_shoulder_height/4}" />
                 </geometry>
             </collision>
@@ -77,12 +72,13 @@
             </xacro:link_box_inertial>
             <visual>
+                <origin xyz="0 0 0" rpy="0 0 1.57079632679"/>
+                <!-- <origin xyz="${shoulder_link_com}" rpy="0 0 0"/> -->
+                <geometry>
+                    <mesh filename="file://$(find predator_description)/meshes/Predator-base_centralized.dae"/>
+                </geometry>
+            </visual>
+            <collision>
                 <origin xyz="${shoulder_link_com}" rpy="0 0 0"/>
                 <geometry>
-                    <mesh filename="file://$(find predator_description)/meshes/Predator-base.dae"/>
-                </geometry>
-            </visual>
-            <collision>
-                <origin xyz="${shoulder_link_com}" rpy="0 0 0"/>
-                <geometry>
                     <cylinder radius="${predator_shoulder_radius}" length="${predator_shoulder_height}" />
                 </geometry>
@@ -90,4 +86,6 @@
         </link>
         <joint name="${namespace}/azimuth" type="revolute">
+            <origin xyz="0 0 0" rpy="0 0 0"/>
+            <!-- <origin xyz="0 -0.1 0.1" rpy="0 0 0"/> -->
             <parent link="${namespace}/base"/>
             <child link="${namespace}/shoulder_link"/>
@@ -108,13 +106,11 @@
             </xacro:link_box_inertial>
             <visual>
-                <origin xyz="${predator_upper_arm_length/2} 0 0" rpy="0 ${0.5*pi} 0"/>
-                <geometry>
-                    <mesh filename="file://$(find predator_description)/meshes/Predator-upperarm.dae"/>
-                <!-- Predator-upperarm.dae -->
-                    <!-- <cylinder radius="${0.5 * upper_arm_width}" length="${predator_upper_arm_length}"/> -->
-                </geometry>
-            </visual>
-            <collision>
-                <origin xyz="${predator_upper_arm_length/2} 0 0" rpy="0 ${0.5*pi} 0"/>
+                <origin xyz="0 0 0" rpy="0 ${0.5*pi} 0"/>
+                <geometry>
+                    <mesh filename="file://$(find predator_description)/meshes/Predator-upperarm_centralized.dae"/>
+                </geometry>
+            </visual>
+            <collision>
+                <origin xyz="0 0 0" rpy="0 ${0.5*pi} 0"/>
                 <geometry>
                     <cylinder radius="${0.5 * upper_arm_width}" length="${predator_upper_arm_length}"/>
@@ -126,5 +122,5 @@
             <child link="${namespace}/upper_arm"/>
             <!-- <origin xyz="0.06955 0.00015 0.01536" rpy="${0.5*pi} 0 0"/> -->
-            <origin xyz="${predator_joint_1_2_x} 0 ${predator_joint_1_2_z}" rpy="${0.5*pi} 0 0"/>
+            <origin xyz="0.200369 0 0.209467" rpy="${0.5*pi} 0 0"/>
             <axis xyz="0 0 1"/>
             <!-- <dynamics damping="50" friction="200"/> -->
@@ -143,14 +139,11 @@
             </xacro:link_box_inertial>
             <visual>
-                <origin xyz="${elbow_link_x_disp} ${-predator_elbow_length/2} 0" rpy="0 ${0.5*pi} ${0.5*pi}"/>
-                <geometry>
-                    <mesh filename="file://$(find predator_description)/meshes/Predator-forearm.dae"/>
-                    <!-- <mesh filename="file://$(find predator_description)/meshes/Predator-base-bigarm.dae"/> -->
-                    <!-- <mesh filename="file://$(find predator_description)/meshes/Predator-claw-left.dae"/> -->
-                    <!-- <cylinder radius="${0.5 * elbow_link_height}" length="${predator_elbow_length}"/> -->
-                </geometry>
-            </visual>
-            <collision>
-                <origin xyz="${elbow_link_x_disp} ${-predator_elbow_length/2} 0" rpy="0 ${0.5*pi} ${0.5*pi}"/>
+                <origin xyz="0 0 0" rpy="0 ${0.5*pi} ${0.5*pi}"/>
+                <geometry>
+                    <mesh filename="file://$(find predator_description)/meshes/Predator-forearm_centralized.dae"/>
+                </geometry>
+            </visual>
+            <collision>
+                <origin xyz="0 0 0" rpy="0 ${0.5*pi} ${0.5*pi}"/>
                 <geometry>
                     <cylinder radius="${0.5 * elbow_link_height}" length="${predator_elbow_length}"/>
@@ -162,5 +155,5 @@
             <child link="${namespace}/elbow_link"/>
             <!-- <origin xyz="0.55616 -0.01229 0" rpy="0 0 0"/> -->
-            <origin xyz="${predator_upper_arm_length} -0.01229 0" rpy="0 0 0"/>
+            <origin xyz="0.87315 0 0" rpy="0 0 0"/>
             <!-- <dynamics damping="50" friction="200"/> -->
             <dynamics damping="50" friction="150"/>
@@ -179,10 +172,7 @@
             </xacro:link_box_inertial>
             <visual>
-                <origin xyz="0 0 0" rpy="${0.5*PI} 0 0"/>
-                <!-- <origin xyz="${forearm_com}" rpy="${0.5*PI} 0 0"/> -->
-                <geometry>
-                    <mesh filename="file://$(find predator_description)/meshes/Predator-knuckle.dae"/>
-                    <!-- <mesh filename="file://$(find predator_description)/meshes/Predator-hand.dae"/> -->
-                    <!-- <cylinder radius="${0.5 * forearm_width}" length="${forearm_height}"/> -->
+                <origin xyz="0 0 0" rpy="1.57079632679 1.57079632679 -1.57079632679"/>
+                <geometry>
+                    <mesh filename="file://$(find predator_description)/meshes/Predator-knuckle_centralized.dae"/>
                 </geometry>
             </visual>
@@ -197,5 +187,5 @@
             <parent link="${namespace}/elbow_link"/>
             <child link="${namespace}/forearm"/>
-            <origin xyz="${elbow_link_x_disp} ${-predator_joint_3_4_y} 0" rpy="0 0 0"/>
+            <origin xyz="0.11275 -0.55503 0" rpy="0 0 -1.57079632679"/>
             <axis xyz="0 0 1"/>
             <dynamics damping="150" friction="500"/>
@@ -205,36 +195,4 @@
         </joint>
         <xacro:simple_transmission joint="${namespace}/roll" />
-        <!-- WRIST 1  -->
-        <link name="${namespace}/wrist_link">
-            <xacro:link_box_inertial mass="${total_mass * wrist_volume / total_volume_bbox}"
-                        width="${wrist_width}"
-                        length="${predator_wrist_height}"
-                        height="${wrist_height}">
-                <origin xyz="${wrist_com}" rpy="0 0 0"/>
-            </xacro:link_box_inertial>
-            <!-- <visual>
-                <origin xyz="${predator_wrist_height/2} 0 0" rpy="0 ${0.5*pi} 0"/>
-                <geometry>
-                    <cylinder radius="${0.5 * wrist_height}" length="${predator_wrist_height}"/>
-                </geometry>
-            </visual> -->
-            <collision>
-                <origin xyz="${wrist_com}" rpy="0 ${0.5*pi} 0"/>
-                <geometry>
-                    <cylinder radius="${0.5 * wrist_height}" length="${predator_wrist_height}"/>
-                </geometry>
-            </collision>
-        </link>
-        <joint name="${namespace}/pitch" type="revolute">
-            <parent link="${namespace}/forearm"/>
-            <child link="${namespace}/wrist_link"/>
-            <origin xyz="0 ${-forearm_height} 0" rpy="${1.5*PI} ${PI} ${0.5*PI}"/>
-            <axis xyz="0 0 1"/>
-            <!-- <dynamics damping="50" friction="200"/> -->
-            <dynamics damping="10" friction="10"/>
-            <!-- <limit lower="${-90 * d2r}" upper="${90 * d2r}" velocity=".26" effort="200"/> -->
-            <limit lower="${-90 * d2r}" upper="${90 * d2r}" velocity=".3" effort="50"/>
-        </joint>
-        <xacro:simple_transmission joint="${namespace}/pitch" />
         <!-- Adding parallel gripper  -->
         <xacro:include filename="$(find predator_description)/urdf/parallel_gripper_predator.xacro" />
