Commit message: Added the collision models (collision = visual)

File: dave_manipulator/predator_description/urdf/parallel_gripper_predator.xacro (robot description, xacro)
@@ -28,7 +28,11 @@
         </visual>
         <collision>
-            <origin xyz="${gripper_base_com}" rpy="0 0 0"/>
+            <!-- <origin xyz="${gripper_base_com}" rpy="0 0 0"/>
             <geometry>
                 <box size="${gripper_base_length} ${gripper_base_width} ${gripper_base_height}"/>
+            </geometry> -->
+            <origin xyz="0 0 0" rpy="${PI*0.5} 0 ${-PI*0.5}"/>
+            <geometry>
+                <mesh filename="file://$(find predator_description)/meshes/Predator-hand_centralized.dae"/>
             </geometry>
         </collision>
@@ -37,6 +41,4 @@
       <parent link="${namespace}/forearm"/>
       <child link="${namespace}/end_effector"/>
-       <!-- <origin xyz="${predator_wrist_height} 0 0" rpy="${-PI*0.5} 0 0"/> -->
-<!-- 0.00038	-0.12137 -->
        <origin xyz="0.12137 -0.00038 0" rpy="${PI*0.5} 0 0"/>
       <axis xyz="0 0 1"/>
@@ -47,4 +49,5 @@
     <!-- Finger left  -->
     <link name="${namespace}/finger_left">
+        <origin xyz=" 0 0 0" rpy="0 0 -1"/>
         <xacro:link_box_inertial mass="${total_mass * finger_volume / total_volume}"
                     width="${finger_width}"
@@ -54,5 +57,4 @@
         </xacro:link_box_inertial>
         <visual>
-            <!-- <origin xyz="0 0 0" rpy="0 0 0"/> -->
             <origin xyz="0 0 0" rpy="${PI*0.5} 0 ${-PI*0.5}"/>
             <geometry>
@@ -61,7 +63,7 @@
         </visual>
         <collision>
-            <origin xyz="0 0 0" rpy="0 0 0"/>
+            <origin xyz="0 0 0" rpy="${PI*0.5} 0 ${-PI*0.5}"/>
             <geometry>
-                <mesh filename="file://$(find oberon7_description)/meshes/parallel_gripper/visual/Finger.dae"/>
+                <mesh filename="file://$(find predator_description)/meshes/Predator-claw-right_centralized.dae"/>
             </geometry>
         </collision>
@@ -85,7 +87,5 @@
         </xacro:link_box_inertial>
         <visual>
-            <!-- <origin xyz="0 0 0" rpy="${PI/2} 0 ${-PI/2}"/> -->
             <origin xyz="0 0 0" rpy="${PI/2}  0  ${-PI/2}"/>
-            <!-- <origin xyz="0 0 0" rpy="1.57079632679  1.57079632679  1.57079632679"/> -->
             <geometry>
                 <mesh filename="file://$(find predator_description)/meshes/Predator-tip-right_centralized.dae"/>
@@ -93,7 +93,7 @@
         </visual>
         <collision>
-            <origin xyz="0 0 0" rpy="0 0 0"/>
+            <origin xyz="0 0 0" rpy="${PI/2}  0  ${-PI/2}"/>
             <geometry>
-                <mesh filename="file://$(find oberon7_description)/meshes/parallel_gripper/visual/FingerTip.dae"/>
+                <mesh filename="file://$(find predator_description)/meshes/Predator-tip-right_centralized.dae"/>
             </geometry>
         </collision>
@@ -116,5 +116,4 @@
         </xacro:link_box_inertial>
         <visual>
-            <!-- <origin xyz="0 0 0" rpy="0 0 0"/> -->
             <origin xyz="0 0 0" rpy="${PI/2} 0 ${-PI/2}"/>
             <geometry>
@@ -123,7 +122,7 @@
         </visual>
         <collision>
-            <origin xyz="0 0 0" rpy="${PI} 0 0"/>
+            <origin xyz="0 0 0" rpy="${PI/2} 0 ${-PI/2}"/>
             <geometry>
-                <mesh filename="file://$(find oberon7_description)/meshes/parallel_gripper/visual/Finger.dae"/>
+                <mesh filename="file://$(find predator_description)/meshes/Predator-claw-left_centralized.dae"/>
             </geometry>
         </collision>
@@ -154,7 +153,7 @@
         </visual>
         <collision>
-            <origin xyz="0 0 0" rpy="0 0 0"/>
+            <origin xyz="0 0 0" rpy="${PI/2} 0 ${-PI/2}"/>
             <geometry>
-                <mesh filename="file://$(find oberon7_description)/meshes/parallel_gripper/visual/FingerTip.dae"/>
+                <mesh filename="file://$(find predator_description)/meshes/Predator-tip-left_centralized.dae"/>
             </geometry>
         </collision>

File: dave_manipulator/predator_description/urdf/serial_arm_predator.xacro (robot description, xacro)
@@ -53,5 +53,5 @@
                 <origin xyz="0 0 0" rpy="0 0 0"/>
                 <geometry>
-                    <box size="${predator_base_width} ${predator_base_width} ${predator_shoulder_height/4}" />
+                    <mesh filename="file://$(find predator_description)/meshes/Predator-root_centralized.dae"/>
                 </geometry>
             </visual>
@@ -59,5 +59,5 @@
                 <origin xyz="0 0 0" rpy="0 0 0"/>
                 <geometry>
-                    <box size="${predator_base_width} ${predator_base_width} ${predator_shoulder_height/4}" />
+                    <mesh filename="file://$(find predator_description)/meshes/Predator-root_centralized.dae"/>
                 </geometry>
             </collision>
@@ -73,5 +73,4 @@
             <visual>
                 <origin xyz="0 0 0" rpy="0 0 1.57079632679"/>
-                <!-- <origin xyz="${shoulder_link_com}" rpy="0 0 0"/> -->
                 <geometry>
                     <mesh filename="file://$(find predator_description)/meshes/Predator-base_centralized.dae"/>
@@ -79,7 +78,7 @@
             </visual>
             <collision>
-                <origin xyz="${shoulder_link_com}" rpy="0 0 0"/>
+                <origin xyz="0 0 0" rpy="0 0 1.57079632679"/>
                 <geometry>
-                    <cylinder radius="${predator_shoulder_radius}" length="${predator_shoulder_height}" />
+                    <mesh filename="file://$(find predator_description)/meshes/Predator-base_centralized.dae"/>
                 </geometry>
             </collision>
@@ -87,12 +86,10 @@
         <joint name="${namespace}/azimuth" type="revolute">
             <origin xyz="0 0 0" rpy="0 0 0"/>
-            <!-- <origin xyz="0 -0.1 0.1" rpy="0 0 0"/> -->
             <parent link="${namespace}/base"/>
             <child link="${namespace}/shoulder_link"/>
             <axis xyz="0 0 1"/>
-            <!-- <dynamics damping="50" friction="200"/> -->
+            <origin xyz="0 0 0.0003" rpy="0 0 0"/>
             <dynamics damping="100" friction="150"/>
             <limit lower="${-60 * d2r}" upper="${60 * d2r}" velocity="0.17" effort="200"/>
-            <!-- <limit lower="${-60 * d2r}" upper="${60 * d2r}" velocity="0.17" effort="1000"/> -->
         </joint>
         <xacro:simple_transmission joint="${namespace}/azimuth" />
@@ -114,5 +111,5 @@
                 <origin xyz="0 0 0" rpy="0 ${0.5*pi} 0"/>
                 <geometry>
-                    <cylinder radius="${0.5 * upper_arm_width}" length="${predator_upper_arm_length}"/>
+                    <mesh filename="file://$(find predator_description)/meshes/Predator-upperarm_centralized.dae"/>
                 </geometry>
             </collision>
@@ -121,5 +118,4 @@
             <parent link="${namespace}/shoulder_link"/>
             <child link="${namespace}/upper_arm"/>
-            <!-- <origin xyz="0.06955 0.00015 0.01536" rpy="${0.5*pi} 0 0"/> -->
             <origin xyz="0.200369 0 0.209467" rpy="${0.5*pi} 0 0"/>
             <axis xyz="0 0 1"/>
@@ -147,5 +143,5 @@
                 <origin xyz="0 0 0" rpy="0 ${0.5*pi} ${0.5*pi}"/>
                 <geometry>
-                    <cylinder radius="${0.5 * elbow_link_height}" length="${predator_elbow_length}"/>
+                    <mesh filename="file://$(find predator_description)/meshes/Predator-forearm_centralized.dae"/>
                 </geometry>
             </collision>
@@ -154,5 +150,4 @@
             <parent link="${namespace}/upper_arm"/>
             <child link="${namespace}/elbow_link"/>
-            <!-- <origin xyz="0.55616 -0.01229 0" rpy="0 0 0"/> -->
             <origin xyz="0.87315 0 0" rpy="0 0 0"/>
             <!-- <dynamics damping="50" friction="200"/> -->
@@ -160,5 +155,4 @@
             <axis xyz="0 0 1"/>
             <limit lower="${-90 * d2r}" upper="${60 * d2r}" velocity=".15" effort="300"/>
-            <!-- <limit lower="${-90 * d2r}" upper="${60 * d2r}" velocity=".13" effort="1000"/> -->
         </joint>
         <xacro:simple_transmission joint="${namespace}/elbow" />
@@ -178,7 +172,7 @@
             </visual>
             <collision>
-                <origin xyz="${forearm_com}" rpy="${0.5*PI} 0 0"/>
+                <origin xyz="0 0 0" rpy="1.57079632679 1.57079632679 -1.57079632679"/>
                 <geometry>
-                    <cylinder radius="${0.5 * forearm_width}" length="${forearm_height}"/>
+                    <mesh filename="file://$(find predator_description)/meshes/Predator-knuckle_centralized.dae"/>
                 </geometry>
             </collision>
@@ -189,7 +183,5 @@
             <origin xyz="0.11275 -0.55503 0" rpy="0 0 -1.57079632679"/>
             <axis xyz="0 0 1"/>
-            <dynamics damping="150" friction="500"/>
-            <!-- <dynamics damping="300" friction="1000"/> -->
-            <!-- <limit lower="${-135 * d2r}" upper="${135 * d2r}" velocity=".15" effort="200"/> -->
+            <dynamics damping="50" friction="150"/>
             <limit lower="${-135 * d2r}" upper="${135 * d2r}" velocity=".25" effort="1000"/>
         </joint>

Commit message: Make end effector more claw like

File: dave_manipulator/predator_description/urdf/parallel_gripper_predator.xacro (robot description, xacro)
@@ -72,5 +72,5 @@
         <parent link="${namespace}/end_effector"/>
         <child link="${namespace}/finger_left"/>
-        <origin xyz="0.23387 -0.02401 -0.017121" rpy="0 0 0"/>
+        <origin xyz="0.23387 -0.02401 -0.017121" rpy="0 0 ${-15*d2r}"/>
         <axis xyz="0 0 -1"/>
         <dynamics damping="5" friction="10"/>
@@ -102,5 +102,5 @@
         <parent link="${namespace}/finger_left"/>
         <child link="${namespace}/finger_tip_left"/>
-        <origin xyz="0.0805 0.006578 0" rpy="0 0 0"/>
+        <origin xyz="0.0805 0.006578 0" rpy="0 0 ${15*d2r}"/>
         <axis xyz="0 0 1"/>
         <dynamics damping="5" friction="10"/>
@@ -132,5 +132,5 @@
         <child link="${namespace}/finger_right"/>
         <!-- <origin xyz="0.0444267 -0.0391376 0" rpy="${PI} ${PI} ${PI}"/> -->
-        <origin xyz="0.23387 0.02401 -0.017121" rpy="0 0 0"/>
+        <origin xyz="0.23387 0.02401 -0.017121" rpy="0 0 ${15*d2r}"/>
         <axis xyz="0 0 1"/>
         <dynamics damping="5" friction="10"/>
@@ -162,5 +162,5 @@
         <parent link="${namespace}/finger_right"/>
         <child link="${namespace}/finger_tip_right"/>
-        <origin xyz="0.0805 -0.006578 0" rpy="0 0 0"/>
+        <origin xyz="0.0805 -0.006578 0" rpy="0 0 ${-15*d2r}"/>
         <axis xyz="0 0 -1"/>
         <dynamics damping="5" friction="10"/>

Commit message: Remove osculations at end effector

File: dave_manipulator/predator_description/urdf/parallel_gripper_predator.xacro (robot description, xacro)
@@ -74,6 +74,7 @@
         <origin xyz="0.23387 -0.02401 -0.017121" rpy="0 0 ${-15*d2r}"/>
         <axis xyz="0 0 -1"/>
-        <dynamics damping="5" friction="10"/>
-        <limit effort="${gripper_effort}" lower="0" upper="${PI*0.3333}" velocity="${gripper_velocity}"/>
+        <dynamics damping="2" />
+        <!-- <dynamics damping="5" friction="5"/> -->
+        <limit effort="${gripper_effort}" lower="${-10*d2r}" upper="${PI*0.3333}" velocity="0.1"/>
     </joint>
     <xacro:simple_transmission joint="${namespace}/finger_left_joint" />
@@ -134,6 +135,7 @@
         <origin xyz="0.23387 0.02401 -0.017121" rpy="0 0 ${15*d2r}"/>
         <axis xyz="0 0 1"/>
-        <dynamics damping="5" friction="10"/>
-        <limit effort="${gripper_effort}" lower="0" upper="${PI*0.3333}" velocity="${gripper_velocity}"/>
+        <dynamics damping="2" />
+        <!-- <dynamics damping="5" friction="5"/> -->
+        <limit effort="${gripper_effort}" lower="${-10*d2r}" upper="${PI*0.3333}" velocity="0.1"/>
     </joint>
     <xacro:simple_transmission joint="${namespace}/finger_right_joint" />

Commit message: Clean mesh names

File: dave_manipulator/predator_description/urdf/parallel_gripper_predator.xacro (robot description, xacro)
@@ -24,5 +24,5 @@
             <origin xyz="0 0 0" rpy="${PI*0.5} 0 ${-PI*0.5}"/>
             <geometry>
-                <mesh filename="file://$(find predator_description)/meshes/Predator-hand_centralized.dae"/>
+                <mesh filename="file://$(find predator_description)/meshes/hand.dae"/>
             </geometry>
         </visual>
@@ -34,5 +34,5 @@
             <origin xyz="0 0 0" rpy="${PI*0.5} 0 ${-PI*0.5}"/>
             <geometry>
-                <mesh filename="file://$(find predator_description)/meshes/Predator-hand_centralized.dae"/>
+                <mesh filename="file://$(find predator_description)/meshes/hand.dae"/>
             </geometry>
         </collision>
@@ -59,5 +59,5 @@
             <origin xyz="0 0 0" rpy="${PI*0.5} 0 ${-PI*0.5}"/>
             <geometry>
-                <mesh filename="file://$(find predator_description)/meshes/Predator-claw-right_centralized.dae"/>
+                <mesh filename="file://$(find predator_description)/meshes/claw_right.dae"/>
             </geometry>
         </visual>
@@ -65,5 +65,5 @@
             <origin xyz="0 0 0" rpy="${PI*0.5} 0 ${-PI*0.5}"/>
             <geometry>
-                <mesh filename="file://$(find predator_description)/meshes/Predator-claw-right_centralized.dae"/>
+                <mesh filename="file://$(find predator_description)/meshes/claw_right.dae"/>
             </geometry>
         </collision>
@@ -90,5 +90,5 @@
             <origin xyz="0 0 0" rpy="${PI/2}  0  ${-PI/2}"/>
             <geometry>
-                <mesh filename="file://$(find predator_description)/meshes/Predator-tip-right_centralized.dae"/>
+                <mesh filename="file://$(find predator_description)/meshes/tip_right.dae"/>
             </geometry>
         </visual>
@@ -96,5 +96,5 @@
             <origin xyz="0 0 0" rpy="${PI/2}  0  ${-PI/2}"/>
             <geometry>
-                <mesh filename="file://$(find predator_description)/meshes/Predator-tip-right_centralized.dae"/>
+                <mesh filename="file://$(find predator_description)/meshes/tip_right.dae"/>
             </geometry>
         </collision>
@@ -119,5 +119,5 @@
             <origin xyz="0 0 0" rpy="${PI/2} 0 ${-PI/2}"/>
             <geometry>
-                <mesh filename="file://$(find predator_description)/meshes/Predator-claw-left_centralized.dae"/>
+                <mesh filename="file://$(find predator_description)/meshes/claw_left.dae"/>
             </geometry>
         </visual>
@@ -125,5 +125,5 @@
             <origin xyz="0 0 0" rpy="${PI/2} 0 ${-PI/2}"/>
             <geometry>
-                <mesh filename="file://$(find predator_description)/meshes/Predator-claw-left_centralized.dae"/>
+                <mesh filename="file://$(find predator_description)/meshes/claw_left.dae"/>
             </geometry>
         </collision>
@@ -151,5 +151,5 @@
             <origin xyz="0 0 0" rpy="${PI/2} 0 ${-PI/2}"/>
             <geometry>
-                <mesh filename="file://$(find predator_description)/meshes/Predator-tip-left_centralized.dae"/>
+                <mesh filename="file://$(find predator_description)/meshes/tip_left.dae"/>
             </geometry>
         </visual>
@@ -157,5 +157,5 @@
             <origin xyz="0 0 0" rpy="${PI/2} 0 ${-PI/2}"/>
             <geometry>
-                <mesh filename="file://$(find predator_description)/meshes/Predator-tip-left_centralized.dae"/>
+                <mesh filename="file://$(find predator_description)/meshes/tip_left.dae"/>
             </geometry>
         </collision>

File: dave_manipulator/predator_description/urdf/serial_arm_predator.xacro (robot description, xacro)
@@ -53,5 +53,5 @@
                 <origin xyz="0 0 0" rpy="0 0 0"/>
                 <geometry>
-                    <mesh filename="file://$(find predator_description)/meshes/Predator-root_centralized.dae"/>
+                    <mesh filename="file://$(find predator_description)/meshes/base.dae"/>
                 </geometry>
             </visual>
@@ -59,5 +59,5 @@
                 <origin xyz="0 0 0" rpy="0 0 0"/>
                 <geometry>
-                    <mesh filename="file://$(find predator_description)/meshes/Predator-root_centralized.dae"/>
+                    <mesh filename="file://$(find predator_description)/meshes/base.dae"/>
                 </geometry>
             </collision>
@@ -74,5 +74,5 @@
                 <origin xyz="0 0 0" rpy="0 0 1.57079632679"/>
                 <geometry>
-                    <mesh filename="file://$(find predator_description)/meshes/Predator-base_centralized.dae"/>
+                    <mesh filename="file://$(find predator_description)/meshes/shoulder.dae"/>
                 </geometry>
             </visual>
@@ -80,5 +80,5 @@
                 <origin xyz="0 0 0" rpy="0 0 1.57079632679"/>
                 <geometry>
-                    <mesh filename="file://$(find predator_description)/meshes/Predator-base_centralized.dae"/>
+                    <mesh filename="file://$(find predator_description)/meshes/shoulder.dae"/>
                 </geometry>
             </collision>
@@ -105,5 +105,5 @@
                 <origin xyz="0 0 0" rpy="0 ${0.5*pi} 0"/>
                 <geometry>
-                    <mesh filename="file://$(find predator_description)/meshes/Predator-upperarm_centralized.dae"/>
+                    <mesh filename="file://$(find predator_description)/meshes/upperarm.dae"/>
                 </geometry>
             </visual>
@@ -111,5 +111,5 @@
                 <origin xyz="0 0 0" rpy="0 ${0.5*pi} 0"/>
                 <geometry>
-                    <mesh filename="file://$(find predator_description)/meshes/Predator-upperarm_centralized.dae"/>
+                    <mesh filename="file://$(find predator_description)/meshes/upperarm.dae"/>
                 </geometry>
             </collision>
@@ -137,5 +137,5 @@
                 <origin xyz="0 0 0" rpy="0 ${0.5*pi} ${0.5*pi}"/>
                 <geometry>
-                    <mesh filename="file://$(find predator_description)/meshes/Predator-forearm_centralized.dae"/>
+                    <mesh filename="file://$(find predator_description)/meshes/forearm.dae"/>
                 </geometry>
             </visual>
@@ -143,5 +143,5 @@
                 <origin xyz="0 0 0" rpy="0 ${0.5*pi} ${0.5*pi}"/>
                 <geometry>
-                    <mesh filename="file://$(find predator_description)/meshes/Predator-forearm_centralized.dae"/>
+                    <mesh filename="file://$(find predator_description)/meshes/forearm.dae"/>
                 </geometry>
             </collision>
@@ -168,5 +168,5 @@
                 <origin xyz="0 0 0" rpy="1.57079632679 1.57079632679 -1.57079632679"/>
                 <geometry>
-                    <mesh filename="file://$(find predator_description)/meshes/Predator-knuckle_centralized.dae"/>
+                    <mesh filename="file://$(find predator_description)/meshes/knuckle.dae"/>
                 </geometry>
             </visual>
@@ -174,5 +174,5 @@
                 <origin xyz="0 0 0" rpy="1.57079632679 1.57079632679 -1.57079632679"/>
                 <geometry>
-                    <mesh filename="file://$(find predator_description)/meshes/Predator-knuckle_centralized.dae"/>
+                    <mesh filename="file://$(find predator_description)/meshes/knuckle.dae"/>
                 </geometry>
             </collision>

Commit message: Rename links and joints

File: dave_manipulator/predator_description/urdf/parallel_gripper_predator.xacro (robot description, xacro)
@@ -39,5 +39,5 @@
     </link>
     <joint name="${namespace}/wrist" type="revolute">
-      <parent link="${namespace}/forearm"/>
+      <parent link="${namespace}/wrist"/>
       <child link="${namespace}/end_effector"/>
        <origin xyz="0.12137 -0.00038 0" rpy="${PI*0.5} 0 0"/>

File: dave_manipulator/predator_description/urdf/serial_arm.gazebo.xacro (robot description, xacro)
@@ -89,6 +89,5 @@
     <xacro:joint_ft_sensor joint_name="shoulder" namespace="${namespace}"/>
     <xacro:joint_ft_sensor joint_name="elbow" namespace="${namespace}"/>
-    <xacro:joint_ft_sensor joint_name="roll" namespace="${namespace}"/>
-    <!-- <xacro:joint_ft_sensor joint_name="pitch" namespace="${namespace}"/> -->
+    <xacro:joint_ft_sensor joint_name="pitch" namespace="${namespace}"/>
   </xacro:macro>
   <!--

File: dave_manipulator/predator_description/urdf/serial_arm_predator.xacro (robot description, xacro)
@@ -120,12 +120,10 @@
             <origin xyz="0.200369 0 0.209467" rpy="${0.5*pi} 0 0"/>
             <axis xyz="0 0 1"/>
-            <!-- <dynamics damping="50" friction="200"/> -->
             <dynamics damping="50" friction="150"/>
             <limit lower="${-90 * d2r}" upper="${90 * d2r}" velocity=".17" effort="5000"/>
-            <!-- <limit lower="${-90 * d2r}" upper="${90 * d2r}" velocity=".17" effort="1000"/> -->
         </joint>
         <xacro:simple_transmission joint="${namespace}/shoulder" />
-        <!-- ELBOW LINK -->
-        <link name="${namespace}/elbow_link">
+        <!-- FOREARM -->
+        <link name="${namespace}/forearm">
             <xacro:link_box_inertial mass="${total_mass * elbow_link_volume / total_volume_bbox}"
                         width="${elbow_link_width}"
@@ -149,7 +147,6 @@
         <joint name="${namespace}/elbow" type="revolute">
             <parent link="${namespace}/upper_arm"/>
-            <child link="${namespace}/elbow_link"/>
+            <child link="${namespace}/forearm"/>
             <origin xyz="0.87315 0 0" rpy="0 0 0"/>
-            <!-- <dynamics damping="50" friction="200"/> -->
             <dynamics damping="50" friction="150"/>
             <axis xyz="0 0 1"/>
@@ -157,6 +154,6 @@
         </joint>
         <xacro:simple_transmission joint="${namespace}/elbow" />
-        <!-- FOREARM -->
-        <link name="${namespace}/forearm">
+        <!-- WRIST -->
+        <link name="${namespace}/wrist">
             <xacro:link_box_inertial mass="${total_mass * forearm_volume / total_volume_bbox}"
                         width="${forearm_width}"
@@ -178,7 +175,7 @@
             </collision>
         </link>
-        <joint name="${namespace}/roll" type="revolute">
-            <parent link="${namespace}/elbow_link"/>
-            <child link="${namespace}/forearm"/>
+        <joint name="${namespace}/pitch" type="revolute">
+            <parent link="${namespace}/forearm"/>
+            <child link="${namespace}/wrist"/>
             <origin xyz="0.11275 -0.55503 0" rpy="0 0 -1.57079632679"/>
             <axis xyz="0 0 1"/>
@@ -186,5 +183,5 @@
             <limit lower="${-135 * d2r}" upper="${135 * d2r}" velocity=".25" effort="1000"/>
         </joint>
-        <xacro:simple_transmission joint="${namespace}/roll" />
+        <xacro:simple_transmission joint="${namespace}/pitch" />
         <!-- Adding parallel gripper  -->
         <xacro:include filename="$(find predator_description)/urdf/parallel_gripper_predator.xacro" />
