Commit message: Changed joint name _wrist_ to _wrist_joint_

File: dave_manipulator/predator_description/urdf/parallel_gripper_predator.xacro (robot description, xacro)
@@ -38,5 +38,5 @@
         </collision>
     </link>
-    <joint name="${namespace}/wrist" type="revolute">
+    <joint name="${namespace}/wrist_joint" type="revolute">
       <parent link="${namespace}/wrist"/>
       <child link="${namespace}/end_effector"/>
@@ -46,5 +46,5 @@
       <limit effort="10" lower="${-2*PI}" upper="${2*PI}" velocity="${gripper_velocity}"/>
     </joint>
-    <xacro:simple_transmission joint="${namespace}/wrist" />
+    <xacro:simple_transmission joint="${namespace}/wrist_joint" />
     <!-- Finger left  -->
     <link name="${namespace}/finger_left">

File: dave_manipulator/predator_description/urdf/serial_arm.gazebo.xacro (robot description, xacro)
@@ -80,5 +80,5 @@
     </gazebo>
     <!-- Gripper FT sensors -->
-    <xacro:joint_ft_sensor joint_name="wrist" namespace="${namespace}"/>
+    <xacro:joint_ft_sensor joint_name="wrist_joint" namespace="${namespace}"/>
     <xacro:joint_ft_sensor joint_name="finger_left_joint" namespace="${namespace}"/>
     <xacro:joint_ft_sensor joint_name="finger_tip_left_joint" namespace="${namespace}"/>

File: uuv_dave/urdf/serial_arm.gazebo.xacro (robot description, xacro)
@@ -80,5 +80,5 @@
     </gazebo>
     <!-- Gripper FT sensors -->
-    <xacro:joint_ft_sensor joint_name="wrist" namespace="${namespace}"/>
+    <xacro:joint_ft_sensor joint_name="wrist_joint" namespace="${namespace}"/>
     <xacro:joint_ft_sensor joint_name="finger_left_joint" namespace="${namespace}"/>
     <xacro:joint_ft_sensor joint_name="finger_tip_left_joint" namespace="${namespace}"/>
