Commit message: Created "description" packages for all of the WHOI DSL DVL Xacro examples
All sensor description packages are in the urdf/sensors subdirectory as
follows (the "_dsl" portion of the package name differentiates the examples
that use the WHOI DSL plugin from those using the UUV Simulator plugin):

nortek_dvl500_300_uuvsim_description
nortek_dvl500_6000_uuvsim_description
nortek_dvl1000_300_uuvsim_description
nortek_dvl1000_4000_uuvsim_description
sonardyne_syrinx600_uuvsim_description
teledyne_explorer1000_uuvsim_description
teledyne_explorer4000_uuvsim_description
teledyne_whn_uuvsim_description

File: urdf/sensors/nortek_dvl1000_300_dsl_description/urdf/nortek_dvl1000_300.xacro (robot description, xacro)
@@ -44,5 +44,4 @@
       <visual>
         <geometry>
-<!--          <mesh filename="$(find nps_uw_sensors_gazebo)/models/whoi_nortek_dvl1000_300/meshes/DVL1000-300m.dae"/> -->
           <mesh filename="package://nortek_dvl1000_300_dsl_description/meshes/DVL1000-300m.dae"/>
         </geometry>
