Commit message: Fix naming convention (cannot start with num)

File: urdf/robots/rexrov_description/urdf/rexrov_oberon7_sl3.xacro (robot description, xacro)
@@ -20,5 +20,5 @@
   <xacro:include filename="$(find uuv_descriptions)/urdf/rexrov.gazebo.xacro"/>
   <xacro:include filename="$(find dave_oberon7_description)/urdf/oberon7_default.xacro" />
-  <xacro:include filename="$(find 3dad_sl3_description)/urdf/sl3_lidar.xacro"/>
+  <xacro:include filename="$(find lidar_3dad_sl3_description)/urdf/sl3_lidar.xacro"/>
   <xacro:uuv_forward_looking_sonar
       namespace="${namespace}"

File: urdf/sensors/lindar_3dad_sl3_description/urdf/sl3_lidar.xacro (robot description, xacro)
@@ -125,5 +125,5 @@
       <visual>
         <geometry>
-          <mesh filename="package://3dad_sl3_description/meshes/3dad_sl3.dae"/>
+          <mesh filename="package://lidar_3dad_sl3_description/meshes/3dad_sl3.dae"/>
         </geometry>
         <origin xyz="0 0 0.163" rpy="0 0 0"/>
@@ -144,5 +144,5 @@
       <visual>
         <geometry>
-          <mesh filename="package://3dad_sl3_description/meshes/sl3_lidar_mount_tray.dae"/>
+          <mesh filename="package://lidar_3dad_sl3_description/meshes/sl3_lidar_mount_tray.dae"/>
         </geometry>
         <origin xyz="0 0.034 0.163" rpy="0 0 0"/>
@@ -163,5 +163,5 @@
       <visual>
         <geometry>
-          <mesh filename="package://3dad_sl3_description/meshes/sl3_lidar_mount_swivel.dae"/>
+          <mesh filename="package://lidar_3dad_sl3_description/meshes/sl3_lidar_mount_swivel.dae"/>
         </geometry>
         <origin xyz="0 0.034 0.255" rpy="0 0 0"/>
@@ -182,5 +182,5 @@
       <visual>
         <geometry>
-          <mesh filename="package://3dad_sl3_description/meshes/sl3_lidar_mount_base.dae"/>
+          <mesh filename="package://lidar_3dad_sl3_description/meshes/sl3_lidar_mount_base.dae"/>
         </geometry>
         <origin xyz="0 0.034 0.375" rpy="0 0 0"/>
