Commit message: first version working with craftsman

File: urdf/robots/rexrov_description/urdf/rexrov_base.xacro (robot description, xacro)
@@ -26,5 +26,5 @@
   <xacro:include filename="$(find uuv_gazebo_ros_plugins)/urdf/snippets.xacro"/>
   <!-- Parameters -->
-  <xacro:property name="namespace" value="rexrov"/>
+  <xacro:property name="namespace" value="rexrov/rexrov"/>
   <xacro:property name="visual_mesh_file" value="file://$(find uuv_descriptions)/meshes/RexROV_no_props.dae"/>
   <xacro:property name="prop_mesh_file" value="file://$(find uuv_descriptions)/meshes/prop.dae"/>
