Commit message: Added args for effort or position controller in dave_oberon_moveit that changes urdf transmission values

File: urdf/robots/rexrov_description/urdf/rexrov_robot.urdf.xacro (robot description, xacro)
@@ -5,4 +5,5 @@
 	<xacro:arg name="debug" default="false"/>
 	<xacro:arg name="controller_type" default="effort"/>
+	<xacro:property name="controller" value="$(arg controller_type)"/>
 	<xacro:include filename="$(find rexrov_description)/urdf/rexrov_base.xacro"/>
 	<xacro:include filename="$(find uuv_descriptions)/urdf/rexrov.gazebo.xacro"/>
@@ -26,10 +27,10 @@
   	</xacro:rexrov_base>
 	<!-- oberon7 -->
-	<!-- <xacro:if value="${controller_type == 'effort'}">	 -->
-		<!-- <xacro:arg name="transmission_hw_interface" default="hardware_interface/PositionJointInterface"/> -->
-	<!-- </xacro:if> -->
-	<!-- <xacro:if value="${controller_type == 'position'}"> -->
+	<xacro:if value="${controller == 'position'}">
+		<xacro:arg name="transmission_hw_interface" default="hardware_interface/PositionJointInterface"/>
+	</xacro:if>
+	<xacro:if value="${controller == 'effort'}">
 		<xacro:arg name="transmission_hw_interface" default="hardware_interface/EffortJointInterface"/>
-	<!-- </xacro:if> -->
+	</xacro:if>
 	<xacro:oberon7_arm transmission_hw_interface="$(arg transmission_hw_interface)" namespace="oberon7_r"/>
 	<xacro:oberon7_arm transmission_hw_interface="$(arg transmission_hw_interface)" namespace="oberon7_l"/>

Commit message: Bimanual manipulation update (#241)
* Added hydro model namespaces for both oberon7 arms

* Removed joint_group_position controller from launch

* Condense controllers code for dave_oberon7_moveit example, update hydro model namespace

* Choose effort or position controller argument passed

* Added args for effort or position controller in dave_oberon_moveit that changes urdf transmission values

* Modified launch permissions, added bimanual example world, added position arguments

* Adjusted camera angle for example world

* Modified rov position, added bimanual example world

* Added distorted vase to bimanual demo world

* Modified launch file to accept single controller type rather than two explicit controller args

File: urdf/robots/rexrov_description/urdf/rexrov_robot.urdf.xacro (robot description, xacro)
@@ -4,9 +4,9 @@
 	<xacro:arg name="inertial_reference_frame" default="world"/>
 	<xacro:arg name="debug" default="false"/>
+	<xacro:arg name="controller_type" default="effort"/>
+	<xacro:property name="controller" value="$(arg controller_type)"/>
 	<xacro:include filename="$(find rexrov_description)/urdf/rexrov_base.xacro"/>
 	<xacro:include filename="$(find uuv_descriptions)/urdf/rexrov.gazebo.xacro"/>
-	<!-- <xacro:include filename="$(find dave_oberon7_description)/urdf/serial_arm.gazebo.xacro"/> -->
-	<!-- <xacro:include filename="$(find oberon7_description)/urdf/parameters/serial_arm.xacro"/> -->
-	<!-- <xacro:include filename="$(find dave_oberon7_description)/urdf/oberon7_default.xacro"/> -->
+	<xacro:include filename="$(find dave_oberon7_description)/urdf/oberon7_default.xacro"/>
 	<xacro:include filename="$(find oberon7_description)/urdf/common.gazebo.xacro"/>
 	<xacro:include filename="$(find oberon7_description)/urdf/oberon7.urdf.xacro"/>
@@ -21,12 +21,16 @@
 		    <!-- Adding the hydrodynamic and hydrostatic parameters for the vehicle-->
 		    <xacro:rexrov_hydro_model namespace="$(arg namespace)"/>
-		    <!-- <xacro:oberon7_hydro_model namespace="oberon7"/> -->
+		    <xacro:oberon7_hydro_model namespace="oberon7_r"/>
+		    <xacro:oberon7_hydro_model namespace="oberon7_l"/>
       	</plugin>
     </gazebo>
   	</xacro:rexrov_base>
-<!-- oberon7 -->
-	<xacro:arg name="transmission_hw_interface" default="hardware_interface/PositionJointInterface"/>
-	<!-- <xacro:include filename="$(find oberon7_description)/urdf/common.gazebo.xacro"/> -->
-	<!-- <xacro:include filename="$(find oberon7_description)/urdf/oberon7.urdf.xacro"/> -->
+	<!-- oberon7 -->
+	<xacro:if value="${controller == 'position'}">
+		<xacro:arg name="transmission_hw_interface" default="hardware_interface/PositionJointInterface"/>
+	</xacro:if>
+	<xacro:if value="${controller == 'effort'}">
+		<xacro:arg name="transmission_hw_interface" default="hardware_interface/EffortJointInterface"/>
+	</xacro:if>
 	<xacro:oberon7_arm transmission_hw_interface="$(arg transmission_hw_interface)" namespace="oberon7_r"/>
 	<xacro:oberon7_arm transmission_hw_interface="$(arg transmission_hw_interface)" namespace="oberon7_l"/>
