Commit message: Eliminated "deprecated" warnings with oberon7 and predator xacro
Added the 'hardware_interface/' preface to the EffortJointInterface
contents of the hardwareInterface elements of the transmission macro.

NOTE: This was already in both .xacro files but commented out, so this
change just comments out the previous macro and uncomments this one.
If the original commenting was there for a reason, this change can
be undone (previous commenting for Gazebo 8?)

File: urdf/manipulators/dave_oberon7_description/urdf/serial_arm.xacro (robot description, xacro)
@@ -16,5 +16,5 @@
     <xacro:include filename="$(find oberon7_description)/urdf/parameters/serial_arm.xacro" />
     <!-- Transmission Macro -->
-    <!-- <xacro:macro name="simple_transmission" params="joint">
+    <xacro:macro name="simple_transmission" params="joint">
         <transmission name="${joint}_trans">
             <type>transmission_interface/SimpleTransmission</type>
@@ -27,7 +27,7 @@
             </actuator>
         </transmission>
-    </xacro:macro> -->
+    </xacro:macro>
     <!-- Transmission Macro -->
-    <xacro:macro name="simple_transmission" params="joint">
+    <!-- <xacro:macro name="simple_transmission" params="joint">
       <transmission name="${joint}_trans">
         <type>transmission_interface/SimpleTransmission</type>
@@ -40,5 +40,5 @@
         </actuator>
       </transmission>
-    </xacro:macro>
+    </xacro:macro> -->
     <xacro:macro name="oberon7_serial_arm" params="namespace">
         <!-- Ground base -->

File: urdf/manipulators/predator_description/urdf/serial_arm_predator.xacro (robot description, xacro)
@@ -16,5 +16,5 @@
     <xacro:include filename="$(find predator_description)/urdf/parameters/serial_arm_predator.xacro" />
     <!-- Transmission Macro -->
-    <!-- <xacro:macro name="simple_transmission" params="joint">
+    <xacro:macro name="simple_transmission" params="joint">
         <transmission name="${joint}_trans">
             <type>transmission_interface/SimpleTransmission</type>
@@ -27,7 +27,7 @@
             </actuator>
         </transmission>
-    </xacro:macro> -->
+    </xacro:macro>
     <!-- Transmission Macro -->
-    <xacro:macro name="simple_transmission" params="joint">
+    <!-- <xacro:macro name="simple_transmission" params="joint">
       <transmission name="${joint}_trans">
         <type>transmission_interface/SimpleTransmission</type>
@@ -40,5 +40,5 @@
         </actuator>
       </transmission>
-    </xacro:macro>
+    </xacro:macro> -->
     <xacro:macro name="predator_serial_arm" params="namespace">
         <!-- Ground base -->
