Commit message: Update serial arm parameters
Signed-off-by: Yadunund <yadunund@gmail.com>

File: urdf/manipulators/dave_oberon7_description/urdf/oberon7_default.xacro (robot description, xacro)
@@ -13,6 +13,8 @@
 -->
 <robot name="oberon7" xmlns:xacro="http://www.ros.org/wiki/xacro">
+  <!-- Parameters -->
+  <xacro:property name="namespace" value="rexrov"/>
   <!-- Import serial arm -->
-  <xacro:include filename="$(find dave_oberon7_description)/urdf/serial_arm.xacro" />
+  <xacro:include filename="$(find dave_oberon7_description)/urdf/serial_arm.xacro" joint="${namespace}/anchor"/>
   <!-- Import Gazebo specific macros -->
   <xacro:include filename="$(find dave_oberon7_description)/urdf/serial_arm.gazebo.xacro" />

File: urdf/manipulators/dave_oberon7_description/urdf/serial_arm.xacro (robot description, xacro)
@@ -15,4 +15,6 @@
     <!-- Import arm parameters -->
     <xacro:include filename="$(find oberon7_description)/urdf/parameters/serial_arm.xacro" />
+    <!-- Parameters -->
+    <xacro:property name="joint" value="rexrov/anchor"/>
     <!-- Transmission Macro -->
     <xacro:macro name="simple_transmission" params="joint">
