Commit message: Simplified the alignment checks in the plug_and_socket plugin
Alignment check now compares the pose of the socket and plug links
more directly in a single function.  Alignment is checked in 3 steps:
  Orientation: plug & socket link frame orientations match
  Lateral: plug position is along the socket link X axis
  Distance: plug is within 0.5 meters of the socket link

If all three checks pass, the proximity check (which is unchanged)
is used to determine when to create the prismatic joint.

File: urdf/manipulators/plug_and_socket_description/urdf/socket.xacro (robot description, xacro)
@@ -3,5 +3,5 @@
   <xacro:macro name="socket_macro"
                params="name xyz plug_model_name plug_link_name
-                       roll_tolerance pitch_tolerance yaw_tolerance z_tolerance
+                       roll_tolerance pitch_tolerance yaw_tolerance
                        mating_force unmating_force">
     <!-- Socket tube link -->
@@ -55,8 +55,7 @@
         <plugModel>${plug_model_name}</plugModel>
         <plugLink>${plug_link_name}</plugLink>
-        <rollAlignmentTolerence>${roll_tolerance}</rollAlignmentTolerence>
-        <pitchAlignmentTolerence>${pitch_tolerance}</pitchAlignmentTolerence>
-        <yawAlignmentTolerence>${yaw_tolerance}</yawAlignmentTolerence>
-        <zAlignmentTolerence>${z_tolerance}</zAlignmentTolerence>
+        <rollAlignmentTolerance>${roll_tolerance}</rollAlignmentTolerance>
+        <pitchAlignmentTolerance>${pitch_tolerance}</pitchAlignmentTolerance>
+        <yawAlignmentTolerance>${yaw_tolerance}</yawAlignmentTolerance>
         <matingForce>${mating_force}</matingForce>
         <unmatingForce>${unmating_force}</unmatingForce>

File: urdf/manipulators/plug_and_socket_description/urdf/socket_platform.xacro (robot description, xacro)
@@ -28,6 +28,6 @@
     name="socket1" xyz="0 0 0"
     plug_model_name="plug" plug_link_name="plug" roll_tolerance="0.3"
-    pitch_tolerance="0.3" yaw_tolerance="0.3" z_tolerance="0.5"
-    mating_force="50" unmating_force="190"/>
+    pitch_tolerance="0.3" yaw_tolerance="0.3"
+    mating_force="50" unmating_force="125"/>
   <!-- Revolute joint gets accurately loaded into Gazebo -->
   <joint name="socket1_joint" type="revolute">
@@ -36,10 +36,10 @@
     <parent link="socket_platform_link"/>
     <child link="socket1_link"/>
-  </joint> -->
+  </joint>
   <xacro:socket_macro
     name="socket2" xyz="0 0 0"
     plug_model_name="plug" plug_link_name="plug" roll_tolerance="0.3"
-    pitch_tolerance="0.3" yaw_tolerance="0.3" z_tolerance="0.5"
-    mating_force="50" unmating_force="190"/>
+    pitch_tolerance="0.3" yaw_tolerance="0.3"
+    mating_force="50" unmating_force="125"/>
   <joint name="socket2_joint" type="revolute">
     <limit effort="1.0" lower="0.0" upper="0.0" velocity="0.0"/>
@@ -51,6 +51,6 @@
     name="socket3" xyz="0 0 0"
     plug_model_name="plug" plug_link_name="plug" roll_tolerance="0.3"
-    pitch_tolerance="0.3" yaw_tolerance="0.3" z_tolerance="0.5"
-    mating_force="50" unmating_force="190"/>
+    pitch_tolerance="0.3" yaw_tolerance="0.3"
+    mating_force="50" unmating_force="125"/>
   <joint name="socket3_joint" type="revolute">
     <limit effort="1.0" lower="0.0" upper="0.0" velocity="0.0"/>
@@ -62,6 +62,6 @@
     name="socket4" xyz="0 0 0"
     plug_model_name="plug" plug_link_name="plug" roll_tolerance="0.3"
-    pitch_tolerance="0.3" yaw_tolerance="0.3" z_tolerance="0.5"
-    mating_force="50" unmating_force="190"/>
+    pitch_tolerance="0.3" yaw_tolerance="0.3"
+    mating_force="50" unmating_force="125"/>
   <joint name="socket4_joint" type="revolute">
     <limit effort="1.0" lower="0.0" upper="0.0" velocity="0.0"/>
@@ -73,6 +73,6 @@
     name="socket5" xyz="0 0 0"
     plug_model_name="plug" plug_link_name="plug" roll_tolerance="${pi}"
-    pitch_tolerance="0.3" yaw_tolerance="0.3" z_tolerance="0.5"
-    mating_force="50" unmating_force="190"/>
+    pitch_tolerance="0.3" yaw_tolerance="0.3"
+    mating_force="50" unmating_force="125"/>
   <joint name="socket5_joint" type="revolute">
     <limit effort="1.0" lower="0.0" upper="0.0" velocity="0.0"/>

Commit message: Deleted duplicated meshes from URDF directories
Updated description packages for the DVLs and plug and socket to use the
meshes from the SDF models instead of duplicating them (DVL models are
in the dave_sensor_models package, and the plug and socket models are in
the dave_object_models package).

File: urdf/manipulators/plug_and_socket_description/urdf/socket.xacro (robot description, xacro)
@@ -15,5 +15,5 @@
       <visual>
         <geometry>
-          <mesh filename="package://plug_and_socket_description/meshes/Electrical-Socket.dae" scale="0.12 0.12 0.12"/>
+          <mesh filename="package://dave_object_models/models/socket/meshes/Electrical-Socket.dae" scale="0.12 0.12 0.12"/>
         </geometry>
         <origin xyz="0 0 0" rpy="0 0 ${-pi/2}"/>
@@ -21,5 +21,5 @@
       <collision>
         <geometry>
-          <mesh filename="package://plug_and_socket_description/meshes/Electrical-Socket.dae" scale="0.12 0.12 0.12"/>
+          <mesh filename="package://dave_object_models/models/socket/meshes/Electrical-Socket.dae" scale="0.12 0.12 0.12"/>
         </geometry>
         <origin xyz="0 0 0" rpy="0 0 ${-pi/2}"/>

File: urdf/sensors/nortek_dvl1000_300_dsl_description/urdf/nortek_dvl1000_300.xacro (robot description, xacro)
@@ -44,5 +44,5 @@
       <visual>
         <geometry>
-          <mesh filename="package://nortek_dvl1000_300_dsl_description/meshes/DVL1000-300m.dae"/>
+          <mesh filename="package://dave_sensor_models/models/nortek_dvl1000_300/meshes/DVL1000-300m.dae"/>
         </geometry>
         <origin xyz="${xyz}" rpy="0 ${pi} 0"/>

File: urdf/sensors/nortek_dvl1000_300_uuvsim_description/urdf/nortek_dvl1000_300.xacro (robot description, xacro)
@@ -126,5 +126,5 @@
       <visual>
         <geometry>
-          <mesh filename="package://nortek_dvl1000_300_uuvsim_description/meshes/DVL1000-300m.dae"/>
+          <mesh filename="package://dave_sensor_models/models/nortek_dvl1000_300/meshes/DVL1000-300m.dae"/>
         </geometry>
         <origin xyz="0 0 0" rpy="0 -1.5707963267948966 0"/>

File: urdf/sensors/nortek_dvl1000_4000_dsl_description/urdf/nortek_dvl1000_4000.xacro (robot description, xacro)
@@ -44,5 +44,5 @@
       <visual>
         <geometry>
-          <mesh filename="package://nortek_dvl1000_4000_dsl_description/meshes/DVL1000-4000m.dae"/>
+          <mesh filename="package://dave_sensor_models/models/nortek_dvl1000_4000/meshes/DVL1000-4000m.dae"/>
         </geometry>
         <origin xyz="${xyz}" rpy="0 ${pi} 0"/>

File: urdf/sensors/nortek_dvl1000_4000_uuvsim_description/urdf/nortek_dvl1000_4000.xacro (robot description, xacro)
@@ -126,5 +126,5 @@
       <visual>
         <geometry>
-          <mesh filename="package://nortek_dvl1000_4000_uuvsim_description/meshes/DVL1000-4000m.dae"/>
+          <mesh filename="package://dave_sensor_models/models/nortek_dvl1000_4000/meshes/DVL1000-4000m.dae"/>
         </geometry>
         <origin xyz="0 0 0" rpy="0 -1.5707963267948966 0"/>

File: urdf/sensors/nortek_dvl500_300_dsl_description/urdf/nortek_dvl500_300.xacro (robot description, xacro)
@@ -44,6 +44,5 @@
       <visual>
         <geometry>
-          <!-- Replace mesh with correct one once it's available -->
-          <mesh filename="package://nortek_dvl500_300_dsl_description/meshes/DVL500-300m.dae"/>
+          <mesh filename="package://dave_sensor_models/models/nortek_dvl500_300/meshes/DVL500-300m.dae"/>
         </geometry>
         <origin xyz="${xyz}" rpy="0 ${pi} 0"/>

File: urdf/sensors/nortek_dvl500_300_uuvsim_description/urdf/nortek_dvl500_300.xacro (robot description, xacro)
@@ -126,6 +126,5 @@
       <visual>
         <geometry>
-          <!-- Replace with Nortek DVL500 mesh when available -->
-          <mesh filename="package://nortek_dvl500_300_uuvsim_description/meshes/DVL500-300m.dae"/>
+          <mesh filename="package://dave_sensor_models/models/nortek_dvl500_300/meshes/DVL500-300m.dae"/>
         </geometry>
         <origin xyz="0 0 0" rpy="0 -1.5707963267948966 0"/>

File: urdf/sensors/nortek_dvl500_6000_dsl_description/urdf/nortek_dvl500_6000.xacro (robot description, xacro)
@@ -44,6 +44,5 @@
       <visual>
         <geometry>
-          <!-- Replace mesh with correct one once it's available -->
-          <mesh filename="package://nortek_dvl500_6000_dsl_description/meshes/DVL500-6000m.dae"/>
+          <mesh filename="package://dave_sensor_models/models/nortek_dvl500_6000/meshes/DVL500-6000m.dae"/>
         </geometry>
         <origin xyz="${xyz}" rpy="0 ${pi} 0"/>

File: urdf/sensors/nortek_dvl500_6000_uuvsim_description/urdf/nortek_dvl500_6000.xacro (robot description, xacro)
@@ -126,6 +126,5 @@
       <visual>
         <geometry>
-          <!-- Replace with Nortek DVL500 mesh when available -->
-          <mesh filename="package://nortek_dvl500_6000_uuvsim_description/meshes/DVL500-6000m.dae"/>
+          <mesh filename="package://dave_sensor_models/models/nortek_dvl500_6000/meshes/DVL500-6000m.dae"/>
         </geometry>
         <origin xyz="0 0 0" rpy="0 -1.5707963267948966 0"/>

File: urdf/sensors/sonardyne_syrinx600_dsl_description/urdf/sonardyne_syrinx600.xacro (robot description, xacro)
@@ -45,5 +45,5 @@
         <geometry>
           <!-- Replace mesh with correct one once it's available -->
-          <mesh filename="package://sonardyne_syrinx600_dsl_description/meshes/Syrinx600.dae"/>
+          <mesh filename="package://dave_sensor_models/models/sonardyne_syrinx600/meshes/Syrinx600.dae"/>
         </geometry>
         <origin xyz="${xyz}" rpy="0 ${pi} 0"/>

File: urdf/sensors/sonardyne_syrinx600_uuvsim_description/urdf/sonardyne_syrinx600.xacro (robot description, xacro)
@@ -127,5 +127,5 @@
         <geometry>
           <!-- Replace with Sonardyne Syrinx 600 mesh when available -->
-          <mesh filename="package://sonardyne_syrinx600_uuvsim_description/meshes/Syrinx600.dae"/>
+          <mesh filename="package://dave_sensor_models/models/sonardyne_syrinx600/meshes/Syrinx600.dae"/>
         </geometry>
         <origin xyz="0 0 0" rpy="0 -1.5707963 0"/>

File: urdf/sensors/teledyne_explorer1000_dsl_description/urdf/teledyne_explorer1000.xacro (robot description, xacro)
@@ -45,5 +45,5 @@
       <visual>
         <geometry>
-          <mesh filename="package://teledyne_explorer1000_dsl_description/meshes/MarineExplorer.dae"/>
+          <mesh filename="package://dave_sensor_models/models/teledyne_explorer1000/meshes/MarineExplorer.dae"/>
         </geometry>
         <origin xyz="${xyz}" rpy="${-0.5*pi} 0 ${-0.5*pi}"/>

File: urdf/sensors/teledyne_explorer1000_uuvsim_description/urdf/teledyne_explorer1000.xacro (robot description, xacro)
@@ -128,5 +128,5 @@
       <visual>
         <geometry>
-          <mesh filename="package://teledyne_explorer1000_uuvsim_description/meshes/MarineExplorer.dae"/>
+          <mesh filename="package://dave_sensor_models/models/teledyne_explorer1000/meshes/MarineExplorer.dae"/>
         </geometry>
         <origin xyz="0 0 0" rpy="0 0 1.5707963267948966"/>

File: urdf/sensors/teledyne_explorer4000_dsl_description/urdf/teledyne_explorer4000.xacro (robot description, xacro)
@@ -45,5 +45,5 @@
       <visual>
         <geometry>
-          <mesh filename="package://teledyne_explorer4000_dsl_description/meshes/MarineExplorer.dae"/>
+          <mesh filename="package://dave_sensor_models/models/teledyne_explorer4000/meshes/MarineExplorer.dae"/>
         </geometry>
         <origin xyz="${xyz}" rpy="${-0.5*pi} 0 ${-0.5*pi}"/>

File: urdf/sensors/teledyne_explorer4000_uuvsim_description/urdf/teledyne_explorer4000.xacro (robot description, xacro)
@@ -127,5 +127,5 @@
       <visual>
         <geometry>
-          <mesh filename="package://teledyne_explorer4000_uuvsim_description/meshes/MarineExplorer.dae"/>
+          <mesh filename="package://dave_sensor_models/models/teledyne_explorer4000/meshes/MarineExplorer.dae"/>
         </geometry>
         <origin xyz="0 0 0" rpy="0 0 1.5707963267948966"/>

File: urdf/sensors/teledyne_whn_dsl_description/urdf/teledyne_whn.xacro (robot description, xacro)
@@ -44,5 +44,5 @@
       <visual>
         <geometry>
-          <mesh filename="package://teledyne_whn_dsl_description/meshes/WorkhorseNavigator.dae"/>
+          <mesh filename="package://dave_sensor_models/models/teledyne_whn_dsl/meshes/WorkhorseNavigator.dae"/>
         </geometry>
         <origin xyz="${xyz}" rpy="0 0 0"/>

File: urdf/sensors/teledyne_whn_dsl_description/urdf/teledyne_whn_beams.xacro (robot description, xacro)
@@ -11,5 +11,5 @@
       <visual>
         <geometry>
-          <mesh filename="package://teledyne_whn_dsl_description/meshes/WorkhorseNavigator.dae" scale="${scale}"/>
+          <mesh filename="package://dave_sensor_models/models/teledyne_whn_dsl/meshes/WorkhorseNavigator.dae" scale="${scale}"/>
         </geometry>
         <origin xyz="${xyz}" rpy="0 0 0"/>

File: urdf/sensors/teledyne_whn_uuvsim_description/urdf/teledyne_whn.xacro (robot description, xacro)
@@ -126,5 +126,5 @@
       <visual>
         <geometry>
-          <mesh filename="package://teledyne_whn_uuvsim_description/meshes/WorkhorseNavigator.dae"/>
+          <mesh filename="package://dave_sensor_models/models/teledyne_whn_uuvsim/meshes/WorkhorseNavigator.dae"/>
         </geometry>
         <origin xyz="0 0 0" rpy="0 1.5707963267948966 0"/>
