Commit message: Plug & socket updates to work in various orientations
Updated alignment and joint functionality to work when the socket
is mounted to another model and not aligned with the world X axis
(previous version was using RelativePose when checking the alignment
of the plug and socket).

Also, changed the prismatic joint function to allow it to slide
more reliably before it is locked.

File: urdf/manipulators/plug_and_socket_description/urdf/socket_platform.xacro (robot description, xacro)
@@ -30,10 +30,11 @@
     pitch_tolerance="0.3" yaw_tolerance="0.3" z_tolerance="0.5"
     mating_force="50" unmating_force="190"/>
+  <!-- Revolute joint gets accurately loaded into Gazebo -->
   <joint name="socket1_joint" type="revolute">
     <limit effort="1.0" lower="0.0" upper="0.0" velocity="0.0"/>
-    <origin xyz="0.25 0.8 1.25" rpy="0 0 ${pi/2}"/>
+    <origin xyz="0 0.8 1" rpy="0 0 ${pi/2}"/>
     <parent link="socket_platform_link"/>
     <child link="socket1_link"/>
-  </joint>
+  </joint> -->
   <xacro:socket_macro
     name="socket2" xyz="0 0 0"
@@ -43,5 +44,5 @@
   <joint name="socket2_joint" type="revolute">
     <limit effort="1.0" lower="0.0" upper="0.0" velocity="0.0"/>
-    <origin xyz="0 0.8 1.25" rpy="0 0 ${pi/2}"/>
+    <origin xyz="0.8 0 1" rpy="0 0 0"/>
     <parent link="socket_platform_link"/>
     <child link="socket2_link"/>
@@ -54,5 +55,5 @@
   <joint name="socket3_joint" type="revolute">
     <limit effort="1.0" lower="0.0" upper="0.0" velocity="0.0"/>
-    <origin xyz="-0.25 0.8 1.25" rpy="0 0 ${pi/2}"/>
+    <origin xyz="0 -0.8 1" rpy="0 0 ${-pi/2}"/>
     <parent link="socket_platform_link"/>
     <child link="socket3_link"/>
@@ -65,5 +66,5 @@
   <joint name="socket4_joint" type="revolute">
     <limit effort="1.0" lower="0.0" upper="0.0" velocity="0.0"/>
-    <origin xyz="0.25 0.8 1" rpy="0 0 ${pi/2}"/>
+    <origin xyz="-0.8 0 1" rpy="0 0 ${pi}"/>
     <parent link="socket_platform_link"/>
     <child link="socket4_link"/>
@@ -71,23 +72,12 @@
   <xacro:socket_macro
     name="socket5" xyz="0 0 0"
-    plug_model_name="plug" plug_link_name="plug" roll_tolerance="0.3"
+    plug_model_name="plug" plug_link_name="plug" roll_tolerance="${pi/2}"
     pitch_tolerance="0.3" yaw_tolerance="0.3" z_tolerance="0.5"
     mating_force="50" unmating_force="190"/>
   <joint name="socket5_joint" type="revolute">
     <limit effort="1.0" lower="0.0" upper="0.0" velocity="0.0"/>
-    <origin xyz="0 0.8 1" rpy="0 0 ${pi/2}"/>
+    <origin xyz="0 0 1.55" rpy="0 -${pi/2} 0"/>
     <parent link="socket_platform_link"/>
     <child link="socket5_link"/>
   </joint>
-  <xacro:socket_macro
-    name="socket6" xyz="0 0 0"
-    plug_model_name="plug" plug_link_name="plug" roll_tolerance="0.3"
-    pitch_tolerance="0.3" yaw_tolerance="0.3" z_tolerance="0.5"
-    mating_force="50" unmating_force="190"/>
-  <joint name="socket6_joint" type="revolute">
-    <limit effort="1.0" lower="0.0" upper="0.0" velocity="0.0"/>
-    <origin xyz="-0.25 0.8 1" rpy="0 0 ${pi/2}"/>
-    <parent link="socket_platform_link"/>
-    <child link="socket6_link"/>
-  </joint>
 </robot>

Commit message: Model Update ISO new Electrical Lead Models
Electrical platform model added that uses new mesh
dave_demo_launch/dave_electrical_mate.launch and
dave_demo_launch/dave_plug_and_socket_demo.launch both
updated to use the new electrical platform.

Plug and socket model names were changed (m_to_f_plug & m_to_f_socket)
to differentiate them from the new plug and receptacle models
(the new models are female-plug-to-male receptacle) which will be
added shortly.

File: urdf/manipulators/plug_and_socket_description/urdf/socket_platform.xacro (robot description, xacro)
@@ -1,6 +1,5 @@
 <?xml version="1.0"?>
 <robot xmlns:xacro="http://www.ros.org/wiki/xacro" name="socket">
-  <xacro:include filename="$(find plug_and_socket_description)/urdf/socket.xacro"/>
-  <!-- This is only temporary until there's a better model to mount sockets to -->
+  <xacro:include filename="$(find plug_and_socket_description)/urdf/m_to_f_socket.xacro"/>
   <link name="socket_platform_link">
       <inertial name="socket_platform_inertial">
@@ -8,24 +7,24 @@
         <origin xyz="0 0 0" rpy="0 0 0"/>
         <inertia ixx="750" ixy="0" ixz="0"
-                 iyy="750" iyz="0" izz="187.5"/>
+                 iyy="195" iyz="0" izz="750"/>
         <origin xyz="0 0 0" rpy="0 0 0"/>
       </inertial>
       <visual name="socket_platform_visual">
         <geometry>
-          <box size="1.5 1.5 3"/>
+          <mesh filename="package://dave_object_models/models/electrical_panel/meshes/Underwater-Frame.dae" scale="1 1 1"/>
         </geometry>
-        <origin xyz="0 0 0" rpy="0 0 0"/>
+        <origin xyz="0 0 0" rpy="0 0 ${pi}"/>
       </visual>
       <collision name="socket_platform_collision">
         <geometry>
-          <box size="1.5 1.5 3"/>
+          <mesh filename="package://dave_object_models/models/electrical_panel/meshes/COLLISION-Underwater-Frame.dae" scale="1 1 1"/>
         </geometry>
-        <origin xyz="0 0 0" rpy="0 0 0"/>
+        <origin xyz="0 0 0" rpy="0 0 ${pi}"/>
       </collision>
   </link>
   <!-- Generate the sockets & attach them to the platform link -->
-  <xacro:socket_macro
+  <xacro:m_to_f_socket_macro
     name="socket1" xyz="0 0 0"
-    plug_model_name="plug" plug_link_name="plug" roll_tolerance="0.3"
+    plug_model_name="m_to_f_plug" plug_link_name="plug" roll_tolerance="0.3"
     pitch_tolerance="0.3" yaw_tolerance="0.3"
     mating_force="25" unmating_force="125"/>
@@ -33,51 +32,29 @@
   <joint name="socket1_joint" type="revolute">
     <limit effort="1.0" lower="0.0" upper="0.0" velocity="0.0"/>
-    <origin xyz="0 0.8 1" rpy="0 0 ${pi/2}"/>
+    <origin xyz="-0.31 0.51 1.34" rpy="0 ${-pi/4} ${pi/2}"/>
     <parent link="socket_platform_link"/>
     <child link="socket1_link"/>
   </joint>
-  <xacro:socket_macro
+  <xacro:m_to_f_socket_macro
     name="socket2" xyz="0 0 0"
-    plug_model_name="plug" plug_link_name="plug" roll_tolerance="0.3"
+    plug_model_name="m_to_f_plug" plug_link_name="plug" roll_tolerance="0.3"
     pitch_tolerance="0.3" yaw_tolerance="0.3"
     mating_force="25" unmating_force="125"/>
   <joint name="socket2_joint" type="revolute">
     <limit effort="1.0" lower="0.0" upper="0.0" velocity="0.0"/>
-    <origin xyz="0.8 0 1" rpy="0 0 0"/>
+    <origin xyz="0.125 0.475 1.315" rpy="0 ${-pi/4} ${pi/2}"/>
     <parent link="socket_platform_link"/>
     <child link="socket2_link"/>
   </joint>
-  <xacro:socket_macro
+  <xacro:m_to_f_socket_macro
     name="socket3" xyz="0 0 0"
-    plug_model_name="plug" plug_link_name="plug" roll_tolerance="0.3"
+    plug_model_name="m_to_f_plug" plug_link_name="plug" roll_tolerance="0.3"
     pitch_tolerance="0.3" yaw_tolerance="0.3"
     mating_force="25" unmating_force="125"/>
   <joint name="socket3_joint" type="revolute">
     <limit effort="1.0" lower="0.0" upper="0.0" velocity="0.0"/>
-    <origin xyz="0 -0.8 1" rpy="0 0 ${-pi/2}"/>
+    <origin xyz="-0.98 0.56 1.33" rpy="0 ${-pi/4} ${pi/2}"/>
     <parent link="socket_platform_link"/>
     <child link="socket3_link"/>
   </joint>
-  <xacro:socket_macro
-    name="socket4" xyz="0 0 0"
-    plug_model_name="plug" plug_link_name="plug" roll_tolerance="0.3"
-    pitch_tolerance="0.3" yaw_tolerance="0.3"
-    mating_force="25" unmating_force="125"/>
-  <joint name="socket4_joint" type="revolute">
-    <limit effort="1.0" lower="0.0" upper="0.0" velocity="0.0"/>
-    <origin xyz="-0.8 0 1" rpy="0 0 ${pi}"/>
-    <parent link="socket_platform_link"/>
-    <child link="socket4_link"/>
-  </joint>
-  <xacro:socket_macro
-    name="socket5" xyz="0 0 0"
-    plug_model_name="plug" plug_link_name="plug" roll_tolerance="${pi}"
-    pitch_tolerance="0.3" yaw_tolerance="0.3"
-    mating_force="25" unmating_force="125"/>
-  <joint name="socket5_joint" type="revolute">
-    <limit effort="1.0" lower="0.0" upper="0.0" velocity="0.0"/>
-    <origin xyz="0 0 1.55" rpy="0 -${pi/2} 0"/>
-    <parent link="socket_platform_link"/>
-    <child link="socket5_link"/>
-  </joint>
 </robot>

Commit message: Model updates ISO new Electrical Lead models
Added female plug to male socket models and URDF (xacro) templates.
Incorporated updated models into the
dave_demo_launch/dave_plug_and_socket_demo.launch demo.  The demo
now contains one of the male-to-female plug/socket pairs and two of
the female-to-male plug/receptacle pairs.

File: urdf/manipulators/plug_and_socket_description/urdf/socket_platform.xacro (robot description, xacro)
@@ -2,4 +2,5 @@
 <robot xmlns:xacro="http://www.ros.org/wiki/xacro" name="socket">
   <xacro:include filename="$(find plug_and_socket_description)/urdf/m_to_f_socket.xacro"/>
+  <xacro:include filename="$(find plug_and_socket_description)/urdf/f_to_m_receptacle.xacro"/>
   <link name="socket_platform_link">
       <inertial name="socket_platform_inertial">
@@ -24,15 +25,15 @@
   </link>
   <!-- Generate the sockets & attach them to the platform link -->
-  <xacro:m_to_f_socket_macro
-    name="socket1" xyz="0 0 0"
-    plug_model_name="m_to_f_plug" plug_link_name="plug" roll_tolerance="0.3"
+  <xacro:f_to_m_receptacle_macro
+    name="receptacle1" xyz="0 0 0"
+    plug_model_name="f_to_m_plug" plug_link_name="plug" roll_tolerance="0.3"
     pitch_tolerance="0.3" yaw_tolerance="0.3"
     mating_force="25" unmating_force="125"/>
   <!-- Revolute joint gets accurately loaded into Gazebo -->
-  <joint name="socket1_joint" type="revolute">
+  <joint name="receptacle1_joint" type="revolute">
     <limit effort="1.0" lower="0.0" upper="0.0" velocity="0.0"/>
-    <origin xyz="-0.31 0.51 1.34" rpy="0 ${-pi/4} ${pi/2}"/>
+    <origin xyz="-0.31 0.43 1.26" rpy="0 ${-pi/4} ${pi/2}"/>
     <parent link="socket_platform_link"/>
-    <child link="socket1_link"/>
+    <child link="receptacle1_link"/>
   </joint>
   <xacro:m_to_f_socket_macro
@@ -47,14 +48,14 @@
     <child link="socket2_link"/>
   </joint>
-  <xacro:m_to_f_socket_macro
-    name="socket3" xyz="0 0 0"
-    plug_model_name="m_to_f_plug" plug_link_name="plug" roll_tolerance="0.3"
+  <xacro:f_to_m_receptacle_macro
+    name="receptacle3" xyz="0 0 0"
+    plug_model_name="f_to_m_plug" plug_link_name="plug" roll_tolerance="0.3"
     pitch_tolerance="0.3" yaw_tolerance="0.3"
     mating_force="25" unmating_force="125"/>
-  <joint name="socket3_joint" type="revolute">
+  <joint name="receptacle3_joint" type="revolute">
     <limit effort="1.0" lower="0.0" upper="0.0" velocity="0.0"/>
-    <origin xyz="-0.98 0.56 1.33" rpy="0 ${-pi/4} ${pi/2}"/>
+    <origin xyz="-0.98 0.48 1.25" rpy="0 ${-pi/4} ${pi/2}"/>
     <parent link="socket_platform_link"/>
-    <child link="socket3_link"/>
+    <child link="receptacle3_link"/>
   </joint>
 </robot>
