Commit message: Small update to female-to-male plug recepatacle collision mesh scale
Decreasing the scale a little bit to make the fit more forgiving.

File: urdf/manipulators/plug_and_socket_description/urdf/f_to_m_receptacle.xacro (robot description, xacro)
@@ -15,5 +15,6 @@
       <visual>
         <geometry>
-          <mesh filename="package://dave_object_models/models/f_to_m_receptacle/meshes/Plug-Receptacle.dae" scale="0.4 0.4 0.4"/>
+          <mesh filename="package://dave_object_models/models/f_to_m_receptacle/meshes/Plug-Receptacle.dae"
+                scale="0.4 0.4 0.4"/>
         </geometry>
         <origin xyz="0 0 0" rpy="${pi/2} 0 ${pi/2}"/>
@@ -21,5 +22,6 @@
       <collision>
         <geometry>
-          <mesh filename="package://dave_object_models/models/f_to_m_receptacle/meshes/COLLISION-Plug-Receptacle.dae" scale="0.4 0.4 0.4"/>
+          <mesh filename="package://dave_object_models/models/f_to_m_receptacle/meshes/COLLISION-Plug-Receptacle.dae"
+                scale="0.375 0.375 0.375"/> <!-- A little smaller to make the fit more forgiving -->
         </geometry>
         <origin xyz="0 0 0" rpy="${pi/2} 0 ${pi/2}"/>

Commit message: Plug and socket plugin code update to improve performance
Also updated all of the models to avoid name conflicts if
they're used multiple times in the same world.

File: urdf/manipulators/plug_and_socket_description/urdf/f_to_m_receptacle.xacro (robot description, xacro)
@@ -15,6 +15,7 @@
       <visual>
         <geometry>
+          <!-- Smaller scale than plug to make the fit more forgiving -->
           <mesh filename="package://dave_object_models/models/f_to_m_receptacle/meshes/Plug-Receptacle.dae"
-                scale="0.4 0.4 0.4"/>
+                scale="0.375 0.375 0.375"/>
         </geometry>
         <origin xyz="0 0 0" rpy="${pi/2} 0 ${pi/2}"/>
@@ -23,5 +24,5 @@
         <geometry>
           <mesh filename="package://dave_object_models/models/f_to_m_receptacle/meshes/COLLISION-Plug-Receptacle.dae"
-                scale="0.375 0.375 0.375"/> <!-- A little smaller to make the fit more forgiving -->
+                scale="0.375 0.375 0.375"/>
         </geometry>
         <origin xyz="0 0 0" rpy="${pi/2} 0 ${pi/2}"/>
@@ -40,5 +41,5 @@
           <cylinder length="0.01" radius="0.06"/>
         </geometry>
-        <origin xyz="0.02 0 0" rpy="0 ${-pi/2} 0"/>
+        <origin xyz="0.01 0 0" rpy="0 ${-pi/2} 0"/>
       </collision>
     </link>

File: urdf/manipulators/plug_and_socket_description/urdf/m_to_f_socket.xacro (robot description, xacro)
@@ -38,5 +38,5 @@
           <cylinder length="0.01" radius="0.06"/>
         </geometry>
-        <origin xyz="0 0 0" rpy="0 ${-pi/2} 0"/>
+        <origin xyz="0.01 0 0" rpy="0 ${-pi/2} 0"/>
       </collision>
     </link>

File: urdf/manipulators/plug_and_socket_description/urdf/socket_platform.xacro (robot description, xacro)
@@ -27,5 +27,5 @@
   <xacro:f_to_m_receptacle_macro
     name="receptacle1" xyz="0 0 0"
-    plug_model_name="f_to_m_plug" plug_link_name="plug" roll_tolerance="0.3"
+    plug_model_name="f_to_m_plug" plug_link_name="f_to_m_plug" roll_tolerance="0.3"
     pitch_tolerance="0.3" yaw_tolerance="0.3"
     mating_force="25" unmating_force="125"/>
@@ -33,5 +33,5 @@
   <joint name="receptacle1_joint" type="revolute">
     <limit effort="1.0" lower="0.0" upper="0.0" velocity="0.0"/>
-    <origin xyz="-0.31 0.43 1.26" rpy="0 ${-pi/4} ${pi/2}"/>
+    <origin xyz="-0.31 0.424 1.254" rpy="0 ${-pi/4} ${pi/2}"/>
     <parent link="socket_platform_link"/>
     <child link="receptacle1_link"/>
@@ -39,5 +39,5 @@
   <xacro:m_to_f_socket_macro
     name="socket2" xyz="0 0 0"
-    plug_model_name="m_to_f_plug" plug_link_name="plug" roll_tolerance="0.3"
+    plug_model_name="m_to_f_plug" plug_link_name="m_to_f_plug" roll_tolerance="0.3"
     pitch_tolerance="0.3" yaw_tolerance="0.3"
     mating_force="25" unmating_force="125"/>
@@ -50,10 +50,10 @@
   <xacro:f_to_m_receptacle_macro
     name="receptacle3" xyz="0 0 0"
-    plug_model_name="f_to_m_plug" plug_link_name="plug" roll_tolerance="0.3"
+    plug_model_name="f_to_m_plug" plug_link_name="f_to_m_plug" roll_tolerance="0.3"
     pitch_tolerance="0.3" yaw_tolerance="0.3"
     mating_force="25" unmating_force="125"/>
   <joint name="receptacle3_joint" type="revolute">
     <limit effort="1.0" lower="0.0" upper="0.0" velocity="0.0"/>
-    <origin xyz="-0.98 0.48 1.25" rpy="0 ${-pi/4} ${pi/2}"/>
+    <origin xyz="-0.98 0.475 1.245" rpy="0 ${-pi/4} ${pi/2}"/>
     <parent link="socket_platform_link"/>
     <child link="receptacle3_link"/>
