Commit message: Pass namespace parameters for sensors
Signed-off-by: Yadunund <yadunund@gmail.com>

File: urdf/dave_snippets/urdf/sensor_snippets.xacro (robot description, xacro)
@@ -14,4 +14,8 @@
 <!-- modified for custom sonar_snippets path -->
 <robot xmlns:xacro="http://www.ros.org/wiki/xacro">
+  <!-- Parameters -->
+  <xacro:property name="namespace" value="rexrov"/>
+  <xacro:property name="parent_link" value="rexrov/base_link"/>
+  <xacro:property name="suffix" value="down"/>
   <xacro:include filename="$(find uuv_sensor_ros_plugins)/urdf/imu_snippets.xacro" />
   <xacro:include filename="$(find uuv_sensor_ros_plugins)/urdf/magnetometer_snippets.xacro" />
@@ -20,5 +24,5 @@
   <xacro:include filename="$(find uuv_sensor_ros_plugins)/urdf/dvl_snippets.xacro" />
   <xacro:include filename="$(find uuv_sensor_ros_plugins)/urdf/rpt_snippets.xacro" />
-  <xacro:include filename="$(find dave_snippets)/urdf/sonar_snippets.xacro" />
+  <xacro:include filename="$(find dave_snippets)/urdf/sonar_snippets.xacro" namespace="${namespace}" parent_link="${parent_link}" suffix="${suffix}"/>
   <xacro:include filename="$(find uuv_sensor_ros_plugins)/urdf/stereo_snippets.xacro" />
   <xacro:include filename="$(find uuv_sensor_ros_plugins)/urdf/gps_sensor_snippets.xacro" />

File: urdf/robots/rexrov_description/urdf/rexrov_base.xacro (robot description, xacro)
@@ -21,12 +21,12 @@
             thesis. Institutt for marin teknikk, 2012.
   -->
-  <!-- includes -->
-  <xacro:include filename="$(find uuv_descriptions)/urdf/common.urdf.xacro"/>
-  <xacro:include filename="$(find dave_snippets)/urdf/sensor_snippets.xacro"/>
-  <xacro:include filename="$(find uuv_gazebo_ros_plugins)/urdf/snippets.xacro"/>
   <!-- Parameters -->
   <xacro:property name="namespace" value="rexrov"/>
   <xacro:property name="visual_mesh_file" value="file://$(find uuv_descriptions)/meshes/RexROV_no_props.dae"/>
   <xacro:property name="prop_mesh_file" value="file://$(find uuv_descriptions)/meshes/prop.dae"/>
+  <!-- includes -->
+  <xacro:include filename="$(find uuv_descriptions)/urdf/common.urdf.xacro" namespace="${namespace}"/>
+  <xacro:include filename="$(find dave_snippets)/urdf/sensor_snippets.xacro" namespace="${namespace}" parent_link="${namespace}/base_link" suffix="down"/>
+  <xacro:include filename="$(find uuv_gazebo_ros_plugins)/urdf/snippets.xacro" namespace="${namespace}"/>
   <!-- Mass, see p.28 in Berg2012 -->
   <xacro:property name="mass" value="1862.87"/>

File: urdf/robots/rexrov_description/urdf/rexrov_oberon7.xacro (robot description, xacro)
@@ -17,7 +17,7 @@
   <xacro:arg name="inertial_reference_frame" default="world"/>
   <!-- Include the ROV macro file -->
-  <xacro:include filename="$(find rexrov_description)/urdf/rexrov_base.xacro"/>
-  <xacro:include filename="$(find uuv_descriptions)/urdf/rexrov.gazebo.xacro"/>
-  <xacro:include filename="$(find dave_oberon7_description)/urdf/oberon7_default.xacro" />
+  <xacro:include filename="$(find rexrov_description)/urdf/rexrov_base.xacro" namespace="$(arg namespace)"/>
+  <xacro:include filename="$(find uuv_descriptions)/urdf/rexrov.gazebo.xacro" namespace="$(arg namespace)"/>
+  <xacro:include filename="$(find dave_oberon7_description)/urdf/oberon7_default.xacro" namespace="$(arg namespace)"/>
   <!-- This implements the image_sonar_ros_plugin.so implemented in uuv_simulator.
        See the source code https://github.com/uuvsimulator/uuv_simulator/blob/master/uuv_sensor_plugins/uuv_sensor_ros_plugins/src/gazebo_ros_image_sonar.cpp
