Commit message: Adjusted sensor positions

File: urdf/robots/virgil_description/urdf/virgil_sensors.xacro (robot description, xacro)
@@ -18,5 +18,5 @@
     parent_link="${namespace}/base_link"
     inertial_reference_frame="${inertial_reference_frame}">
-    <origin xyz="-1.4 0 -0.312" rpy="0 ${0.5*pi} 0"/>
+    <origin xyz="0.5 0 -0.85" rpy="0 ${0.5*pi} 0"/>
   </xacro:default_dvl_macro>
   <!-- Magnetometer  -->
