Commit message: File cleanup

File: urdf/robots/virgil_description/urdf/virgil.xacro (robot description, xacro)
@@ -1,10 +1,9 @@
 <?xml version="1.0"?>
-<robot name="doc_ricketts" xmlns:xacro="https://www.ros.org/wiki/xacro">
+<robot name="virgil" xmlns:xacro="https://www.ros.org/wiki/xacro">
     <xacro:arg name="debug" default="false"/>
-    <xacro:arg name="namespace" default="doc_ricketts"/>
+    <xacro:arg name="namespace" default="virgil"/>
     <!-- "Dummy" base link to eliminate root link inertia warning -->
     <link name="$(arg namespace)/base_link"/>
-    <link name="$(arg namespace)/doc_ricketts_link">
-        <!-- Values loosely based on https://www.mbari.org/at-sea/vehicles/remotely-operated-vehicles/rov-docricketts-specifications-2/ -->
+    <link name="$(arg namespace)/virgil_link">
         <!-- Inertia values based on uniform mass distribution -->
         <inertial>
@@ -19,5 +18,5 @@
             <origin xyz="0 0 0" rpy="0 0 0"/>
             <geometry>
-                <mesh filename="package://doc_ricketts_description/meshes/ROV.dae" scale="1 1 1"/>
+                <mesh filename="package://virgil_description/meshes/ROV.dae" scale="1 1 1"/>
             </geometry>
         </visual>
@@ -25,12 +24,12 @@
             <origin xyz="0 0 0" rpy="0 0 0"/>
             <geometry>
-                <mesh filename="package://doc_ricketts_description/meshes/ROV.dae" scale="1 1 1"/>
+                <mesh filename="package://virgil_description/meshes/ROV.dae" scale="1 1 1"/>
             </geometry>
         </collision>
     </link>
-    <joint name="$(arg namespace)/doc_ricketts_base_joint" type="fixed">
+    <joint name="$(arg namespace)/virgil_base_joint" type="fixed">
         <origin xyz="0 0 0" rpy="0 0 0"/>
         <parent link="$(arg namespace)/base_link"/>
-        <child link="$(arg namespace)/doc_ricketts_link"/>
+        <child link="$(arg namespace)/virgil_link"/>
     </joint>
     <gazebo>
@@ -86,10 +85,10 @@
         <plugin name="gazebo_ros_control" filename="libgazebo_ros_control.so">
             <robotNamespace>$(arg namespace)</robotNamespace>
-            <robotParam>$(arg namespace)/doc_ricketts</robotParam>
+            <robotParam>$(arg namespace)/virgil</robotParam>
         </plugin>
     </gazebo> -->
-    <!-- <xacro:include filename="$(find doc_ricketts_description)/urdf/doc_ricketts.gazebo.xacro"/> -->
-    <!-- <xacro:include filename="$(find doc_ricketts_description)/urdf/doc_ricketts.actuators.xacro"/> -->
-    <!-- <xacro:doc_ricketts_gazebo namespace="$(arg namespace)"/> -->
+    <!-- <xacro:include filename="$(find virgil_description)/urdf/virgil.gazebo.xacro"/> -->
+    <!-- <xacro:include filename="$(find virgil_description)/urdf/virgil.actuators.xacro"/> -->
+    <!-- <xacro:virgil_gazebo namespace="$(arg namespace)"/> -->
     <xacro:property name="prop_mesh_file" value="file://$(find eca_a9_description)/mesh/eca_a9_propeller.dae"/>
     <xacro:include filename="$(find uuv_descriptions)/urdf/common.urdf.xacro"/>

Commit message: Changed mesh names

File: urdf/robots/virgil_description/urdf/virgil.xacro (robot description, xacro)
@@ -18,5 +18,5 @@
             <origin xyz="0 0 0" rpy="0 0 0"/>
             <geometry>
-                <mesh filename="package://virgil_description/meshes/ROV.dae" scale="1 1 1"/>
+                <mesh filename="package://virgil_description/meshes/virgil.dae" scale="1 1 1"/>
             </geometry>
         </visual>
@@ -24,5 +24,5 @@
             <origin xyz="0 0 0" rpy="0 0 0"/>
             <geometry>
-                <mesh filename="package://virgil_description/meshes/ROV.dae" scale="1 1 1"/>
+                <mesh filename="package://virgil_description/meshes/virgil.dae" scale="1 1 1"/>
             </geometry>
         </collision>
@@ -94,35 +94,35 @@
     <xacro:include filename="$(find uuv_descriptions)/urdf/common.urdf.xacro"/>
     <xacro:include filename="$(find uuv_gazebo_ros_plugins)/urdf/thruster_snippets.xacro"/>
-    <xacro:macro name="thruster_macro" params="thruster_id *origin">
-        <xacro:thruster_module_first_order_basic_fcn_macro namespace="$(arg namespace)" thruster_id="${thruster_id}" mesh_filename="${prop_mesh_file}" dyn_time_constant="0.05" rotor_constant="0.00031">
+    <xacro:macro name="thruster_macro" params="thruster_id mesh_file *origin">
+        <xacro:thruster_module_first_order_basic_fcn_macro namespace="$(arg namespace)" thruster_id="${thruster_id}" mesh_filename="${mesh_file}" dyn_time_constant="0.05" rotor_constant="0.00031">
             <xacro:insert_block name="origin"/>
         </xacro:thruster_module_first_order_basic_fcn_macro>
     </xacro:macro>
     <!-- Port-Aft RL-->
-    <xacro:thruster_macro thruster_id="0">
+    <xacro:thruster_macro thruster_id="0" mesh_file="file://$(find eca_a9_description)/mesh/eca_a9_propeller.dae">
         <origin xyz="0.53491 1.51341 1.18597" rpy="1.5708 0.0 0.610865"/>
     </xacro:thruster_macro>
     <!-- Starboard-Aft RR-->
-    <xacro:thruster_macro thruster_id="1">
+    <xacro:thruster_macro thruster_id="1" mesh_file="file://$(find eca_a9_description)/mesh/eca_a9_propeller.dae">
         <origin xyz="-0.536834 1.51248 1.18592" rpy="1.5708 0.0 -0.610865"/>
     </xacro:thruster_macro>
     <!-- Port-Forward FL-->
-    <xacro:thruster_macro thruster_id="2">
+    <xacro:thruster_macro thruster_id="2" mesh_file="file://$(find eca_a9_description)/mesh/eca_a9_propeller.dae">
         <origin xyz="0.539848 -1.28724 1.18875" rpy="1.5708 0.0 -0.610865"/>
     </xacro:thruster_macro>
     <!-- Starboard-Forward FR-->
-    <xacro:thruster_macro thruster_id="3">
+    <xacro:thruster_macro thruster_id="3" mesh_file="file://$(find eca_a9_description)/mesh/eca_a9_propeller.dae">
         <origin xyz="-0.536692 -1.28841 1.1888" rpy="1.5708 0.0 -2.53073"/>
     </xacro:thruster_macro>
     <!-- Port-Forward-Vertical TL-->
-    <xacro:thruster_macro thruster_id="4">
+    <xacro:thruster_macro thruster_id="4" mesh_file="file://$(find eca_a9_description)/mesh/eca_a9_propeller.dae">
         <origin xyz="0.706649 -0.761326 1.8604" rpy="0.0 -0.174533 0.0"/>
     </xacro:thruster_macro>
     <!-- Starboard-Forward-Vertical TR-->
-    <xacro:thruster_macro thruster_id="5">
+    <xacro:thruster_macro thruster_id="5" mesh_file="file://$(find eca_a9_description)/mesh/eca_a9_propeller.dae">
         <origin xyz="-0.70968 -0.761276 1.85086" rpy="0.0 0.174533 0.0"/>
     </xacro:thruster_macro>
     <!-- Aft-Vertical (central)-->
-    <xacro:thruster_macro thruster_id="6">
+    <xacro:thruster_macro thruster_id="6" mesh_file="file://$(find eca_a9_description)/mesh/eca_a9_propeller.dae">
         <origin xyz="2.54822e-05 1.63582 1.78479" rpy="0.0 0.0 0.0"/>
     </xacro:thruster_macro>

Commit message: Added separated mesh files

File: urdf/robots/virgil_description/urdf/virgil.xacro (robot description, xacro)
@@ -91,38 +91,38 @@
     <!-- <xacro:include filename="$(find virgil_description)/urdf/virgil.actuators.xacro"/> -->
     <!-- <xacro:virgil_gazebo namespace="$(arg namespace)"/> -->
-    <xacro:property name="prop_mesh_file" value="file://$(find eca_a9_description)/mesh/eca_a9_propeller.dae"/>
+    <xacro:property name="prop_mesh_file" value="file://$(find virgil_description)/mesh/virgil_propeller.dae"/>
     <xacro:include filename="$(find uuv_descriptions)/urdf/common.urdf.xacro"/>
     <xacro:include filename="$(find uuv_gazebo_ros_plugins)/urdf/thruster_snippets.xacro"/>
     <xacro:macro name="thruster_macro" params="thruster_id mesh_file *origin">
-        <xacro:thruster_module_first_order_basic_fcn_macro namespace="$(arg namespace)" thruster_id="${thruster_id}" mesh_filename="${mesh_file}" dyn_time_constant="0.05" rotor_constant="0.00031">
+        <xacro:thruster_module_first_order_basic_fcn_macro namespace="$(arg namespace)" thruster_id="${thruster_id}" mesh_filename="${prop_mesh_file}" dyn_time_constant="0.05" rotor_constant="0.00031">
             <xacro:insert_block name="origin"/>
         </xacro:thruster_module_first_order_basic_fcn_macro>
     </xacro:macro>
     <!-- Port-Aft RL-->
-    <xacro:thruster_macro thruster_id="0" mesh_file="file://$(find eca_a9_description)/mesh/eca_a9_propeller.dae">
+    <xacro:thruster_macro thruster_id="0">
         <origin xyz="0.53491 1.51341 1.18597" rpy="1.5708 0.0 0.610865"/>
     </xacro:thruster_macro>
     <!-- Starboard-Aft RR-->
-    <xacro:thruster_macro thruster_id="1" mesh_file="file://$(find eca_a9_description)/mesh/eca_a9_propeller.dae">
+    <xacro:thruster_macro thruster_id="1">
         <origin xyz="-0.536834 1.51248 1.18592" rpy="1.5708 0.0 -0.610865"/>
     </xacro:thruster_macro>
     <!-- Port-Forward FL-->
-    <xacro:thruster_macro thruster_id="2" mesh_file="file://$(find eca_a9_description)/mesh/eca_a9_propeller.dae">
+    <xacro:thruster_macro thruster_id="2">
         <origin xyz="0.539848 -1.28724 1.18875" rpy="1.5708 0.0 -0.610865"/>
     </xacro:thruster_macro>
     <!-- Starboard-Forward FR-->
-    <xacro:thruster_macro thruster_id="3" mesh_file="file://$(find eca_a9_description)/mesh/eca_a9_propeller.dae">
+    <xacro:thruster_macro thruster_id="3">
         <origin xyz="-0.536692 -1.28841 1.1888" rpy="1.5708 0.0 -2.53073"/>
     </xacro:thruster_macro>
     <!-- Port-Forward-Vertical TL-->
-    <xacro:thruster_macro thruster_id="4" mesh_file="file://$(find eca_a9_description)/mesh/eca_a9_propeller.dae">
+    <xacro:thruster_macro thruster_id="4">
         <origin xyz="0.706649 -0.761326 1.8604" rpy="0.0 -0.174533 0.0"/>
     </xacro:thruster_macro>
     <!-- Starboard-Forward-Vertical TR-->
-    <xacro:thruster_macro thruster_id="5" mesh_file="file://$(find eca_a9_description)/mesh/eca_a9_propeller.dae">
+    <xacro:thruster_macro thruster_id="5">
         <origin xyz="-0.70968 -0.761276 1.85086" rpy="0.0 0.174533 0.0"/>
     </xacro:thruster_macro>
     <!-- Aft-Vertical (central)-->
-    <xacro:thruster_macro thruster_id="6" mesh_file="file://$(find eca_a9_description)/mesh/eca_a9_propeller.dae">
+    <xacro:thruster_macro thruster_id="6">
         <origin xyz="2.54822e-05 1.63582 1.78479" rpy="0.0 0.0 0.0"/>
     </xacro:thruster_macro>

Commit message: Removed unused mesh file arg

File: urdf/robots/virgil_description/urdf/virgil.xacro (robot description, xacro)
@@ -94,5 +94,5 @@
     <xacro:include filename="$(find uuv_descriptions)/urdf/common.urdf.xacro"/>
     <xacro:include filename="$(find uuv_gazebo_ros_plugins)/urdf/thruster_snippets.xacro"/>
-    <xacro:macro name="thruster_macro" params="thruster_id mesh_file *origin">
+    <xacro:macro name="thruster_macro" params="thruster_id *origin">
         <xacro:thruster_module_first_order_basic_fcn_macro namespace="$(arg namespace)" thruster_id="${thruster_id}" mesh_filename="${prop_mesh_file}" dyn_time_constant="0.05" rotor_constant="0.00031">
             <xacro:insert_block name="origin"/>

Commit message: Added aligned props, substitute from RexROV

File: urdf/robots/virgil_description/urdf/virgil.xacro (robot description, xacro)
@@ -18,5 +18,5 @@
             <origin xyz="0 0 0" rpy="0 0 0"/>
             <geometry>
-                <mesh filename="package://virgil_description/meshes/virgil.dae" scale="1 1 1"/>
+                <mesh filename="file://$(find virgil_description)/meshes/virgil.dae" scale="1 1 1"/>
             </geometry>
         </visual>
@@ -24,5 +24,5 @@
             <origin xyz="0 0 0" rpy="0 0 0"/>
             <geometry>
-                <mesh filename="package://virgil_description/meshes/virgil.dae" scale="1 1 1"/>
+                <mesh filename="file://$(find virgil_description)/meshes/virgil.dae" scale="1 1 1"/>
             </geometry>
         </collision>
@@ -82,48 +82,59 @@
         </plugin>
     </gazebo>
-<!--     <gazebo>
+    <gazebo>
         <plugin name="gazebo_ros_control" filename="libgazebo_ros_control.so">
             <robotNamespace>$(arg namespace)</robotNamespace>
             <robotParam>$(arg namespace)/virgil</robotParam>
         </plugin>
-    </gazebo> -->
-    <!-- <xacro:include filename="$(find virgil_description)/urdf/virgil.gazebo.xacro"/> -->
-    <!-- <xacro:include filename="$(find virgil_description)/urdf/virgil.actuators.xacro"/> -->
-    <!-- <xacro:virgil_gazebo namespace="$(arg namespace)"/> -->
-    <xacro:property name="prop_mesh_file" value="file://$(find virgil_description)/mesh/virgil_propeller.dae"/>
+    </gazebo>
+    <xacro:property name="prop_mesh_file" value="file://$(find uuv_descriptions)/meshes/prop.dae"/>
     <xacro:include filename="$(find uuv_descriptions)/urdf/common.urdf.xacro"/>
     <xacro:include filename="$(find uuv_gazebo_ros_plugins)/urdf/thruster_snippets.xacro"/>
+  <!-- Thruster joint and link snippet
+       Wrapper for the the thruster_module_first_order_basic_fcn_macro
+       defined in uuv_gazebo_ros_plugins/urdf/thruster_snippet.
+       Uses the "thruster_cf_basic_macro"
+         1) Basic curve
+       Input: x
+       Output: thrust
+       Function: thrust = rotorConstant * x * abs(x)
+  -->
     <xacro:macro name="thruster_macro" params="thruster_id *origin">
-        <xacro:thruster_module_first_order_basic_fcn_macro namespace="$(arg namespace)" thruster_id="${thruster_id}" mesh_filename="${prop_mesh_file}" dyn_time_constant="0.05" rotor_constant="0.00031">
+        <xacro:thruster_module_first_order_basic_fcn_macro
+            namespace="$(arg namespace)"
+            thruster_id="${thruster_id}"
+            mesh_filename="${prop_mesh_file}"
+            dyn_time_constant="0.05"
+            rotor_constant="0.00031">
             <xacro:insert_block name="origin"/>
         </xacro:thruster_module_first_order_basic_fcn_macro>
     </xacro:macro>
     <!-- Port-Aft RL-->
-    <xacro:thruster_macro thruster_id="0">
-        <origin xyz="0.53491 1.51341 1.18597" rpy="1.5708 0.0 0.610865"/>
+     <xacro:thruster_macro thruster_id="0">
+        <origin xyz="0.53491 1.51341 1.18597" rpy="0.0 0.0 ${1.5708+0.610865}"/>
+     </xacro:thruster_macro>
+     <!-- Starboard-Aft RR -->
+    <xacro:thruster_macro thruster_id="1">
+        <origin xyz="-0.536834 1.51248 1.18592" rpy="0.0 0.0 ${1.5708-0.610865}"/>
     </xacro:thruster_macro>
-    <!-- Starboard-Aft RR-->
-    <xacro:thruster_macro thruster_id="1">
-        <origin xyz="-0.536834 1.51248 1.18592" rpy="1.5708 0.0 -0.610865"/>
-    </xacro:thruster_macro>
-    <!-- Port-Forward FL-->
+    <!-- Port-Forward FL -->
     <xacro:thruster_macro thruster_id="2">
-        <origin xyz="0.539848 -1.28724 1.18875" rpy="1.5708 0.0 -0.610865"/>
+        <origin xyz="0.539848 -1.28724 1.18875" rpy="0.0 0.0 ${-1.5708-0.610865}"/>
     </xacro:thruster_macro>
     <!-- Starboard-Forward FR-->
     <xacro:thruster_macro thruster_id="3">
-        <origin xyz="-0.536692 -1.28841 1.1888" rpy="1.5708 0.0 -2.53073"/>
+        <origin xyz="-0.536692 -1.28841 1.1888" rpy="0.0 0.0 ${1.5708-2.53073}"/>
     </xacro:thruster_macro>
     <!-- Port-Forward-Vertical TL-->
     <xacro:thruster_macro thruster_id="4">
-        <origin xyz="0.706649 -0.761326 1.8604" rpy="0.0 -0.174533 0.0"/>
+        <origin xyz="0.706649 -0.761326 1.8604" rpy="0.0 ${-1.5708-0.174533} 0.0"/>
     </xacro:thruster_macro>
     <!-- Starboard-Forward-Vertical TR-->
     <xacro:thruster_macro thruster_id="5">
-        <origin xyz="-0.70968 -0.761276 1.85086" rpy="0.0 0.174533 0.0"/>
+        <origin xyz="-0.70968 -0.761276 1.85086" rpy="0.0 ${-1.5708+0.174533} 0.0"/>
     </xacro:thruster_macro>
-    <!-- Aft-Vertical (central)-->
+        <!-- Aft-Vertical (central)-->
     <xacro:thruster_macro thruster_id="6">
-        <origin xyz="2.54822e-05 1.63582 1.78479" rpy="0.0 0.0 0.0"/>
+        <origin xyz="2.54822e-05 1.63582 1.78479" rpy="0.0 -1.5708 0.0"/>
     </xacro:thruster_macro>
 </robot>

Commit message: Adjusted ROV axis, aligned props, shifted COG

File: urdf/robots/virgil_description/urdf/virgil.xacro (robot description, xacro)
@@ -16,5 +16,5 @@
         </inertial>
         <visual>
-            <origin xyz="0 0 0" rpy="0 0 0"/>
+            <origin xyz="0 0 -0.9" rpy="0 0 1.5708"/>
             <geometry>
                 <mesh filename="file://$(find virgil_description)/meshes/virgil.dae" scale="1 1 1"/>
@@ -22,5 +22,5 @@
         </visual>
         <collision>
-            <origin xyz="0 0 0" rpy="0 0 0"/>
+            <origin xyz="0 0 -0.9" rpy="0 0 1.5708"/>
             <geometry>
                 <mesh filename="file://$(find virgil_description)/meshes/virgil.dae" scale="1 1 1"/>
@@ -85,5 +85,5 @@
         <plugin name="gazebo_ros_control" filename="libgazebo_ros_control.so">
             <robotNamespace>$(arg namespace)</robotNamespace>
-            <robotParam>$(arg namespace)/virgil</robotParam>
+            <robotParam>$(arg namespace)</robotParam>
         </plugin>
     </gazebo>
@@ -112,29 +112,29 @@
     <!-- Port-Aft RL-->
      <xacro:thruster_macro thruster_id="0">
-        <origin xyz="0.53491 1.51341 1.18597" rpy="0.0 0.0 ${1.5708+0.610865}"/>
+        <origin xyz="-1.51341 0.53491 ${1.18597-0.9}" rpy="0.0 0.0 ${3.14159+0.610865}"/>
      </xacro:thruster_macro>
      <!-- Starboard-Aft RR -->
     <xacro:thruster_macro thruster_id="1">
-        <origin xyz="-0.536834 1.51248 1.18592" rpy="0.0 0.0 ${1.5708-0.610865}"/>
+        <origin xyz="-1.51248 -0.536834 ${1.18592-0.9}" rpy="0.0 0.0 ${3.14159-0.610865}"/>
     </xacro:thruster_macro>
     <!-- Port-Forward FL -->
     <xacro:thruster_macro thruster_id="2">
-        <origin xyz="0.539848 -1.28724 1.18875" rpy="0.0 0.0 ${-1.5708-0.610865}"/>
+        <origin xyz="1.28724 0.539848 ${1.18875-0.9}" rpy="0.0 0.0 -0.610865"/>
     </xacro:thruster_macro>
     <!-- Starboard-Forward FR-->
     <xacro:thruster_macro thruster_id="3">
-        <origin xyz="-0.536692 -1.28841 1.1888" rpy="0.0 0.0 ${1.5708-2.53073}"/>
+        <origin xyz="1.28841 -0.536692 ${1.1888-0.9}" rpy="0.0 0.0 ${3.14159-2.53073}"/>
     </xacro:thruster_macro>
     <!-- Port-Forward-Vertical TL-->
     <xacro:thruster_macro thruster_id="4">
-        <origin xyz="0.706649 -0.761326 1.8604" rpy="0.0 ${-1.5708-0.174533} 0.0"/>
+        <origin xyz="0.761326 0.706649 ${1.8604-0.9}" rpy="0.0 ${-1.5708-0.174533} 0.0"/>
     </xacro:thruster_macro>
     <!-- Starboard-Forward-Vertical TR-->
     <xacro:thruster_macro thruster_id="5">
-        <origin xyz="-0.70968 -0.761276 1.85086" rpy="0.0 ${-1.5708+0.174533} 0.0"/>
+        <origin xyz="0.761276 -0.70968 ${1.85086-0.9}" rpy="0.0 ${-1.5708+0.174533} 0.0"/>
     </xacro:thruster_macro>
         <!-- Aft-Vertical (central)-->
     <xacro:thruster_macro thruster_id="6">
-        <origin xyz="2.54822e-05 1.63582 1.78479" rpy="0.0 -1.5708 0.0"/>
+        <origin xyz="-1.63582 2.54822e-05 ${1.78479-0.9}" rpy="0.0 -1.5708 0.0"/>
     </xacro:thruster_macro>
 </robot>

Commit message: Added sensors

File: urdf/robots/virgil_description/urdf/virgil.xacro (robot description, xacro)
@@ -138,3 +138,9 @@
         <origin xyz="-1.63582 2.54822e-05 ${1.78479-0.9}" rpy="0.0 -1.5708 0.0"/>
     </xacro:thruster_macro>
+    <!-- includes -->
+    <xacro:property name="namespace" value="$(arg namespace)"/>
+    <xacro:property name="inertial_reference_frame" value="world"/>
+    <xacro:include filename="$(find uuv_sensor_ros_plugins)/urdf/sensor_snippets.xacro"/>
+    <xacro:include filename="$(find uuv_gazebo_ros_plugins)/urdf/snippets.xacro"/>
+    <xacro:include filename="$(find virgil_description)/urdf/virgil_sensors.xacro"/>
 </robot>

Commit message: Added new virgil props

File: urdf/robots/virgil_description/urdf/virgil.xacro (robot description, xacro)
@@ -88,5 +88,5 @@
         </plugin>
     </gazebo>
-    <xacro:property name="prop_mesh_file" value="file://$(find uuv_descriptions)/meshes/prop.dae"/>
+    <xacro:property name="prop_mesh_file" value="file://$(find virgil_description)/meshes/virgil_prop.dae"/>
     <xacro:include filename="$(find uuv_descriptions)/urdf/common.urdf.xacro"/>
     <xacro:include filename="$(find uuv_gazebo_ros_plugins)/urdf/thruster_snippets.xacro"/>
@@ -112,29 +112,29 @@
     <!-- Port-Aft RL-->
      <xacro:thruster_macro thruster_id="0">
-        <origin xyz="-1.51341 0.53491 ${1.18597-0.9}" rpy="0.0 0.0 ${3.14159+0.610865}"/>
+        <origin xyz="-1.51341 0.53491 ${1.18597-0.88}" rpy="1.5708 0.0 ${1.5708+0.610865}"/>
      </xacro:thruster_macro>
      <!-- Starboard-Aft RR -->
     <xacro:thruster_macro thruster_id="1">
-        <origin xyz="-1.51248 -0.536834 ${1.18592-0.9}" rpy="0.0 0.0 ${3.14159-0.610865}"/>
+        <origin xyz="-1.51248 -0.536834 ${1.18592-0.88}" rpy="1.5708 0.0 ${1.5708-0.610865}"/>
     </xacro:thruster_macro>
     <!-- Port-Forward FL -->
     <xacro:thruster_macro thruster_id="2">
-        <origin xyz="1.28724 0.539848 ${1.18875-0.9}" rpy="0.0 0.0 -0.610865"/>
+        <origin xyz="1.28724 0.539848 ${1.18875-0.88}" rpy="1.5708 0.0 ${1.5708-0.610865}"/>
     </xacro:thruster_macro>
     <!-- Starboard-Forward FR-->
     <xacro:thruster_macro thruster_id="3">
-        <origin xyz="1.28841 -0.536692 ${1.1888-0.9}" rpy="0.0 0.0 ${3.14159-2.53073}"/>
+        <origin xyz="1.28841 -0.536692 ${1.1888-0.88}" rpy="1.5708 0.0 ${1.5708-2.53073}"/>
     </xacro:thruster_macro>
     <!-- Port-Forward-Vertical TL-->
     <xacro:thruster_macro thruster_id="4">
-        <origin xyz="0.761326 0.706649 ${1.8604-0.9}" rpy="0.0 ${-1.5708-0.174533} 0.0"/>
+        <origin xyz="0.761326 ${0.02+0.706649} ${1.8604-0.88}" rpy="0.0 -0.174533 0.0"/>
     </xacro:thruster_macro>
     <!-- Starboard-Forward-Vertical TR-->
     <xacro:thruster_macro thruster_id="5">
-        <origin xyz="0.761276 -0.70968 ${1.85086-0.9}" rpy="0.0 ${-1.5708+0.174533} 0.0"/>
+        <origin xyz="0.761276 ${-0.70968+0.02} ${1.85086-0.88}" rpy="0.0 0.174533 0.0"/>
     </xacro:thruster_macro>
         <!-- Aft-Vertical (central)-->
     <xacro:thruster_macro thruster_id="6">
-        <origin xyz="-1.63582 2.54822e-05 ${1.78479-0.9}" rpy="0.0 -1.5708 0.0"/>
+        <origin xyz="-1.63582 ${2.54822e-05+0.02} ${1.78479-0.88}" rpy="0.0 0.0 0.0"/>
     </xacro:thruster_macro>
     <!-- includes -->
