Commit message: Fix for prop orientation and joy teleop

File: urdf/robots/virgil_description/urdf/virgil.xacro (robot description, xacro)
@@ -104,4 +104,7 @@
             namespace="$(arg namespace)"
             thruster_id="${thruster_id}"
+            x_axis="0"
+            y_axis="0"
+            z_axis="1"
             mesh_filename="${prop_mesh_file}"
             dyn_time_constant="0.05"
@@ -112,29 +115,29 @@
     <!-- Port-Aft RL-->
      <xacro:thruster_macro thruster_id="0">
-        <origin xyz="-1.51341 0.53491 ${1.18597-0.88}" rpy="1.5708 0.0 ${1.5708+0.610865}"/>
+        <origin xyz="-1.51341 0.53491 ${1.18597-0.9}" rpy="1.5708 0.0 ${1.5708+0.610865}"/>
      </xacro:thruster_macro>
      <!-- Starboard-Aft RR -->
     <xacro:thruster_macro thruster_id="1">
-        <origin xyz="-1.51248 -0.536834 ${1.18592-0.88}" rpy="1.5708 0.0 ${1.5708-0.610865}"/>
+        <origin xyz="-1.51248 -0.536834 ${1.18592-0.9}" rpy="1.5708 0.0 ${1.5708-0.610865}"/>
     </xacro:thruster_macro>
     <!-- Port-Forward FL -->
     <xacro:thruster_macro thruster_id="2">
-        <origin xyz="1.28724 0.539848 ${1.18875-0.88}" rpy="1.5708 0.0 ${1.5708-0.610865}"/>
+        <origin xyz="1.28724 0.539848 ${1.18875-0.9}" rpy="1.5708 0.0 ${1.5708-0.610865}"/>
     </xacro:thruster_macro>
     <!-- Starboard-Forward FR-->
     <xacro:thruster_macro thruster_id="3">
-        <origin xyz="1.28841 -0.536692 ${1.1888-0.88}" rpy="1.5708 0.0 ${1.5708-2.53073}"/>
+        <origin xyz="1.28841 -0.536692 ${1.1888-0.9}" rpy="1.5708 0.0 ${1.5708-2.53073}"/>
     </xacro:thruster_macro>
     <!-- Port-Forward-Vertical TL-->
     <xacro:thruster_macro thruster_id="4">
-        <origin xyz="0.761326 ${0.02+0.706649} ${1.8604-0.88}" rpy="0.0 -0.174533 0.0"/>
+        <origin xyz="0.761326 ${0.706649} ${1.8604-0.9}" rpy="0.0 -0.174533 0.0"/>
     </xacro:thruster_macro>
     <!-- Starboard-Forward-Vertical TR-->
     <xacro:thruster_macro thruster_id="5">
-        <origin xyz="0.761276 ${-0.70968+0.02} ${1.85086-0.88}" rpy="0.0 0.174533 0.0"/>
+        <origin xyz="0.761276 ${-0.70968} ${1.85086-0.9}" rpy="0.0 0.174533 0.0"/>
     </xacro:thruster_macro>
         <!-- Aft-Vertical (central)-->
     <xacro:thruster_macro thruster_id="6">
-        <origin xyz="-1.63582 ${2.54822e-05+0.02} ${1.78479-0.88}" rpy="0.0 0.0 0.0"/>
+        <origin xyz="-1.63582 ${2.54822e-05} ${1.78479-0.9}" rpy="0.0 0.0 0.0"/>
     </xacro:thruster_macro>
     <!-- includes -->
