Commit message: move glider launch/xacros

File: urdf/robots/glider_description/urdf/glider_hybrid_whoi.xacro (robot description, xacro)
@@ -15,6 +15,6 @@
   <!-- includes -->
   <xacro:include filename="$(find uuv_descriptions)/urdf/common.urdf.xacro" />
-  <xacro:include filename="$(find uuv_dave)/urdf/sensor_snippets.xacro"/>
-  <xacro:include filename="$(find uuv_dave)/urdf/glider_hybrid_whoi_snippets.xacro"/>
+  <xacro:include filename="$(find dave_snippets)/urdf/sensor_snippets.xacro"/>
+  <xacro:include filename="$(find glider_description)/urdf/glider_hybrid_whoi_snippets.xacro"/>
   <xacro:include filename="$(find uuv_gazebo_ros_plugins)/urdf/snippets.xacro"/>
   <!-- Properties -->
@@ -29,8 +29,8 @@
   <xacro:property name="length" value="1.5" />
   <xacro:property name="namespace" value="glider_hybrid_whoi"/>
-  <xacro:property name="visual_mesh_file" value="file://$(find uuv_dave)/models/glider_hybrid_whoi/mesh/glider_hybrid_whoi_body.dae" />
-  <xacro:property name="collision_mesh_file" value="file://$(find uuv_dave)/models/glider_hybrid_whoi/mesh/glider_hybrid_whoi_collision.dae" />
-  <xacro:property name="left_prop_mesh_file" value="file://$(find uuv_dave)/models/glider_hybrid_whoi/mesh/glider_hybrid_whoi_left_propeller.dae" />
-  <xacro:property name="right_prop_mesh_file" value="file://$(find uuv_dave)/models/glider_hybrid_whoi/mesh/glider_hybrid_whoi_right_propeller.dae" />
+  <xacro:property name="visual_mesh_file" value="file://$(find glider_description)/models/glider_hybrid_whoi/mesh/glider_hybrid_whoi_body.dae" />
+  <xacro:property name="collision_mesh_file" value="file://$(find glider_description)/models/glider_hybrid_whoi/mesh/glider_hybrid_whoi_collision.dae" />
+  <xacro:property name="left_prop_mesh_file" value="file://$(find glider_description)/models/glider_hybrid_whoi/mesh/glider_hybrid_whoi_left_propeller.dae" />
+  <xacro:property name="right_prop_mesh_file" value="file://$(find glider_description)/models/glider_hybrid_whoi/mesh/glider_hybrid_whoi_right_propeller.dae" />
   <xacro:macro name="glider_hybrid_whoi" params="namespace debug inertial_reference_frame">
     <link name="${namespace}/base_link">
@@ -170,5 +170,5 @@
     <!-- TODO: Parametrize the battery unit -->
     <xacro:basic_linear_battery_macro namespace="${namespace}" parent_link="${namespace}/base_link" prefix="" open_circuit_voltage_constant_coef="3.7" open_circuit_voltage_linear_coef="-3.1424" initial_charge="1.1665" capacity="0.5" resistance="0.002" smooth_current_tau="1.9499" voltage="4.2" update_rate="2.0" />
-    <xacro:include filename="$(find uuv_dave)/urdf/glider_hybrid_whoi_sensors.xacro" />
+    <xacro:include filename="$(find glider_description)/urdf/glider_hybrid_whoi_sensors.xacro" />
   </xacro:macro>
 </robot>

File: urdf/robots/glider_description/urdf/glider_hybrid_whoi_default.urdf.xacro (robot description, xacro)
@@ -12,12 +12,12 @@
      limitations under the License.
 -->
-<robot name="glider_slocum" xmlns:xacro="http://www.ros.org/wiki/xacro" >
+<robot name="glider_hybrid_whoi" xmlns:xacro="http://www.ros.org/wiki/xacro" >
   <xacro:arg name="debug" default="0"/>
-  <xacro:arg name="namespace" default="glider_slocum"/>
+  <xacro:arg name="namespace" default="glider_hybrid_whoi"/>
   <xacro:arg name="inertial_reference_frame" default="world"/>
   <!-- Include the UUV macro file -->
-  <xacro:include filename="$(find uuv_dave)/urdf/glider_slocum.xacro"/>
-  <!-- Create the glider_slocum -->
-  <xacro:glider_slocum
+  <xacro:include filename="$(find glider_description)/urdf/glider_hybrid_whoi.xacro"/>
+  <!-- Create the glider_hybrid_whoi -->
+  <xacro:glider_hybrid_whoi
     namespace="$(arg namespace)"
     debug="$(arg debug)"

File: urdf/robots/glider_description/urdf/glider_slocum.xacro (robot description, xacro)
@@ -15,5 +15,5 @@
   <!-- includes -->
   <xacro:include filename="$(find uuv_descriptions)/urdf/common.urdf.xacro" />
-  <xacro:include filename="$(find uuv_dave)/urdf/sensor_snippets.xacro"/>
+  <xacro:include filename="$(find dave_snippets)/urdf/sensor_snippets.xacro"/>
   <xacro:include filename="$(find uuv_gazebo_ros_plugins)/urdf/snippets.xacro"/>
   <!-- Properties -->
@@ -28,8 +28,8 @@
   <xacro:property name="length" value="1.5" />
   <xacro:property name="namespace" value="glider_slocum"/>
-  <xacro:property name="visual_mesh_file" value="file://$(find uuv_dave)/models/glider_slocum/mesh/Slocum-Glider.dae" />
-  <xacro:property name="collision_mesh_file" value="file://$(find uuv_dave)/models/glider_slocum/mesh/COLLISION-Slocum-Glider.dae" />
-  <!--<xacro:property name="prop_mesh_file" value="file://$(find uuv_dave)/models/glider_slocum/mesh/Slocum-Glider-Propeller.dae" />-->
-  <!-- <xacro:property name="rudder_mesh_file" value="file://$(find uuv_dave)/models/glider_slocum/mesh/Slocum-Glider-TopRudder.dae" /> -->
+  <xacro:property name="visual_mesh_file" value="file://$(find glider_description)/models/glider_slocum/mesh/Slocum-Glider.dae" />
+  <xacro:property name="collision_mesh_file" value="file://$(find glider_description)/models/glider_slocum/mesh/COLLISION-Slocum-Glider.dae" />
+  <!--<xacro:property name="prop_mesh_file" value="file://$(find glider_description)/models/glider_slocum/mesh/Slocum-Glider-Propeller.dae" />-->
+  <!-- <xacro:property name="rudder_mesh_file" value="file://$(find glider_description)/models/glider_slocum/mesh/Slocum-Glider-TopRudder.dae" /> -->
   <xacro:macro name="glider_slocum" params="namespace debug inertial_reference_frame">
     <link name="${namespace}/base_link">
@@ -98,5 +98,5 @@
       update_rate="2.0"/>
     <!-- Include sensor modules -->
-    <xacro:include filename="$(find uuv_dave)/urdf/glider_slocum_sensors.xacro"/>
+    <xacro:include filename="$(find glider_description)/urdf/glider_slocum_sensors.xacro"/>
   </xacro:macro>
 </robot>

File: urdf/robots/glider_description/urdf/glider_slocum_default.urdf.xacro (robot description, xacro)
@@ -12,12 +12,12 @@
      limitations under the License.
 -->
-<robot name="glider_hybrid_whoi" xmlns:xacro="http://www.ros.org/wiki/xacro" >
+<robot name="glider_slocum" xmlns:xacro="http://www.ros.org/wiki/xacro" >
   <xacro:arg name="debug" default="0"/>
-  <xacro:arg name="namespace" default="glider_hybrid_whoi"/>
+  <xacro:arg name="namespace" default="glider_slocum"/>
   <xacro:arg name="inertial_reference_frame" default="world"/>
   <!-- Include the UUV macro file -->
-  <xacro:include filename="$(find uuv_dave)/urdf/glider_hybrid_whoi.xacro"/>
-  <!-- Create the glider_hybrid_whoi -->
-  <xacro:glider_hybrid_whoi
+  <xacro:include filename="$(find glider_description)/urdf/glider_slocum.xacro"/>
+  <!-- Create the glider_slocum -->
+  <xacro:glider_slocum
     namespace="$(arg namespace)"
     debug="$(arg debug)"

File: urdf/robots/glider_description/urdf/glider_wave.xacro (robot description, xacro)
@@ -15,6 +15,6 @@
   <!-- includes -->
   <xacro:include filename="$(find uuv_descriptions)/urdf/common.urdf.xacro" />
-  <xacro:include filename="$(find uuv_dave)/urdf/sensor_snippets.xacro" />
-  <xacro:include filename="$(find uuv_dave)/urdf/glider_wave_snippets.xacro" />
+  <xacro:include filename="$(find dave_snippets)/urdf/sensor_snippets.xacro" />
+  <xacro:include filename="$(find glider_description)/urdf/glider_wave_snippets.xacro" />
   <xacro:include filename="$(find uuv_gazebo_ros_plugins)/urdf/snippets.xacro" />
   <!-- Properties -->
@@ -31,11 +31,11 @@
   <xacro:property name="length" value="1.5" />
   <xacro:property name="namespace" value="glider_wave" />
-  <xacro:property name="visual_mesh_file" value="file://$(find uuv_dave)/models/glider_wave/mesh/Wave Glider-Float.dae" />
-  <xacro:property name="collision_mesh_file" value="file://$(find uuv_dave)/models/glider_wave/mesh/COLLISION-Wave Glider-float.dae" />
-  <xacro:property name="sub_visual_mesh_file" value="file://$(find uuv_dave)/models/glider_wave/mesh/Wave Glider-Sub.dae" />
-  <xacro:property name="sub_collision_mesh_file" value="file://$(find uuv_dave)/models/glider_wave/mesh/COLLISION-Wave Glider-sub.dae" />
-  <xacro:property name="umbilicaljoint_visual_mesh_file" value="file://$(find uuv_dave)/models/glider_wave/mesh/Wave Glider-Joint.dae" />
-  <xacro:property name="umbilical_visual_mesh_file" value="file://$(find uuv_dave)/models/glider_wave/mesh/Wave Glider-Umbilical.dae" />
-  <xacro:property name="umbilical_collision_mesh_file" value="file://$(find uuv_dave)/models/glider_wave/mesh/COLLISION-Wave Glider-umbilical.dae" />
+  <xacro:property name="visual_mesh_file" value="file://$(find glider_description)/models/glider_wave/mesh/Wave Glider-Float.dae" />
+  <xacro:property name="collision_mesh_file" value="file://$(find glider_description)/models/glider_wave/mesh/COLLISION-Wave Glider-float.dae" />
+  <xacro:property name="sub_visual_mesh_file" value="file://$(find glider_description)/models/glider_wave/mesh/Wave Glider-Sub.dae" />
+  <xacro:property name="sub_collision_mesh_file" value="file://$(find glider_description)/models/glider_wave/mesh/COLLISION-Wave Glider-sub.dae" />
+  <xacro:property name="umbilicaljoint_visual_mesh_file" value="file://$(find glider_description)/models/glider_wave/mesh/Wave Glider-Joint.dae" />
+  <xacro:property name="umbilical_visual_mesh_file" value="file://$(find glider_description)/models/glider_wave/mesh/Wave Glider-Umbilical.dae" />
+  <xacro:property name="umbilical_collision_mesh_file" value="file://$(find glider_description)/models/glider_wave/mesh/COLLISION-Wave Glider-umbilical.dae" />
   <xacro:macro name="glider_wave" params="namespace debug inertial_reference_frame">
     <link name="${namespace}/base_link">
@@ -194,5 +194,5 @@
       </plugin> -->
     </gazebo>
-    <xacro:include filename="$(find uuv_dave)/urdf/glider_wave_sensors.xacro" />
+    <xacro:include filename="$(find glider_description)/urdf/glider_wave_sensors.xacro" />
   </xacro:macro>
 </robot>

File: urdf/robots/glider_description/urdf/glider_wave_default.urdf.xacro (robot description, xacro)
@@ -17,5 +17,5 @@
   <xacro:arg name="inertial_reference_frame" default="world"/>
   <!-- Include the UUV macro file -->
-  <xacro:include filename="$(find uuv_dave)/urdf/glider_wave.xacro"/>
+  <xacro:include filename="$(find glider_description)/urdf/glider_wave.xacro"/>
   <!-- Create the glider_wave_ -->
   <xacro:glider_wave

Commit message: Fixed a couple of conflicts after rebasing on origin/master
Also fixed a couple of mesh paths in the glider demos.

All demos in the "examples" directories have been retested and seem
to be working ok.

File: urdf/robots/glider_description/urdf/glider_hybrid_whoi.xacro (robot description, xacro)
@@ -29,8 +29,8 @@
   <xacro:property name="length" value="1.5" />
   <xacro:property name="namespace" value="glider_hybrid_whoi"/>
-  <xacro:property name="visual_mesh_file" value="file://$(find glider_description)/models/glider_hybrid_whoi/mesh/glider_hybrid_whoi_body.dae" />
-  <xacro:property name="collision_mesh_file" value="file://$(find glider_description)/models/glider_hybrid_whoi/mesh/glider_hybrid_whoi_collision.dae" />
-  <xacro:property name="left_prop_mesh_file" value="file://$(find glider_description)/models/glider_hybrid_whoi/mesh/glider_hybrid_whoi_left_propeller.dae" />
-  <xacro:property name="right_prop_mesh_file" value="file://$(find glider_description)/models/glider_hybrid_whoi/mesh/glider_hybrid_whoi_right_propeller.dae" />
+  <xacro:property name="visual_mesh_file" value="file://$(find dave_robot_models)/models/glider_hybrid_whoi/mesh/glider_hybrid_whoi_body.dae" />
+  <xacro:property name="collision_mesh_file" value="file://$(find dave_robot_models)/models/glider_hybrid_whoi/mesh/glider_hybrid_whoi_collision.dae" />
+  <xacro:property name="left_prop_mesh_file" value="file://$(find dave_robot_models)/models/glider_hybrid_whoi/mesh/glider_hybrid_whoi_left_propeller.dae" />
+  <xacro:property name="right_prop_mesh_file" value="file://$(find dave_robot_models)/models/glider_hybrid_whoi/mesh/glider_hybrid_whoi_right_propeller.dae" />
   <xacro:macro name="glider_hybrid_whoi" params="namespace debug inertial_reference_frame">
     <link name="${namespace}/base_link">

File: urdf/robots/glider_description/urdf/glider_slocum.xacro (robot description, xacro)
@@ -28,8 +28,8 @@
   <xacro:property name="length" value="1.5" />
   <xacro:property name="namespace" value="glider_slocum"/>
-  <xacro:property name="visual_mesh_file" value="file://$(find glider_description)/models/glider_slocum/mesh/Slocum-Glider.dae" />
-  <xacro:property name="collision_mesh_file" value="file://$(find glider_description)/models/glider_slocum/mesh/COLLISION-Slocum-Glider.dae" />
-  <!--<xacro:property name="prop_mesh_file" value="file://$(find glider_description)/models/glider_slocum/mesh/Slocum-Glider-Propeller.dae" />-->
-  <!-- <xacro:property name="rudder_mesh_file" value="file://$(find glider_description)/models/glider_slocum/mesh/Slocum-Glider-TopRudder.dae" /> -->
+  <xacro:property name="visual_mesh_file" value="file://$(find dave_robot_models)/models/glider_slocum/mesh/Slocum-Glider.dae" />
+  <xacro:property name="collision_mesh_file" value="file://$(find dave_robot_models)/models/glider_slocum/mesh/COLLISION-Slocum-Glider.dae" />
+  <!--<xacro:property name="prop_mesh_file" value="file://$(find dave_robot_models)/models/glider_slocum/mesh/Slocum-Glider-Propeller.dae" />-->
+  <!-- <xacro:property name="rudder_mesh_file" value="file://$(find dave_robot_models)/models/glider_slocum/mesh/Slocum-Glider-TopRudder.dae" /> -->
   <xacro:macro name="glider_slocum" params="namespace debug inertial_reference_frame">
     <link name="${namespace}/base_link">

File: urdf/robots/glider_description/urdf/glider_wave.xacro (robot description, xacro)
@@ -31,11 +31,11 @@
   <xacro:property name="length" value="1.5" />
   <xacro:property name="namespace" value="glider_wave" />
-  <xacro:property name="visual_mesh_file" value="file://$(find glider_description)/models/glider_wave/mesh/Wave Glider-Float.dae" />
-  <xacro:property name="collision_mesh_file" value="file://$(find glider_description)/models/glider_wave/mesh/COLLISION-Wave Glider-float.dae" />
-  <xacro:property name="sub_visual_mesh_file" value="file://$(find glider_description)/models/glider_wave/mesh/Wave Glider-Sub.dae" />
-  <xacro:property name="sub_collision_mesh_file" value="file://$(find glider_description)/models/glider_wave/mesh/COLLISION-Wave Glider-sub.dae" />
-  <xacro:property name="umbilicaljoint_visual_mesh_file" value="file://$(find glider_description)/models/glider_wave/mesh/Wave Glider-Joint.dae" />
-  <xacro:property name="umbilical_visual_mesh_file" value="file://$(find glider_description)/models/glider_wave/mesh/Wave Glider-Umbilical.dae" />
-  <xacro:property name="umbilical_collision_mesh_file" value="file://$(find glider_description)/models/glider_wave/mesh/COLLISION-Wave Glider-umbilical.dae" />
+  <xacro:property name="visual_mesh_file" value="file://$(find dave_robot_models)/models/glider_wave/mesh/Wave Glider-Float.dae" />
+  <xacro:property name="collision_mesh_file" value="file://$(find dave_robot_models)/models/glider_wave/mesh/COLLISION-Wave Glider-float.dae" />
+  <xacro:property name="sub_visual_mesh_file" value="file://$(find dave_robot_models)/models/glider_wave/mesh/Wave Glider-Sub.dae" />
+  <xacro:property name="sub_collision_mesh_file" value="file://$(find dave_robot_models)/models/glider_wave/mesh/COLLISION-Wave Glider-sub.dae" />
+  <xacro:property name="umbilicaljoint_visual_mesh_file" value="file://$(find dave_robot_models)/models/glider_wave/mesh/Wave Glider-Joint.dae" />
+  <xacro:property name="umbilical_visual_mesh_file" value="file://$(find dave_robot_models)/models/glider_wave/mesh/Wave Glider-Umbilical.dae" />
+  <xacro:property name="umbilical_collision_mesh_file" value="file://$(find dave_robot_models)/models/glider_wave/mesh/COLLISION-Wave Glider-umbilical.dae" />
   <xacro:macro name="glider_wave" params="namespace debug inertial_reference_frame">
     <link name="${namespace}/base_link">

Commit message: scaling glider meshes to match physical dimensions

File: urdf/robots/glider_description/urdf/glider_hybrid_whoi.xacro (robot description, xacro)
@@ -38,5 +38,5 @@
         <origin xyz="0 0 0" rpy="0 0 -1.5708" />
         <geometry>
-          <mesh filename="${visual_mesh_file}" scale="1 1 1" />
+          <mesh filename="${visual_mesh_file}" scale="2.3 2.3 2.3" />
         </geometry>
       </visual>
@@ -44,5 +44,5 @@
         <origin xyz="0 0 0" rpy="0 0 -1.5708" />
         <geometry>
-          <mesh filename="${collision_mesh_file}" scale="1 1 1" />
+          <mesh filename="${collision_mesh_file}" scale="2.3 2.3 2.3" />
         </geometry>
       </collision>
@@ -57,5 +57,5 @@
         <origin xyz="0 0 0" rpy="0 0 0 " />
         <geometry>
-          <mesh filename="${left_prop_mesh_file}" scale="1 1 1" />
+          <mesh filename="${left_prop_mesh_file}" scale="2.3 2.3 2.3" />
         </geometry>
       </visual>
@@ -71,5 +71,5 @@
         <origin xyz="0 0 0" rpy="0 0 0" />
         <geometry>
-          <mesh filename="${right_prop_mesh_file}" scale="1 1 1" />
+          <mesh filename="${right_prop_mesh_file}" scale="2.3 2.3 2.3" />
         </geometry>
       </visual>

File: urdf/robots/glider_description/urdf/glider_slocum.xacro (robot description, xacro)
@@ -37,5 +37,5 @@
         <origin xyz="0 0 0" rpy="0 0 -1.5708" />
         <geometry>
-          <mesh filename="${visual_mesh_file}" scale="1 1 1" />
+          <mesh filename="${visual_mesh_file}" scale="0.5 0.5 0.5" />
         </geometry>
       </visual>
@@ -43,5 +43,5 @@
         <origin xyz="0 0 0" rpy="0 0 -1.5708" />
         <geometry>
-          <mesh filename="${collision_mesh_file}" scale="1 1 1" />
+          <mesh filename="${collision_mesh_file}" scale="0.5 0.5 0.5" />
         </geometry>
       </collision>
